File: src/HardwareDesign/HW_RPI_DAQ.brd (EAGLE design)
At the start: 155 x 100 mm, 65 parts, among them IC2 AP22653W6, IC3 74LVC1G07, IC4 RT9742NGV, J1 10164227-1001A1RLF, J2 10164227-1001A1RLF, J3 692141030100, J4 685119136923, J5 685119136923, J6 629722000214, X1 ASEK-32.768KHz-LRT

Commit message: add DAQ to design
Parts:
- removed U$3: M.2, ds_con:M.2
- added C100, C101: 10pF, ds_passive:0402
- added C102, C104: 10uF, ds_passive:1206
- added C103, C106, C107: 10nF, ds_passive:0402
- added C105, C99: 220nF, ds_passive:0402
- added C108, C109, C93, C94, C95, C96, C97, C98: 22uF, ds_passive:1206
- added C110, C47, C70, C90: 10uF, ds_passive:0805
- added C111, C123, C152, C154, C156, C158, C160, C162, C164, C166, C168, C170, C171, C51, C53, C55, C57, C59, C61, C63, C65, C67, C69, C71, C73: 100nF, ds_passive:0603
- added C114, C116, C120, C121, C125, C126, C128, C129, C131, C132, C134, C135, C137, C138, C140, C141, C143, C144, C146, C147, C149, C150, C45, C46, C49, C75, C76: 100nF, ds_passive:0402
- added C115, C117: 4.7uF, ds_passive:0603
- added C118, C119: 100uF, rcl:153CLV-0605
- added C122, C124, C151, C153, C155, C157, C159, C161, C163, C165, C167, C169, C50, C52, C54, C56, C58, C60, C62, C64, C66, C68, C72: 1uF, ds_passive:0603
- added C127, C130, C133, C136, C139, C142, C145, C148: 20nF, ds_passive:0402
- added C23, C24, C42, C43: 270pF, ds_passive:0402
- added C41, C44: 680pF, ds_passive:0402
- added C48, C74: (no value), ds_passive:0805
- added C85: 4.7uF, ds_passive:0805
- added C86: 100nF, ds_passive:0805
- added C91: 10nF, ds_passive:0805
- added C92: 4.7nF, ds_passive:0805
- added D3, D4: SS12, Diodes:SMA
- added IC10: ADS9234RIRHBR, ds_ic_peripherals:VQFN32-5X5
- added IC11, IC13, IC23, IC24, IC25, IC26, IC27, IC28, IC29, IC30, IC31: MCP6001RT, ds_ic_opa:SOT23-5
- added IC12: REF3025, maxim:SOT23
- added IC14: TPS65131, ds_ic_vreg:VQFN24-4X4-THERMAL2.5X2.5
- added IC15: TPS7A39, ds_ic_vreg:WSON10-3X3
- added IC20: MIC5504-3.3YM5-TR, ds_ic_vreg:SOT23-5
- added IC21: LD117ADT33TR, v-reg:DPACK
- added IC22: DAC8568, ds_ic_peripherals:TSSOP16
- added IC32, IC33, IC34, IC35: LSF0108, ds_ic_peripherals:VQFN20
- added IC36: MCP23S18, ds_ic_peripherals:QFN50P400X400X100-25T265
- added IC37: (no value), ds_ic_peripherals:QFN50P400X400X100-25T265
- added IC38: (no value), ds_ic_peripherals:SOP50P310X90-8N
- added IC39: 74LVC1G04, ds_ic_logic:SOT95P280X145-5N
- added IC6, IC8: DG409, ds_ic_peripherals:TSSOP16
- added IC7, IC9: ADA4254ACPZ, ds_ic_opa:QFN50P500X500X75-29T314N
- added L3, L4: B8246284-4.7uH, inductor-coilcraft:MSS7341
- added R100, R103, R104, R107, R108, R111, R112, R115, R116, R73, R76, R87, R88, R91, R92, R95, R96, R99: 10K 0.1%, ds_passive:0402
- added R101, R105, R109, R113, R117, R89, R93, R97: 43K 0.1%, ds_passive:0402
- added R102, R106, R110, R114, R118, R90, R94, R98: 68R 1%, ds_passive:0402
- added R119, R120, R121, R122, R123, R124, R125, R126: YC164-JR-0733RL, Resistor Array:YC164-JR-0733RL
- added R127, R128, R129, R130: 200K, ds_passive:0402
- added R14: 100R, ds_passive:1206
- added R15, R17, R18, R81, R82: 0R, ds_passive:0402
- added R16: 10K, ds_passive:0402
- added R19: 950K 0.1%, ds_passive:0402
- added R20, R21, R22, R23: 200R, ds_passive:0402
- added R24, R42, R43, R44, R45, R46, R47, R48, R51, R52: 0R, ds_passive:0603
- added R49, R77, R78: 20K, pot:3223G
- added R50: 100R, ds_passive:0402
- added R57: 102K 0.1%, ds_passive:0402
- added R58: 1.2M 0.1%, ds_passive:0402
- added R59: 137K 0.1%, ds_passive:0402
- added R60: 75K 0.1%, ds_passive:0402
- added R74: 90K 0.1%, ds_passive:0402
- added R79, R80: 250K, pot:3223G
- added R86: CRA034RF100RP05Z, Resistor Array:YC164-JR-0733RL
- added T2: IRLML5203, transistor-power:MICRO3
- added TP100, TP101, TP102, TP103, TP104, TP105, TP106, TP17, TP18, TP19, TP20, TP21, TP22, TP23, TP24, TP25, TP26, TP27, TP28, TP29, TP30, TP31, TP32, TP33, TP34, TP35, TP36, TP37, TP38, TP39, TP40, TP46, TP47, TP48, TP49, TP50, TP51, TP53, TP54, TP55, TP56, TP57, TP80, TP81, TP82, TP83, TP84, TP85, TP89, TP90, TP91, TP92, TP93, TP94, TP95, TP96, TP97, TP98, TP99: PTR1B1,27, testpad:B1,27
- moved BT1 57.7 mm to (-2.10, 121.8)
Connections:
- new net !ADC_RST: IC10.26, R16.2, TP39.TP
- new net !CS1_ADC: IC10.14, R15.1, TP40.TP
- new net !CS_ADA_A: IC7.11
- new net !CS_ADA_B: IC9.11
- new net !DIO_LEVEL_SELECT: IC38.3, IC39.4
- new net +12V: C107.2, C108.1, IC15.10, R60.1, TP53.TP
- new net +14V: C100.1, C104.1, C93.1, C94.1, C95.1, D3.C, IC14.23, IC15.1, IC15.2, R19.1, TP46.TP
- new net +3V3_EXT: C119.+, C121.1, IC21.4
- new net -12V: C106.1, C109.1, IC15.6, R76.2, TP54.TP
- new net -14V: C101.1, C102.1, C96.1, C97.1, C98.1, D4.A, IC14.15, IC15.5, R59.2, TP47.TP
- new net ADA_A_IO0: IC6.1, IC7.18
- new net ADA_A_IO1: IC6.16, IC7.17
- new net ADA_A_IO2: IC6.2, IC7.16
- new net ADA_B_IO0: IC8.1, IC9.18
- new net ADA_B_IO1: IC8.16, IC9.17
- new net ADA_B_IO2: IC8.2, IC9.16
- new net ADC_AIN_N: C24.2, C41.2, R21.1, R46.1, TP22.TP
- new net ADC_AIN_P: C23.1, C41.1, R20.1, R45.2, TP21.TP
- new net ADC_BIN_N: C43.2, C44.2, R23.1, R48.2, TP24.TP
- new net ADC_BIN_P: C42.1, C44.1, R22.1, R47.1, TP23.TP
- new net ADC_IN0: IC10.1, R45.1, TP17.TP
- new net ADC_IN1: IC10.2, R46.2, TP18.TP
- new net ADC_IN2: IC10.8, R48.1, TP19.TP
- new net ADC_IN3: IC10.7, R47.2, TP20.TP
- new net ADC_RDY: IC10.25, TP28.TP
- new net AO_0: C127.1, R89.2, R90.2
- new net AO_1: C130.1, R93.2, R94.2
- new net AO_2: C133.1, R97.2, R98.2
- new net AO_3: C136.1, R101.2, R102.2
- new net AO_4: C139.1, R105.2, R106.2
- new net AO_5: C142.1, R109.2, R110.2
- new net AO_6: C145.1, R113.2, R114.2
- new net AO_7: C148.1, R117.2, R118.2
- new net BSW_G: IC14.7, T2.1, TP51.TP
- new net BUF: C105.2, IC15.8, R74.1, TP57.TP
- new net DAC_!CLR: IC22.9, R86.1, TP93.TP
- new net DAC_!LDAC: IC22.1, R86.3, TP89.TP
- new net DAC_!SYNC: IC22.2, R86.2, TP91.TP
- new net DAC_0: IC22.4, IC24.3, TP90.TP
- new net DAC_1: IC22.13, IC25.3, TP92.TP
- new net DAC_2: IC22.5, IC26.3, TP94.TP
- new net DAC_3: IC22.12, IC27.3, TP96.TP
- new net DAC_4: IC22.6, IC28.3, TP97.TP
- new net DAC_5: IC22.11, IC29.3, TP98.TP
- new net DAC_6: IC22.7, IC30.3, TP99.TP
- new net DAC_7: IC22.10, IC31.3, TP100.TP
- new net DIO_0: R119.8
- new net DIO_1: R119.7
- new net DIO_10: R121.6
- new net DIO_11: R121.5
- new net DIO_12: R122.8
- new net DIO_13: R122.7
- new net DIO_14: R122.6
- new net DIO_15: R122.5
- new net DIO_16: R123.8
- new net DIO_17: R123.7
- new net DIO_18: R123.6
- new net DIO_19: R123.5
- new net DIO_2: R119.6
- new net DIO_20: R124.8
- new net DIO_21: R124.7
- new net DIO_22: R124.6
- new net DIO_23: R124.5
- new net DIO_24: R125.8
- new net DIO_25: R125.7
- new net DIO_26: R125.6
- new net DIO_27: R125.5
- new net DIO_28: R126.8
- new net DIO_29: R126.7
- new net DIO_3: R119.5
- new net DIO_30: R126.6
- new net DIO_31: R126.5
- new net DIO_4: R120.8
- new net DIO_5: R120.7
- new net DIO_6: R120.6
- new net DIO_7: R120.5
- new net DIO_8: R121.8
- new net DIO_9: R121.7
- new net DIO_CS1: IC36.9, TP104.TP
- new net DIO_CS2: IC37.9
- new net DIO_EN: IC32.20, IC33.20, IC34.20, IC35.20, TP103.TP
- new net DIO_LEVEL_SELECT: IC38.7, IC39.2, TP101.TP, TP106.TP
- new net DIO_RESET: IC36.13, IC37.13, TP105.TP
- new net IN0+: IC6.4
- new net IN1-: IC6.13
- new net IN10+: IC8.5
- new net IN11-: IC8.12
- new net IN12+: IC8.6
- new net IN13-: IC8.11
- new net IN14+: IC8.7
- new net IN15-: IC8.10
- new net IN2+: IC6.5
- new net IN3-: IC6.12
- new net IN4+: IC6.6
- new net IN5-: IC6.11
- new net IN6+: IC6.7
- new net IN7-: IC6.10
- new net IN8+: IC8.4
- new net IN9-: IC8.13
- new net MISO: IC36.12, IC37.12, IC7.8, IC9.8
- new net MOSI: IC10.15, IC22.15, IC36.11, IC37.11, IC7.9, IC9.9
- new net MUX_A_OUTA: IC6.8, R43.2, TP33.TP
- new net MUX_A_OUTB: IC6.9, R44.1, TP34.TP
- new net MUX_B_OUTA: IC8.8, R24.2, TP35.TP
- new net MUX_B_OUTB: IC8.9, R42.1, TP36.TP
- new net N$100: IC34.18, R123.1
- new net N$101: IC34.17, R123.2
- new net N$102: IC34.16, R123.3
- new net N$103: IC34.15, R123.4
- new net N$104: IC34.14, R124.1
- new net N$105: IC34.13, R124.2
- new net N$106: IC34.12, R124.3
- new net N$107: IC34.11, R124.4
- new net N$108: IC35.5, IC37.2
- new net N$109: IC35.6, IC37.3
- new net N$110: IC35.7, IC37.4
- new net N$111: IC35.8, IC37.5
- new net N$112: IC35.9, IC37.6
- new net N$113: IC35.10, IC37.7
- new net N$114: IC35.4, IC37.1
- new net N$115: IC35.3, IC37.24
- new net N$116: IC35.18, R125.1
- new net N$117: IC35.17, R125.2
- new net N$118: IC35.16, R125.3
- new net N$119: IC35.15, R125.4
- new net N$12: IC7.19, R20.2
- new net N$120: IC35.14, R126.1
- new net N$121: IC35.13, R126.2
- new net N$122: IC35.12, R126.3
- new net N$123: IC35.11, R126.4
- new net N$124: IC32.19, R127.1
- new net N$125: IC33.19, R128.1
- new net N$126: IC35.19, R129.1
- new net N$127: IC34.19, R130.1
- new net N$13: IC7.20, R21.2
- new net N$14: C129.2, IC24.1, R90.1
- new net N$15: IC9.19, R22.2
- new net N$16: IC9.20, R23.2
- new net N$17: C129.1, IC24.4, R87.2, R88.2, R89.1
- new net N$18: IC10.13, R15.2
- new net N$19: C72.2, C73.2, R49.1
- new net N$20: C74.1, R49.2, R50.1
- new net N$21: IC11.3, R50.2
- new net N$22: C132.1, IC25.4, R91.2, R92.2, R93.1
- new net N$23: C132.2, IC25.1, R94.1
- new net N$24: D3.A, IC14.1, IC14.24, L3.2
- new net N$25: C135.1, IC26.4, R95.2, R96.2, R97.1
- new net N$26: C135.2, IC26.1, R98.1
- new net N$27: C138.1, IC27.4, R100.2, R101.1, R99.2
- new net N$28: C138.2, IC27.1, R102.1
- new net N$29: IC33.4, IC36.1
- new net N$30: C90.1, L3.1, T2.3
- new net N$31: C141.1, IC28.4, R103.2, R104.2, R105.1
- new net N$32: C86.1, IC14.10, IC14.11, IC14.4, IC14.8, IC14.9, R14.1
- new net N$33: C141.2, IC28.1, R106.1
- new net N$34: C144.1, IC29.4, R107.2, R108.2, R109.1
- new net N$35: C91.1, IC14.21
- new net N$36: C92.1, IC14.18
- new net N$37: D4.C, IC14.13, IC14.14, L4.2
- new net N$38: R60.2, R77.2, R77.3
- new net N$39: C103.1, IC15.3
- new net N$40: C144.2, IC29.1, R110.1
- new net N$41: C147.1, IC30.4, R111.2, R112.2, R113.1
- new net N$42: R74.2, R78.2, R78.3
- new net N$43: R19.2, R79.2, R79.3
- new net N$44: R58.2, R80.2, R80.3
- new net N$58: C147.2, IC30.1, R114.1
- new net N$59: C150.1, IC31.4, R115.2, R116.2, R117.1
- new net N$60: C150.2, IC31.1, R118.1
- new net N$61: IC32.3, IC36.15
- new net N$62: IC32.4, IC36.16
- new net N$63: IC32.5, IC36.17
- new net N$64: IC32.6, IC36.18
- new net N$65: IC32.7, IC36.19
- new net N$66: IC32.8, IC36.20
- new net N$67: IC32.9, IC36.21
- new net N$68: IC32.10, IC36.22
- new net N$69: IC32.18, R119.1
- new net N$70: IC32.17, R119.2
- new net N$71: IC32.16, R119.3
- new net N$72: IC32.15, R119.4
- new net N$73: IC32.14, R120.1
- new net N$74: IC32.13, R120.2
- new net N$75: IC32.12, R120.3
- new net N$76: IC32.11, R120.4
- new net N$77: IC33.3, IC36.24
- new net N$78: IC33.5, IC36.2
- new net N$79: IC33.6, IC36.3
- new net N$80: IC33.7, IC36.4
- new net N$81: IC33.8, IC36.5
- new net N$82: IC33.9, IC36.6
- new net N$83: IC33.10, IC36.7
- new net N$84: IC33.18, R121.1
- new net N$85: IC33.17, R121.2
- new net N$86: IC33.16, R121.3
- new net N$87: IC33.15, R121.4
- new net N$88: IC33.14, R122.1
- new net N$89: IC33.13, R122.2
- new net N$90: IC33.12, R122.3
- new net N$91: IC33.11, R122.4
- new net N$92: IC34.3, IC37.15
- new net N$93: IC34.4, IC37.16
- new net N$94: IC34.5, IC37.17
- new net N$95: IC34.6, IC37.18
- new net N$96: IC34.7, IC37.19
- new net N$97: IC34.8, IC37.20
- new net N$98: IC34.9, IC37.21
- new net N$99: IC34.10, IC37.22
- new net PGA_A_IN+: IC7.1, R43.1, TP29.TP
- new net PGA_A_IN-: IC7.2, IC7.3, R44.2, TP30.TP
- new net PGA_B_IN+: IC9.1, R24.1, TP31.TP
- new net PGA_B_IN-: IC9.2, IC9.3, R42.2, TP32.TP
- new net REFBY2: C71.1, IC10.3, TP85.TP
- new net REFM_A: C70.2, IC10.32, TP81.TP
- new net REFM_B: C110.2, IC10.9, TP83.TP
- new net REFOUT: C111.1, IC10.5, TP84.TP
- new net REFP_A: C70.1, IC10.31, TP80.TP
- new net REFP_B: C110.1, IC10.10, TP82.TP
- new net SCK: IC10.16, IC22.16, IC36.10, IC37.10, IC7.10, IC9.10
- new net SDO_A_0: IC10.24, R17.2
- new net SDO_A_1: IC10.23, R18.2
- new net SDO_A_2: IC10.22, R81.2
- new net SDO_A_3: IC10.21, R82.2
- new net SDO_B_0: IC10.20, R17.1
- new net SDO_B_1: IC10.19, R18.1
- new net SDO_B_2: IC10.18, R81.1
- new net SDO_B_3: IC10.17, R82.1
- new net V+: C52.1, C53.1, C56.1, C57.1, C60.1, C61.1, C66.1, C67.1, IC6.14, IC7.26, IC8.14, IC9.26
- new net V-: C54.1, C55.1, C58.1, C59.1, C62.1, C63.1, C68.1, C69.1, IC6.3, IC7.27, IC7.29, IC8.3, IC9.27, IC9.29
- new net VFB_12VN: C106.2, IC15.7, R76.1, R78.1, TP56.TP
- new net VFB_12VP: C107.1, IC15.9, R73.1, R77.1, TP55.TP
- new net VFB_14VN: C101.2, IC14.16, R59.1, R80.1, TP49.TP
- new net VFB_14VP: C100.2, IC14.22, R57.1, R79.1, TP48.TP
- new net VOCM_A: IC7.21, R51.2, TP37.TP
- new net VOCM_B: IC9.21, R52.1, TP38.TP
- new net VREF_ADC: C46.1, C72.1, C73.1, IC13.1, IC13.4, IC7.23, IC9.23, R49.3, TP25.TP
- new net VREF_ADC/2: C75.1, IC11.1, IC11.4, R51.1, R52.2, TP27.TP
- new net VREF_ADC_RAW: C48.1, IC12.2, IC13.3, TP26.TP
- new net VREF_DAC: C125.1, IC23.1, IC23.4, R100.1, R104.1, R108.1, R112.1, R116.1, R88.1, R92.1, R96.1
- new net VREF_DAC_OUT: C124.1, IC22.8, IC23.3, TP95.TP
- new net VREF_TPS: C99.2, IC14.17, R58.1, TP50.TP
- new net V_OUT_REF: C153.1, C154.1, C157.1, C158.1, C161.1, C162.1, C165.1, C166.1, IC38.2, IC38.6, R127.2, R128.2, R129.2, R130.2, TP102.TP
- net +3V3: now also C116.1, C117.1, C122.1, C123.1, C126.1, C128.1, C131.1, C134.1, C137.1, C140.1, C143.1, C146.1, C149.1, C151.1, C152.1, C155.1, C156.1, C159.1, C160.1, C163.1, C164.1, C167.1, C168.1, C169.1, C170.1, C171.1, C45.1, C47.1, C49.1, C50.1, C51.1, C64.1, C65.1, C76.1, IC10.12, IC10.28, IC10.29, IC11.2, IC12.1, IC13.2, IC20.5, IC22.3, IC23.2, IC24.2, IC25.2, IC26.2, IC27.2, IC28.2, IC29.2, IC30.2, IC31.2, IC32.2, IC33.2, IC34.2, IC35.2, IC36.8, IC37.8, IC38.1, IC38.8, IC39.5, IC7.7, IC9.7, R16.1, R86.6, R86.7, R86.8
- net +5V: now also C114.1, C115.1, C118.+, C120.1, C85.1, IC14.5, IC14.6, IC20.1, IC20.3, IC21.3, IC38.5, R14.2, T2.2
- net GND: now also C102.2, C103.2, C104.2, C105.1, C108.2, C109.2, C111.2, C114.2, C115.2, C116.2, C117.2, C118.-, C119.-, C120.2, C121.2, C122.2, C123.2, C124.2, C125.2, C126.2, C127.2, C128.2, C130.2, C131.2, C133.2, C134.2, C136.2, C137.2, C139.2, C140.2, C142.2, C143.2, C145.2, C146.2, C148.2, C149.2, C151.2, C152.2, C153.2, C154.2, C155.2, C156.2, C157.2, C158.2, C159.2, C160.2, C161.2, C162.2, C163.2, C164.2, C165.2, C166.2, C167.2, C168.2, C169.2, C170.2, C171.2, C23.2, C24.1, C42.2, C43.1, C45.2, C46.2, C47.2, C48.2, C49.2, C50.2, C51.2, C52.2, C53.2, C54.2, C55.2, C56.2, C57.2, C58.2, C59.2, C60.2, C61.2, C62.2, C63.2, C64.2, C65.2, C66.2, C67.2, C68.2, C69.2, C71.2, C74.2, C75.2, C76.2, C85.2, C86.2, C90.2, C91.2, C92.2, C93.2, C94.2, C95.2, C96.2, C97.2, C98.2, C99.1, IC10.11, IC10.27, IC10.30, IC10.33, IC10.4, IC11.5, IC12.3, IC13.5, IC14.19, IC14.2, IC14.25, IC14.3, IC15.4, IC15.PAD, IC15.PAD1, IC15.PAD2, IC15.PAD3, IC15.PAD4, IC20.2, IC21.1, IC22.14, IC23.5, IC24.5, IC25.5, IC26.5, IC27.5, IC28.5, IC29.5, IC30.5, IC31.5, IC32.1, IC32.PAD, IC33.1, IC33.PAD, IC34.1, IC34.PAD, IC35.1, IC35.PAD, IC36.23, IC36.25, IC37.23, IC37.25, IC38.4, IC39.3, IC6.15, IC7.22, IC7.24, IC7.25, IC7.4, IC7.6, IC8.15, IC9.22, IC9.24, IC9.25, IC9.4, IC9.6, L4.1, R103.1, R107.1, R111.1, R115.1, R57.2, R73.2, R87.1, R91.1, R95.1, R99.1
Routing:
- net +14V: track 0.00 -> 170.5 mm
- net GND: track 880.0 -> 1039.3 mm, vias 107 -> 143
- net -14V: track 0.00 -> 147.5 mm
- net N$37: track 0.00 -> 83.1 mm
- net VBAT: track 119.6 -> 78.8 mm, vias 2 -> 1
- net N$24: track 0.00 -> 31.8 mm
- net -12V: track 0.00 -> 24.4 mm
- net BSW_G: track 0.00 -> 19.8 mm
- net VFB_14VP: track 0.00 -> 18.2 mm
- net +12V: track 0.00 -> 16.3 mm
- net N$30: track 0.00 -> 15.8 mm
- net VFB_12VN: track 0.00 -> 14.4 mm
- net N$43: track 0.00 -> 12.2 mm
- net VFB_12VP: track 0.00 -> 11.9 mm
- net N$44: track 0.00 -> 9.91 mm, vias 0 -> 2
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Other:
- board size 155 x 100 mm -> 170 x 100 mm

Commit message: create PCB
Parts:
- removed C114, C116: 100nF, ds_passive:0402
- removed C115, C117: 4.7uF, ds_passive:0603
- removed IC20: MIC5504-3.3YM5-TR, ds_ic_vreg:SOT23-5
- removed R81, R82: 0R, ds_passive:0402
- removed TP100, TP101, TP102, TP103, TP104, TP105, TP106, TP17, TP18, TP19, TP20, TP21, TP22, TP23, TP24, TP25, TP26, TP27, TP28, TP29, TP30, TP31, TP32, TP33, TP34, TP35, TP36, TP37, TP38, TP39, TP40, TP46, TP47, TP48, TP49, TP50, TP51, TP53, TP54, TP55, TP56, TP57, TP80, TP81, TP82, TP83, TP84, TP85, TP89, TP90, TP91, TP92, TP93, TP94, TP95, TP96, TP97, TP98, TP99: PTR1B1,27, testpad:B1,27
- added 12VN, 12VP, 14VN, 14VP, BUF, CLR, DIO_CS, DIO_EN, DIO_GND, DIO_LS, DIO_RST, DIO_VREF, LDAC, REF/2, REFBY2, REFOUT, SPI1_CS0, SYNC, TP9, TPD0, TP_3V3, TP_BSW_G, TP_GND, TP_VFB_14VN, TP_VFB_14VP, TP_VREF_TPS, VCOMB, VFB12VN, VFB12VP, VOCMA, VREFR, VREF_DAC: TP, ds_passive:TP
- added C21: 100nF, ds_passive:0603
- added C22, C25: 100nF, ds_passive:0402
- added IC16: SN74LVC2G66, ds_ic_peripherals:SOP50P310X90-8N
- added IC17: 74LVC1G04, ds_ic_logic:SOT95P280X145-5N
- added J7: 2-5174225-5, Connector_D-Sub:2-5174225-5
- added JP4: POE, jumper:JP2Q
- added R25, R26, R27, R28, R29, R30, R31, R32, R33, R34, R35, R36, R37, R38, R39, R40, R41: 0R, ds_passive:0603
- C110, C70: device ds_passive:0805 -> ds_passive:0603
- C111, C151, C152, C153, C154, C155, C156, C157, C158, C159, C160, C161, C162, C163, C164, C165, C166, C167, C168, C169, C170, C51, C53, C55, C57, C59, C61, C63, C65, C67, C69, C71, R24, R42, R43, R44, R45, R46, R47, R48: device ds_passive:0603 -> ds_passive:0402
- ETH1: value (none) -> G16LX-188S7-1G-GO-Y; device ds_con:RJ45 -> ds_con:MAGJACK_POE
- IC38: value (none) -> SN74LVC2G66
- R17, R18: device ds_passive:0402 -> ds_passive:0603
- moved C74 168.3 mm to (0.30, 40.9), turned to 90 degrees
- moved C44 164.8 mm to (29.8, 14.9), turned to 270 degrees
- moved C54 163.2 mm to (19.8, 22.8), turned to 90 degrees
- moved R20 163.0 mm to (29.3, 23.5), turned to 180 degrees
- moved R17 162.3 mm to (54.0, 32.4), turned to 180 degrees
- moved R45 161.6 mm to (31.6, 22.4), turned to 180 degrees
- moved R18 159.9 mm to (54.0, 34.0), turned to 180 degrees
- moved IC10 159.0 mm to (36.8, 18.1)
- moved R42 158.7 mm to (17.3, 22.6), turned to 270 degrees
- moved R46 157.9 mm to (31.6, 21.3)
- moved R21 157.3 mm to (29.2, 20.2), turned to 180 degrees
- moved C55 156.4 mm to (21.3, 22.8), turned to 90 degrees
- moved C56 156.2 mm to (12.8, 26.7), turned to 180 degrees
- moved C73 152.9 mm to (0.32, 47.5), turned to 270 degrees
- moved R47 151.9 mm to (31.5, 15.5)
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- renumbered J3 to USB3, J4 to HDMI2, J5 to HDMI1, J6 to USBC, SV2 to GPIO, U$1 to SD1, U$2 to PCIE
Connections:
- removed net !CS1_ADC: IC10.14, R15.1, TP40.TP
- removed net !CS_ADA_A: IC7.11
- removed net !CS_ADA_B: IC9.11
- removed net DIO_CS1: IC36.9, TP104.TP
- removed net DIO_CS2: IC37.9
- removed net EEPROM_WP: JP2.4
- removed net MISO: IC36.12, IC37.12, IC7.8, IC9.8
- removed net MOSI: IC10.15, IC22.15, IC36.11, IC37.11, IC7.9, IC9.9
- removed net SCK: IC10.16, IC22.16, IC36.10, IC37.10, IC7.10, IC9.10
- removed net SDO_A_1: IC10.23, R18.2
- removed net SDO_A_2: IC10.22, R81.2
- removed net SDO_A_3: IC10.21, R82.2
- removed net SDO_B_1: IC10.19, R18.1
- removed net SDO_B_2: IC10.18, R81.1
- removed net SDO_B_3: IC10.17, R82.1
- removed net USBOTG: JP2.10
- removed net V+: C52.1, C53.1, C56.1, C57.1, C60.1, C61.1, C66.1, C67.1, IC6.14, IC7.26, IC8.14, IC9.26
- removed net V-: C54.1, C55.1, C58.1, C59.1, C62.1, C63.1, C68.1, C69.1, IC6.3, IC7.27, IC7.29, IC8.3, IC9.27, IC9.29
- new net !MISO_SEL: IC16.3, IC17.4
- new net MISO_SEL: IC16.7, IC17.2
- new net SPI0_CS0: DIO_CS.TP, IC36.9, R29.1
- new net SPI0_CS1: IC37.9, R30.1
- new net SPI0_MISO: IC36.12, IC37.12, R27.1
- new net SPI0_MOSI: IC22.15, IC36.11, IC37.11, R28.1
- new net SPI0_SCK: IC22.16, IC36.10, IC37.10, R26.1
- new net SPI1_CS0: IC10.14, R15.1, R32.1, SPI1_CS0.TP
- new net SPI1_CS1: IC7.11, R33.1
- new net SPI1_CS2: IC9.11, R34.1
- new net SPI1_MISO: IC16.2, IC16.6, IC7.8, IC9.8, R18.1
- new net SPI1_MOSI: IC10.15, IC7.9, IC9.9, R17.1
- new net SPI1_SCK: IC10.16, IC7.10, IC9.10, R25.1
- new net TR0_TAP: ETH1.VC1, JP4.3
- new net TR1_TAP: ETH1.VC2, JP4.1
- new net TR2_TAP: ETH1.VC3, JP4.2
- new net TR3_TAP: ETH1.VC4, JP4.4
- net !ADC_RST: now also R38.1; no longer TP39.TP
- net +12V: now also 12VP.TP, C52.1, C53.1, C56.1, C57.1, C60.1, C61.1, C66.1, C67.1, IC6.14, IC7.26, IC8.14, IC9.26; no longer TP53.TP
- net +14V: now also 14VP.TP; no longer TP46.TP
- net +3V3: now also C21.1, C22.1, C25.1, ETH1.18, ETH1.20, IC16.8, IC17.5, R86.5, TP_3V3.TP; no longer C116.1, C117.1, ETH1.P11, ETH1.P14, IC20.5
- net +3V3_EXT: now also J7.52, J7.67
- net +5V: now also J7.18, J7.33; no longer C114.1, C115.1, IC20.1, IC20.3
- net -12V: now also 12VN.TP, C54.1, C55.1, C58.1, C59.1, C62.1, C63.1, C68.1, C69.1, IC6.3, IC7.27, IC7.29, IC8.3, IC9.27, IC9.29; no longer TP54.TP
- net -14V: now also 14VN.TP; no longer TP47.TP
- net ADC_AIN_N: no longer TP22.TP
- net ADC_AIN_P: no longer TP21.TP
- net ADC_BIN_N: no longer TP24.TP
- net ADC_BIN_P: no longer TP23.TP
- net ADC_IN0: no longer TP17.TP
- net ADC_IN1: no longer TP18.TP
- net ADC_IN2: no longer TP19.TP
- net ADC_IN3: no longer TP20.TP
- net ADC_RDY: now also R36.1; no longer TP28.TP
- net AO_0: now also J7.29
- net AO_1: now also J7.63
- net AO_2: now also J7.30
- net AO_3: now also J7.64
- net AO_4: now also J7.31
- net AO_5: now also J7.65
- net AO_6: now also J7.32
- net AO_7: now also J7.66
- net BSW_G: now also TP_BSW_G.TP; no longer TP51.TP
- net BUF: now also BUF.TP; no longer TP57.TP
- net DAC_!CLR: now also CLR.TP, R37.1, R86.4; no longer R86.1, TP93.TP
- net DAC_!LDAC: now also LDAC.TP, R35.1, R86.2; no longer R86.3, TP89.TP
- net DAC_!SYNC: now also R31.1, R86.3, SYNC.TP; no longer R86.2, TP91.TP
- net DAC_0: now also TPD0.TP; no longer TP90.TP
- net DAC_1: no longer TP92.TP
- net DAC_2: no longer TP94.TP
- net DAC_3: no longer TP96.TP
- net DAC_4: no longer TP97.TP
- net DAC_5: no longer TP98.TP
- net DAC_6: no longer TP99.TP
- net DAC_7: no longer TP100.TP
- net DIO_0: now also J7.2, R120.5; no longer R119.8
- net DIO_1: now also J7.3, R120.6; no longer R119.7
- net DIO_10: now also J7.12, R122.7; no longer R121.6
- net DIO_11: now also J7.13, R122.8; no longer R121.5
- net DIO_12: now also J7.14, R121.5; no longer R122.8
- net DIO_13: now also J7.15, R121.6; no longer R122.7
- net DIO_14: now also J7.16, R121.7; no longer R122.6
- net DIO_15: now also J7.17, R121.8; no longer R122.5
- net DIO_16: now also J7.36, R124.5; no longer R123.8
- net DIO_17: now also J7.37, R124.6; no longer R123.7
- net DIO_18: now also J7.38, R124.7; no longer R123.6
- net DIO_19: now also J7.39, R124.8; no longer R123.5
- net DIO_2: now also J7.4, R120.7; no longer R119.6
- net DIO_20: now also J7.40, R123.5; no longer R124.8
- net DIO_21: now also J7.41, R123.6; no longer R124.7
- net DIO_22: now also J7.42, R123.7; no longer R124.6
- net DIO_23: now also J7.43, R123.8; no longer R124.5
- net DIO_24: now also J7.44, R126.5; no longer R125.8
- net DIO_25: now also J7.45, R126.6; no longer R125.7
- net DIO_26: now also J7.46, R126.7; no longer R125.6
- net DIO_27: now also J7.47, R126.8; no longer R125.5
- net DIO_28: now also J7.48, R125.5; no longer R126.8
- net DIO_29: now also J7.49, R125.6; no longer R126.7
- net DIO_3: now also J7.5, R120.8; no longer R119.5
- net DIO_30: now also J7.50, R125.7; no longer R126.6
- net DIO_31: now also J7.51, R125.8; no longer R126.5
- net DIO_4: now also J7.6, R119.5; no longer R120.8
- net DIO_5: now also J7.7, R119.6; no longer R120.7
- net DIO_6: now also J7.8, R119.7; no longer R120.6
- net DIO_7: now also J7.9, R119.8; no longer R120.5
- net DIO_8: now also J7.10, R122.5; no longer R121.8
- net DIO_9: now also J7.11, R122.6; no longer R121.7
- net DIO_EN: now also DIO_EN.TP, R41.1; no longer TP103.TP
- net DIO_LEVEL_SELECT: now also DIO_LS.TP, R40.1; no longer TP101.TP, TP106.TP
- net DIO_RESET: now also DIO_RST.TP, R39.1; no longer TP105.TP
- net EEPROM_NWP: now also JP2.4
- net GND: now also C21.2, C22.2, C25.2, DIO_GND.TP, IC16.4, IC17.3, J7.1, J7.23, J7.28, J7.34, J7.35, J7.57, J7.62, J7.68, J7.MH1, J7.MH2, TP_GND.TP; no longer C114.2, C115.2, C116.2, C117.2, IC20.2
- net GPIO10: now also R28.2
- net GPIO11: now also R26.2
- net GPIO13: now also R40.2
- net GPIO16: now also R34.2
- net GPIO17: now also R33.2
- net GPIO18: now also R32.2
- net GPIO19: now also R18.2
- net GPIO20: now also R17.2
- net GPIO21: now also R25.2
- net GPIO23: now also R31.2
- net GPIO24: now also R36.2
- net GPIO25: now also R38.2
- net GPIO27: now also R35.2
- net GPIO4: now also R37.2
- net GPIO5: now also R41.2
- net GPIO6: now also R39.2
- net GPIO7: now also R30.2
- net GPIO8: now also R29.2
- net GPIO9: now also R27.2
- net IN0+: now also J7.19
- net IN1-: now also J7.53
- net IN10+: now also J7.25
- net IN11-: now also J7.59
- net IN12+: now also J7.26
- net IN13-: now also J7.60
- net IN14+: now also J7.27
- net IN15-: now also J7.61
- net IN2+: now also J7.20
- net IN3-: now also J7.54
- net IN4+: now also J7.21
- net IN5-: now also J7.55
- net IN6+: now also J7.22
- net IN7-: now also J7.56
- net IN8+: now also J7.24
- net IN9-: now also J7.58
- net MUX_A_OUTA: no longer TP33.TP
- net MUX_A_OUTB: no longer TP34.TP
- net MUX_B_OUTA: no longer TP35.TP
- net MUX_B_OUTB: no longer TP36.TP
- net N$108: now also IC35.8; no longer IC35.5
- net N$109: now also IC35.7; no longer IC35.6
- net N$110: now also IC35.6; no longer IC35.7
- net N$111: now also IC35.5; no longer IC35.8
- net N$112: now also IC35.4; no longer IC35.9
- net N$113: now also IC35.3; no longer IC35.10
- net N$114: now also IC35.9; no longer IC35.4
- net N$115: now also IC35.10; no longer IC35.3
- net N$29: now also IC33.9; no longer IC33.4
- net N$4: now also ETH1.CT1, ETH1.CT2, ETH1.CT3, ETH1.CT4; no longer ETH1.P1, ETH1.P10
- net N$5: now also ETH1.17; no longer ETH1.P13
- net N$61: now also IC32.10; no longer IC32.3
- net N$62: now also IC32.9; no longer IC32.4
- net N$63: now also IC32.8; no longer IC32.5
- net N$64: now also IC32.7; no longer IC32.6
- net N$65: now also IC32.6; no longer IC32.7
- net N$66: now also IC32.5; no longer IC32.8
- net N$67: now also IC32.4; no longer IC32.9
- net N$68: now also IC32.3; no longer IC32.10
- net N$77: now also IC33.10; no longer IC33.3
- net N$78: now also IC33.8; no longer IC33.5
- net N$79: now also IC33.7; no longer IC33.6
- net N$8: now also ETH1.19; no longer ETH1.P12
- net N$80: now also IC33.6; no longer IC33.7
- net N$81: now also IC33.5; no longer IC33.8
- net N$82: now also IC33.4; no longer IC33.9
- net N$83: now also IC33.3; no longer IC33.10
- net N$92: now also IC34.10; no longer IC34.3
- net N$93: now also IC34.9; no longer IC34.4
- net N$94: now also IC34.8; no longer IC34.5
- net N$95: now also IC34.7; no longer IC34.6
- net N$96: now also IC34.6; no longer IC34.7
- net N$97: now also IC34.5; no longer IC34.8
- net N$98: now also IC34.4; no longer IC34.9
- net N$99: now also IC34.3; no longer IC34.10
- net PGA_A_IN+: no longer TP29.TP
- net PGA_A_IN-: no longer TP30.TP
- net PGA_B_IN+: no longer TP31.TP
- net PGA_B_IN-: no longer TP32.TP
- net REFBY2: now also REFBY2.TP; no longer TP85.TP
- net REFM_A: no longer TP81.TP
- net REFM_B: no longer TP83.TP
- net REFOUT: now also REFOUT.TP; no longer TP84.TP
- net REFP_A: no longer TP80.TP
- net REFP_B: no longer TP82.TP
- net SDO_A_0: now also IC16.1; no longer R17.2
- net SDO_B_0: now also IC16.5; no longer R17.1
- net TRD0_N: now also ETH1.TD1-; no longer ETH1.P3
- net TRD0_P: now also ETH1.TD1+; no longer ETH1.P2
- net TRD1_N: now also ETH1.TD2-; no longer ETH1.P5
- net TRD1_P: now also ETH1.TD2+; no longer ETH1.P4
- net TRD2_N: now also D1.4, D1.7, ETH1.TD3-; no longer D1.2, D1.9, ETH1.P7
- net TRD2_P: now also D1.5, D1.6, ETH1.TD3+; no longer D1.1, D1.10, ETH1.P6
- net TRD3_N: now also D1.2, D1.9, ETH1.TD4-; no longer D1.4, D1.7, ETH1.P9
- net TRD3_P: now also D1.1, D1.10, ETH1.TD4+; no longer D1.5, D1.6, ETH1.P8
- net USBOTG_ID: now also JP2.10
- net VFB_12VN: now also VFB12VN.TP; no longer TP56.TP
- net VFB_12VP: now also VFB12VP.TP; no longer TP55.TP
- net VFB_14VN: now also TP_VFB_14VN.TP; no longer TP49.TP
- net VFB_14VP: now also TP_VFB_14VP.TP; no longer TP48.TP
- net VOCM_A: now also VOCMA.TP; no longer TP37.TP
- net VOCM_B: now also VCOMB.TP; no longer TP38.TP
- net VREF_ADC: now also TP9.TP; no longer TP25.TP
- net VREF_ADC/2: now also REF/2.TP; no longer TP27.TP
- net VREF_ADC_RAW: now also VREFR.TP; no longer TP26.TP
- net VREF_DAC_OUT: now also VREF_DAC.TP; no longer TP95.TP
- net VREF_TPS: now also TP_VREF_TPS.TP; no longer TP50.TP
- net V_OUT_REF: now also DIO_VREF.TP; no longer TP102.TP
Routing:
- net GND: track 1039.3 -> 1943.7 mm, vias 143 -> 284
- net +3V3: track 249.3 -> 747.9 mm, vias 5 -> 31
- net +5V: track 596.2 -> 766.3 mm, vias 25 -> 32
- net SPI1_CS1: track 0.00 -> 125.9 mm, vias 0 -> 4
- net +12V: track 16.3 -> 135.8 mm, vias 0 -> 7
- net DIO_31: track 0.00 -> 114.6 mm, vias 0 -> 1
- net -12V: track 24.4 -> 136.5 mm, vias 0 -> 9
- net VREF_ADC: track 0.00 -> 111.7 mm, vias 0 -> 4
- net DIO_30: track 0.00 -> 111.1 mm, vias 0 -> 1
- net DIO_29: track 0.00 -> 110.1 mm, vias 0 -> 1
- net SPI1_MISO: track 0.00 -> 107.2 mm, vias 0 -> 8
- net DIO_28: track 0.00 -> 104.4 mm, vias 0 -> 1
- net DIO_27: track 0.00 -> 101.1 mm, vias 0 -> 1
- net SPI1_MOSI: track 0.00 -> 99.4 mm, vias 0 -> 7
- net SPI1_SCK: track 0.00 -> 98.2 mm, vias 0 -> 7
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Other:
- board size 170 x 100 mm -> 180 x 100 mm
- board text added: "BT_DIS WL_DIS"
- board text added: "DataForge-PI"
- board text added: "ID_SD ID_SC"
- board text added: "PWRBU PMICEN OTG SYNC EEWP NRBT"

Commit message: create PCB
Parts:
- moved R39 112.1 mm to (-20.9, 77.8)
- moved R40 112.1 mm to (-20.9, 76.0)
- moved R41 112.1 mm to (-20.9, 74.2)
- moved R36 86.6 mm to (45.9, 33.3), turned to 90 degrees
- moved R38 85.7 mm to (45.9, 29.9), turned to 90 degrees
Routing:
- net GPIO5: track 75.9 -> 175.5 mm, vias 1 -> 2
- net GPIO13: track 76.7 -> 167.9 mm, vias 1 -> 2
- net GPIO6: track 75.7 -> 165.9 mm, vias 1 -> 2
- net GPIO23: track 71.0 -> 131.0 mm, vias 1 -> 2
- net GPIO27: track 62.0 -> 106.8 mm, vias 1 -> 2
- net GPIO4: track 64.5 -> 101.7 mm, vias 1 -> 2
- net GPIO25: track 75.7 -> 108.2 mm, vias 1 -> 2
- net GPIO24: track 73.6 -> 104.8 mm
- net DIO_LEVEL_SELECT: track 7.51 -> 37.9 mm, vias 0 -> 3
- net DIO_RESET: track 32.4 -> 49.2 mm
- net ADC_RDY: track 0.00 -> 15.7 mm, vias 0 -> 2
- net !ADC_RST: track 3.98 -> 13.9 mm
- net DIO_EN: track 50.5 -> 56.0 mm
- net SPI0_CS0: track 91.7 -> 92.9 mm

Commit message: 3D render
Parts:
- removed C118, C119: 100uF, rcl:153CLV-0605
- removed IC21: LD117ADT33TR, v-reg:DPACK
- removed R77, R78: 20K, pot:3223G
- removed R79, R80: 250K, pot:3223G
- removed S1: (no value), adafruit:B3F-31XX
- removed SV1: (no value), con-lstb:MA04-1
- removed X1: ASEK-32.768KHz-LRT, crystal-geyer_V1_0:3.2X2.5_KXO-V96
- added C26, C27: 100uF 16V, ds_passive:100UF-16V
- added CON1: (no value), ds_con:1X4
- added IC18: (no value), ds_ic_vreg:SOT230
- added R53, R54, R55, R56: (no value), ds_passive:TC33X
- added SW1: 1825027-8, ds_passive:SW2_1825027-C_TEC
- added X2: CRYSTAL, ds_passive:OSCCC500X320X130
- C8: value 100uF -> 100uF 16V; device rcl:153CLV-0505 -> ds_passive:100UF-16V
- GPIO: device con-lstb:MA20-2 -> ds_con:2X20
- IC12: value REF3025 -> MCP1525T-I/TT; device maxim:SOT23 -> ds_ic_vreg:SOT23
- IC6, IC8: device ds_ic_peripherals:TSSOP16 -> ds_ic_peripherals:TSSOP2
- JP1, JP3, JP4: device jumper:JP2Q -> ds_con:2X2
- JP2: device jumper:JP7Q -> ds_con:2X7
- L1: value (none) -> L; device rcl:L5038P -> ds_passive:SRR5228A
- L3, L4: value B8246284-4.7uH -> SRR5228A-4R7Y; device inductor-coilcraft:MSS7341 -> ds_passive:SRR5228A
- R49: value 20K -> (none); device pot:3223G -> ds_passive:TC33X
- SD1: value MICROSD -> (none); device adafruit:MICROSD -> ds_con:MICROSD
- moved SD1 11.9 mm to (49.5, 6.20)
- moved C8 4.96 mm to (69.5, 25.3), turned to 0 degrees
- moved L4 0.60 mm to (23.9, 60.4)
- moved L1 0.51 mm to (123.5, 32.9), turned to 90 degrees
- moved R49 0.26 mm to (-2.75, 42.6), turned to 180 degrees
- moved IC12 0.11 mm to (-1.75, 55.4)
- moved JP2 0.07 mm to (118.9, 89.4), turned to 180 degrees
- turned JP4 to 270 degrees
- turned JP1 to 180 degrees
- turned JP3 to 180 degrees
- turned GPIO to 0 degrees
Connections:
- net +3V3_EXT: now also C27.1, IC18.2, IC18.4; no longer C119.+, IC21.4
- net +5V: now also C26.1, CON1.4, IC18.3; no longer C118.+, IC21.3, SV1.4
- net GND: now also C26.2, C27.2, C8.2, CON1.2, IC18.1, SD1.MT3, SD1.MT4, SD1.VSS, SW1.1, SW1.3, SW1.4, X2.2; no longer C118.-, C119.-, C8.-, IC21.1, S1.2, SD1.6, SV1.2, X1.2
- net M2_3V3: now also X2.3, X2.4; no longer X1.1, X1.4
- net N$11: now also X2.1; no longer X1.3
- net N$38: now also R55.2, R55.3; no longer R77.2, R77.3
- net N$42: now also R56.2, R56.3; no longer R78.2, R78.3
- net N$43: now also R53.2, R53.3; no longer R79.2, R79.3
- net N$44: now also R54.2, R54.3; no longer R80.2, R80.3
- net PWM: now also CON1.3; no longer SV1.3
- net PWR_BUT: now also SW1.2; no longer S1.1
- net SD_CLK: now also SD1.CLK; no longer SD1.5
- net SD_CMD: now also SD1.CMD; no longer SD1.3
- net SD_DAT0: now also SD1.DAT0; no longer SD1.7
- net SD_DAT1: now also SD1.DAT1; no longer SD1.8
- net SD_DAT2: now also SD1.DAT2; no longer SD1.1
- net SD_DAT3: now also SD1.DAT3/CD; no longer SD1.2
- net SD_PWR: now also SD1.VDD; no longer SD1.4
- net TACHO: now also CON1.1; no longer SV1.1
- net VBUS: now also C8.1; no longer C8.+
- net VFB_12VN: now also R56.1; no longer R78.1
- net VFB_12VP: now also R55.1; no longer R77.1
- net VFB_14VN: now also R54.1; no longer R80.1
- net VFB_14VP: now also R53.1; no longer R79.1
Routing:
- net GND: track 1943.7 -> 2082.3 mm, vias 284 -> 291
- net PWM: track 42.1 -> 28.0 mm
- net N$30: track 15.8 -> 29.5 mm
- net N$37: track 83.1 -> 92.2 mm
- net TACHO: track 37.6 -> 28.8 mm
- net VBUS: track 55.5 -> 64.1 mm
- net SD_DAT1: track 134.5 -> 140.9 mm
- net +5V: track 766.3 -> 772.7 mm
- net SD_DAT0: track 132.2 -> 138.4 mm
- net SD_DAT3: track 126.4 -> 132.2 mm
- net +3V3_EXT: track 81.9 -> 87.5 mm
- net VFB_14VN: track 21.6 -> 27.1 mm, vias 2 -> 3
- net SD_CLK: track 126.7 -> 132.0 mm
- net SD_DAT2: track 131.3 -> 136.6 mm
- net SD_CMD: track 114.2 -> 119.5 mm
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Other:
- outline, holes or cut-outs redrawn
