File: src/HardwareDesign/HW_RPI_DAQ.sch (EAGLE design)
At the start: 64 parts, among them IC2 AP22653W6, IC3 74LVC1G07, IC4 RT9742NGV, J1 10164227-1001A1RLF, J2 10164227-1001A1RLF, J3 692141030100, J4 685119136923, J5 685119136923, X1 ASEK-32.768KHz-LRT

Commit message: add DAQ to design
Parts:
- removed USB1: (no value), ds_con:USB_C
- added C100, C101: 10pF, ds_passive:C0402
- added C102, C104: 10uF, ds_passive:C1206
- added C103, C106, C107: 10nF, ds_passive:C0402
- added C105, C99: 220nF, ds_passive:C0402
- added C108, C109, C93, C94, C95, C96, C97, C98: 22uF, ds_passive:C1206
- added C110, C47, C70, C90: 10uF, ds_passive:C0805
- added C111, C123, C152, C154, C156, C158, C160, C162, C164, C166, C168, C170, C171, C51, C53, C55, C57, C59, C61, C63, C65, C67, C69, C71, C73: 100nF, ds_passive:C0603
- added C114, C116, C120, C121, C125, C126, C128, C129, C131, C132, C134, C135, C137, C138, C140, C141, C143, C144, C146, C147, C149, C150, C45, C46, C49, C75, C76: 100nF, ds_passive:C0402
- added C115, C117: 4.7uF, ds_passive:C0603
- added C118, C119: 100uF, rcl:CPOL-EU153CLV-0605
- added C122, C124, C151, C153, C155, C157, C159, C161, C163, C165, C167, C169, C50, C52, C54, C56, C58, C60, C62, C64, C66, C68, C72: 1uF, ds_passive:C0603
- added C127, C130, C133, C136, C139, C142, C145, C148: 20nF, ds_passive:C0402
- added C23, C24, C42, C43: 270pF, ds_passive:C0402
- added C41, C44: 680pF, ds_passive:C0402
- added C48, C74: (no value), ds_passive:C0805
- added C85: 4.7uF, ds_passive:C0805
- added C86: 100nF, ds_passive:C0805
- added C91: 10nF, ds_passive:C0805
- added C92: 4.7nF, ds_passive:C0805
- added D3, D4: SS12, Diodes:SS12
- added IC10: ADS9234RIRHBR, ds_ic_peripherals:ADS9234RIRHBR
- added IC11, IC13, IC23, IC24, IC25, IC26, IC27, IC28, IC29, IC30, IC31: MCP6001RT, ds_ic_opa:MCP6001RT
- added IC12: REF3025, maxim:MAX6520
- added IC14: TPS65131, ds_ic_vreg:TPS65131TRGERQ1
- added IC15: TPS7A39, ds_ic_vreg:TPS7A3901DSCR
- added IC20: MIC5504-3.3YM5-TR, ds_ic_vreg:MIC5504-3.3YM5-TR
- added IC21: LD117ADT33TR, v-reg:LD117ADT33TR
- added IC22: DAC8568, ds_ic_peripherals:DAC8568
- added IC32, IC33, IC34, IC35: LSF0108, ds_ic_peripherals:LSF0108-Q1
- added IC36: MCP23S18, ds_ic_peripherals:MCP23S18
- added IC37: (no value), ds_ic_peripherals:MCP23S18
- added IC38: (no value), ds_ic_peripherals:SN74LVC2G66
- added IC39: 74LVC1G04, ds_ic_logic:74LVC1G04
- added IC6, IC8: DG409, ds_ic_peripherals:DG409
- added IC7, IC9: ADA4254ACPZ, ds_ic_opa:ADA4254ACPZ
- added J6: 629722000214, Wurth_Connectors_WR-USB:629722000214
- added L3, L4: B8246284-4.7uH, inductor-coilcraft:MSS7341
- added R100, R103, R104, R107, R108, R111, R112, R115, R116, R73, R76, R87, R88, R91, R92, R95, R96, R99: 10K 0.1%, ds_passive:R0402
- added R101, R105, R109, R113, R117, R89, R93, R97: 43K 0.1%, ds_passive:R0402
- added R102, R106, R110, R114, R118, R90, R94, R98: 68R 1%, ds_passive:R0402
- added R119, R120, R121, R122, R123, R124, R125, R126: YC164-JR-0733RL, Resistor Array:YC164-JR-0733RL
- added R127, R128, R129, R130: 200K, ds_passive:R0402
- added R14: 100R, ds_passive:R1206
- added R15, R17, R18, R81, R82: 0R, ds_passive:R0402
- added R16: 10K, ds_passive:R0402
- added R19: 950K 0.1%, ds_passive:R0402
- added R20, R21, R22, R23: 200R, ds_passive:R0402
- added R24, R42, R43, R44, R45, R46, R47, R48, R51, R52: 0R, ds_passive:R0603
- added R49, R77, R78: 20K, pot:TRIM_EU-3223G
- added R50: 100R, ds_passive:R0402
- added R57: 102K 0.1%, ds_passive:R0402
- added R58: 1.2M 0.1%, ds_passive:R0402
- added R59: 137K 0.1%, ds_passive:R0402
- added R60: 75K 0.1%, ds_passive:R0402
- added R74: 90K 0.1%, ds_passive:R0402
- added R79, R80: 250K, pot:TRIM_EU-3223G
- added R86: CRA034RF100RP05Z, Resistor Array:YC164-JR-0733RL
- added T2: IRLML5203, transistor-power:IRLML5203
- added TP100, TP101, TP102, TP103, TP104, TP105, TP106, TP17, TP18, TP19, TP20, TP21, TP22, TP23, TP24, TP25, TP26, TP27, TP28, TP29, TP30, TP31, TP32, TP33, TP34, TP35, TP36, TP37, TP38, TP39, TP40, TP46, TP47, TP48, TP49, TP50, TP51, TP53, TP54, TP55, TP56, TP57, TP80, TP81, TP82, TP83, TP84, TP85, TP89, TP90, TP91, TP92, TP93, TP94, TP95, TP96, TP97, TP98, TP99: PTR1B1,27, testpad:PTR1B1,27
Connections:
- removed net TACH0: J2.16
- new net !ADC_RST: IC10.!PD!/!RST, R16.2, TP39.TP
- new net !CS1_ADC: IC10.!CS, R15.1, TP40.TP
- new net !CS_ADA_A: IC7.!CS
- new net !CS_ADA_B: IC9.!CS
- new net !DIO_LEVEL_SELECT: IC38.2C, IC39.OUT
- new net +12V: C107.2, C108.1, IC15.OUTP, R60.1, TP53.TP
- new net +14V: C100.1, C104.1, C93.1, C94.1, C95.1, D3.C, IC14.VPOS, IC15.EN, IC15.INP, R19.1, TP46.TP
- new net +3V3_EXT: C119.+, C121.1, IC21.OUT
- new net -12V: C106.1, C109.1, IC15.OUTN, R76.2, TP54.TP
- new net -14V: C101.1, C102.1, C96.1, C97.1, C98.1, D4.A, IC14.VNEG, IC15.INN, R59.2, TP47.TP
- new net ADA_A_IO0: IC6.A0, IC7.GPIO0
- new net ADA_A_IO1: IC6.A1, IC7.GPIO1
- new net ADA_A_IO2: IC6.EN, IC7.GPIO2
- new net ADA_B_IO0: IC8.A0, IC9.GPIO0
- new net ADA_B_IO1: IC8.A1, IC9.GPIO1
- new net ADA_B_IO2: IC8.EN, IC9.GPIO2
- new net ADC_AIN_N: C24.2, C41.2, R21.1, R46.1, TP22.TP
- new net ADC_AIN_P: C23.1, C41.1, R20.1, R45.2, TP21.TP
- new net ADC_BIN_N: C43.2, C44.2, R23.1, R48.2, TP24.TP
- new net ADC_BIN_P: C42.1, C44.1, R22.1, R47.1, TP23.TP
- new net ADC_IN0: IC10.AINP_A, R45.1, TP17.TP
- new net ADC_IN1: IC10.AINM_A, R46.2, TP18.TP
- new net ADC_IN2: IC10.AINP_B, R48.1, TP19.TP
- new net ADC_IN3: IC10.AINM_B, R47.2, TP20.TP
- new net ADC_RDY: IC10.READY/STROBE, TP28.TP
- new net AO_0: C127.1, R89.2, R90.2
- new net AO_1: C130.1, R93.2, R94.2
- new net AO_2: C133.1, R97.2, R98.2
- new net AO_3: C136.1, R101.2, R102.2
- new net AO_4: C139.1, R105.2, R106.2
- new net AO_5: C142.1, R109.2, R110.2
- new net AO_6: C145.1, R113.2, R114.2
- new net AO_7: C148.1, R117.2, R118.2
- new net BSW_G: IC14.BSW, T2.G, TP51.TP
- new net BUF: C105.2, IC15.BUF, R74.1, TP57.TP
- new net DAC_!CLR: IC22.!CLR, R86.1, TP93.TP
- new net DAC_!LDAC: IC22.!LDAC, R86.3, TP89.TP
- new net DAC_!SYNC: IC22.!SYNC, R86.2, TP91.TP
- new net DAC_0: IC22.VOUT_A, IC24.+IN, TP90.TP
- new net DAC_1: IC22.VOUT_B, IC25.+IN, TP92.TP
- new net DAC_2: IC22.VOUT_C, IC26.+IN, TP94.TP
- new net DAC_3: IC22.VOUT_D, IC27.+IN, TP96.TP
- new net DAC_4: IC22.VOUT_E, IC28.+IN, TP97.TP
- new net DAC_5: IC22.VOUT_F, IC29.+IN, TP98.TP
- new net DAC_6: IC22.VOUT_G, IC30.+IN, TP99.TP
- new net DAC_7: IC22.VOUT_H, IC31.+IN, TP100.TP
- new net DIO_0: R119.8
- new net DIO_1: R119.7
- new net DIO_10: R121.6
- new net DIO_11: R121.5
- new net DIO_12: R122.8
- new net DIO_13: R122.7
- new net DIO_14: R122.6
- new net DIO_15: R122.5
- new net DIO_16: R123.8
- new net DIO_17: R123.7
- new net DIO_18: R123.6
- new net DIO_19: R123.5
- new net DIO_2: R119.6
- new net DIO_20: R124.8
- new net DIO_21: R124.7
- new net DIO_22: R124.6
- new net DIO_23: R124.5
- new net DIO_24: R125.8
- new net DIO_25: R125.7
- new net DIO_26: R125.6
- new net DIO_27: R125.5
- new net DIO_28: R126.8
- new net DIO_29: R126.7
- new net DIO_3: R119.5
- new net DIO_30: R126.6
- new net DIO_31: R126.5
- new net DIO_4: R120.8
- new net DIO_5: R120.7
- new net DIO_6: R120.6
- new net DIO_7: R120.5
- new net DIO_8: R121.8
- new net DIO_9: R121.7
- new net DIO_CS1: IC36.!CS, TP104.TP
- new net DIO_CS2: IC37.!CS
- new net DIO_EN: IC32.EN, IC33.EN, IC34.EN, IC35.EN, TP103.TP
- new net DIO_LEVEL_SELECT: IC38.1C, IC39.IN, TP101.TP, TP106.TP
- new net DIO_RESET: IC36.!RESET, IC37.!RESET, TP105.TP
- new net IN0+: IC6.IN_A_0
- new net IN1-: IC6.IN_B_0
- new net IN10+: IC8.IN_A_1
- new net IN11-: IC8.IN_B_1
- new net IN12+: IC8.IN_A_2
- new net IN13-: IC8.IN_B_2
- new net IN14+: IC8.IN_A_3
- new net IN15-: IC8.IN_B_3
- new net IN2+: IC6.IN_A_1
- new net IN3-: IC6.IN_B_1
- new net IN4+: IC6.IN_A_2
- new net IN5-: IC6.IN_B_2
- new net IN6+: IC6.IN_A_3
- new net IN7-: IC6.IN_B_3
- new net IN8+: IC8.IN_A_0
- new net IN9-: IC8.IN_B_0
- new net MISO: IC36.SO, IC37.SO, IC7.SDO, IC9.SDO
- new net MOSI: IC10.SDI, IC22.DIN, IC36.SI, IC37.SI, IC7.SDI, IC9.SDI
- new net MUX_A_OUTA: IC6.OUT_A, R43.2, TP33.TP
- new net MUX_A_OUTB: IC6.OUT_B, R44.1, TP34.TP
- new net MUX_B_OUTA: IC8.OUT_A, R24.2, TP35.TP
- new net MUX_B_OUTB: IC8.OUT_B, R42.1, TP36.TP
- new net N$100: IC34.B1, R123.1
- new net N$101: IC34.B2, R123.2
- new net N$102: IC34.B3, R123.3
- new net N$103: IC34.B4, R123.4
- new net N$104: IC34.B5, R124.1
- new net N$105: IC34.B6, R124.2
- new net N$106: IC34.B7, R124.3
- new net N$107: IC34.B8, R124.4
- new net N$108: IC35.A3, IC37.GPB2
- new net N$109: IC35.A4, IC37.GPB3
- new net N$110: IC35.A5, IC37.GPB4
- new net N$111: IC35.A6, IC37.GPB5
- new net N$112: IC35.A7, IC37.GPB6
- new net N$113: IC35.A8, IC37.GPB7
- new net N$114: IC35.A2, IC37.GPB1
- new net N$115: IC35.A1, IC37.GPB0
- new net N$116: IC35.B1, R125.1
- new net N$117: IC35.B2, R125.2
- new net N$118: IC35.B3, R125.3
- new net N$119: IC35.B4, R125.4
- new net N$12: IC7.OUT+, R20.2
- new net N$120: IC35.B5, R126.1
- new net N$121: IC35.B6, R126.2
- new net N$122: IC35.B7, R126.3
- new net N$123: IC35.B8, R126.4
- new net N$124: IC32.VREF_B, R127.1
- new net N$125: IC33.VREF_B, R128.1
- new net N$126: IC35.VREF_B, R129.1
- new net N$127: IC34.VREF_B, R130.1
- new net N$13: IC7.OUT-, R21.2
- new net N$14: C129.2, IC24.OUT, R90.1
- new net N$15: IC9.OUT+, R22.2
- new net N$16: IC9.OUT-, R23.2
- new net N$17: C129.1, IC24.-IN, R87.2, R88.2, R89.1
- new net N$18: IC10.CONVST, R15.2
- new net N$19: C72.2, C73.2, R49.A
- new net N$20: C74.1, R49.S, R50.1
- new net N$21: IC11.+IN, R50.2
- new net N$22: C132.1, IC25.-IN, R91.2, R92.2, R93.1
- new net N$23: C132.2, IC25.OUT, R94.1
- new net N$24: D3.A, IC14.INP, L3.2
- new net N$25: C135.1, IC26.-IN, R95.2, R96.2, R97.1
- new net N$26: C135.2, IC26.OUT, R98.1
- new net N$27: C138.1, IC27.-IN, R100.2, R101.1, R99.2
- new net N$28: C138.2, IC27.OUT, R102.1
- new net N$29: IC33.A2, IC36.GPB1
- new net N$30: C90.1, L3.1, T2.D
- new net N$31: C141.1, IC28.-IN, R103.2, R104.2, R105.1
- new net N$32: C86.1, IC14.ENN, IC14.ENP, IC14.PSN, IC14.PSP, IC14.VIN, R14.1
- new net N$33: C141.2, IC28.OUT, R106.1
- new net N$34: C144.1, IC29.-IN, R107.2, R108.2, R109.1
- new net N$35: C91.1, IC14.CP
- new net N$36: C92.1, IC14.CN
- new net N$37: D4.C, IC14.OUTN, L4.2
- new net N$38: R60.2, R77.E, R77.S
- new net N$39: C103.1, IC15.NR/SS
- new net N$40: C144.2, IC29.OUT, R110.1
- new net N$41: C147.1, IC30.-IN, R111.2, R112.2, R113.1
- new net N$42: R74.2, R78.E, R78.S
- new net N$43: R19.2, R79.E, R79.S
- new net N$44: R58.2, R80.E, R80.S
- new net N$58: C147.2, IC30.OUT, R114.1
- new net N$59: C150.1, IC31.-IN, R115.2, R116.2, R117.1
- new net N$60: C150.2, IC31.OUT, R118.1
- new net N$61: IC32.A1, IC36.GPA0
- new net N$62: IC32.A2, IC36.GPA1
- new net N$63: IC32.A3, IC36.GPA2
- new net N$64: IC32.A4, IC36.GPA3
- new net N$65: IC32.A5, IC36.GPA4
- new net N$66: IC32.A6, IC36.GPA5
- new net N$67: IC32.A7, IC36.GPA6
- new net N$68: IC32.A8, IC36.GPA7
- new net N$69: IC32.B1, R119.1
- new net N$70: IC32.B2, R119.2
- new net N$71: IC32.B3, R119.3
- new net N$72: IC32.B4, R119.4
- new net N$73: IC32.B5, R120.1
- new net N$74: IC32.B6, R120.2
- new net N$75: IC32.B7, R120.3
- new net N$76: IC32.B8, R120.4
- new net N$77: IC33.A1, IC36.GPB0
- new net N$78: IC33.A3, IC36.GPB2
- new net N$79: IC33.A4, IC36.GPB3
- new net N$80: IC33.A5, IC36.GPB4
- new net N$81: IC33.A6, IC36.GPB5
- new net N$82: IC33.A7, IC36.GPB6
- new net N$83: IC33.A8, IC36.GPB7
- new net N$84: IC33.B1, R121.1
- new net N$85: IC33.B2, R121.2
- new net N$86: IC33.B3, R121.3
- new net N$87: IC33.B4, R121.4
- new net N$88: IC33.B5, R122.1
- new net N$89: IC33.B6, R122.2
- new net N$90: IC33.B7, R122.3
- new net N$91: IC33.B8, R122.4
- new net N$92: IC34.A1, IC37.GPA0
- new net N$93: IC34.A2, IC37.GPA1
- new net N$94: IC34.A3, IC37.GPA2
- new net N$95: IC34.A4, IC37.GPA3
- new net N$96: IC34.A5, IC37.GPA4
- new net N$97: IC34.A6, IC37.GPA5
- new net N$98: IC34.A7, IC37.GPA6
- new net N$99: IC34.A8, IC37.GPA7
- new net PGA_A_IN+: IC7.IN1+, R43.1, TP29.TP
- new net PGA_A_IN-: IC7.IN1-, IC7.IN2+, R44.2, TP30.TP
- new net PGA_B_IN+: IC9.IN1+, R24.1, TP31.TP
- new net PGA_B_IN-: IC9.IN1-, IC9.IN2+, R42.2, TP32.TP
- new net REFBY2: C71.1, IC10.REFBY2, TP85.TP
- new net REFM_A: C70.2, IC10.REFM_A, TP81.TP
- new net REFM_B: C110.2, IC10.REFM_B, TP83.TP
- new net REFOUT: C111.1, IC10.REFOUT, TP84.TP
- new net REFP_A: C70.1, IC10.REFP_A, TP80.TP
- new net REFP_B: C110.1, IC10.REFP_B, TP82.TP
- new net SCK: IC10.SCLK, IC22.SCLK, IC36.SCK, IC37.SCK, IC7.SCK, IC9.SCK
- new net SDO_A_0: IC10.SDO-0/0A, R17.2
- new net SDO_A_1: IC10.SDO-1/1A, R18.2
- new net SDO_A_2: IC10.SDO-2/2A, R81.2
- new net SDO_A_3: IC10.SDO-3/3A, R82.2
- new net SDO_B_0: IC10.SDO-4/0B, R17.1
- new net SDO_B_1: IC10.SDO-5/1B, R18.1
- new net SDO_B_2: IC10.SDO-6/2B, R81.1
- new net SDO_B_3: IC10.SDO-7/3B, R82.1
- new net V+: C52.1, C53.1, C56.1, C57.1, C60.1, C61.1, C66.1, C67.1, IC6.V+, IC7.VDDH, IC8.V+, IC9.VDDH
- new net V-: C54.1, C55.1, C58.1, C59.1, C62.1, C63.1, C68.1, C69.1, IC6.V-, IC7.PAD, IC7.VSSH, IC8.V-, IC9.PAD, IC9.VSSH
- new net VFB_12VN: C106.2, IC15.FBN, R76.1, R78.A, TP56.TP
- new net VFB_12VP: C107.1, IC15.FBP, R73.1, R77.A, TP55.TP
- new net VFB_14VN: C101.2, IC14.FBN, R59.1, R80.A, TP49.TP
- new net VFB_14VP: C100.2, IC14.FBP, R57.1, R79.A, TP48.TP
- new net VOCM_A: IC7.VOCM, R51.2, TP37.TP
- new net VOCM_B: IC9.VOCM, R52.1, TP38.TP
- new net VREF_ADC: C46.1, C72.1, C73.1, IC13.-IN, IC13.OUT, IC7.AVDD, IC9.AVDD, R49.E, TP25.TP
- new net VREF_ADC/2: C75.1, IC11.-IN, IC11.OUT, R51.1, R52.2, TP27.TP
- new net VREF_ADC_RAW: C48.1, IC12.OUT, IC13.+IN, TP26.TP
- new net VREF_DAC: C125.1, IC23.-IN, IC23.OUT, R100.1, R104.1, R108.1, R112.1, R116.1, R88.1, R92.1, R96.1
- new net VREF_DAC_OUT: C124.1, IC22.VREF_IO, IC23.+IN, TP95.TP
- new net VREF_TPS: C99.2, IC14.VREF, R58.1, TP50.TP
- new net V_OUT_REF: C153.1, C154.1, C157.1, C158.1, C161.1, C162.1, C165.1, C166.1, IC38.1B, IC38.2B, R127.2, R128.2, R129.2, R130.2, TP102.TP
- net +3V3: now also C116.1, C117.1, C122.1, C123.1, C126.1, C128.1, C131.1, C134.1, C137.1, C140.1, C143.1, C146.1, C149.1, C151.1, C152.1, C155.1, C156.1, C159.1, C160.1, C163.1, C164.1, C167.1, C168.1, C169.1, C170.1, C171.1, C45.1, C47.1, C49.1, C50.1, C51.1, C64.1, C65.1, C76.1, IC10.AVDD, IC10.DVDD, IC11.V+, IC12.IN, IC13.V+, IC20.VOUT, IC22.AVDD, IC23.V+, IC24.V+, IC25.V+, IC26.V+, IC27.V+, IC28.V+, IC29.V+, IC30.V+, IC31.V+, IC32.VREF_A, IC33.VREF_A, IC34.VREF_A, IC35.VREF_A, IC36.VDD, IC37.VDD, IC38.1A, IC38.VCC, IC39.V+, IC7.DVDD, IC9.DVDD, R16.1, R86.6, R86.7, R86.8
- net +5V: now also C114.1, C115.1, C118.+, C120.1, C85.1, IC14.INN, IC20.EN, IC20.VIN, IC21.IN, IC38.2A, J6.VBUS, J6.VBUS1, J6.VBUS2, J6.VBUS3, R14.2, T2.S; no longer USB1.VBUS
- net CC1: now also J6.CC1; no longer USB1.CC1
- net CC2: now also J6.CC2; no longer USB1.CC2
- net GND: now also C102.2, C103.2, C104.2, C105.1, C108.2, C109.2, C111.2, C114.2, C115.2, C116.2, C117.2, C118.-, C119.-, C120.2, C121.2, C122.2, C123.2, C124.2, C125.2, C126.2, C127.2, C128.2, C130.2, C131.2, C133.2, C134.2, C136.2, C137.2, C139.2, C140.2, C142.2, C143.2, C145.2, C146.2, C148.2, C149.2, C151.2, C152.2, C153.2, C154.2, C155.2, C156.2, C157.2, C158.2, C159.2, C160.2, C161.2, C162.2, C163.2, C164.2, C165.2, C166.2, C167.2, C168.2, C169.2, C170.2, C171.2, C23.2, C24.1, C42.2, C43.1, C45.2, C46.2, C47.2, C48.2, C49.2, C50.2, C51.2, C52.2, C53.2, C54.2, C55.2, C56.2, C57.2, C58.2, C59.2, C60.2, C61.2, C62.2, C63.2, C64.2, C65.2, C66.2, C67.2, C68.2, C69.2, C71.2, C74.2, C75.2, C76.2, C85.2, C86.2, C90.2, C91.2, C92.2, C93.2, C94.2, C95.2, C96.2, C97.2, C98.2, C99.1, IC10.GND, IC10.PAD, IC11.V-, IC12.GND, IC13.V-, IC14.AGND, IC14.PGND, IC15.GND, IC15.PAD, IC20.GND, IC21.ADJ, IC22.GND, IC23.V-, IC24.V-, IC25.V-, IC26.V-, IC27.V-, IC28.V-, IC29.V-, IC30.V-, IC31.V-, IC32.GND, IC33.GND, IC34.GND, IC35.GND, IC36.VSS, IC37.VSS, IC38.GND, IC39.V-, IC6.GND, IC7.AVSS, IC7.DVSS, IC7.IN2-, IC7.IOUT_HV, IC7.IOUT_LV, IC8.GND, IC9.AVSS, IC9.DVSS, IC9.IN2-, IC9.IOUT_HV, IC9.IOUT_LV, J6.GND, J6.GND1, J6.GND2, J6.GND3, J6.SHIELD, L4.1, R103.1, R107.1, R111.1, R115.1, R57.2, R73.2, R87.1, R91.1, R95.1, R99.1; no longer USB1.GND, USB1.SHILED
- net TACHO: now also J2.16
- net TRD0_N: now also D2.D1-; no longer D2.D1+
- net TRD0_P: now also D2.D1+; no longer D2.D1-
- net TRD1_N: now also D2.D2+; no longer D2.D2-
- net TRD1_P: now also D2.D2-; no longer D2.D2+
- net TRD2_N: now also D1.D1-; no longer D1.D1+
- net TRD2_P: now also D1.D1+; no longer D1.D1-
- net TRD3_N: now also D1.D2+; no longer D1.D2-
- net TRD3_P: now also D1.D2-; no longer D1.D2+
- net USB2_N: now also J6.D-1, J6.D-2; no longer USB1.D-
- net USB2_P: now also J6.D+1, J6.D+2; no longer USB1.D+
Other:
- note added: "+/-14V to +/12V LDO"
- note added: "0 0 1 OUT0"
- note added: "0 1 1 OUT1"
- note added: "1 0 1 OUT2"
- note added: "1 1 1 OUT3"
- note added: "2.5V VREF"
- note added: "3.3V SYTEM LDO"
- note added: "3.3V TARGET LDO"
- note added: "5V to +/-14V BOOST CONVERTER"
- note added: "A1 A0 EN ON"
- note added: "ADS9234R ADC"
- note added: "ANALOG-IN TESTPOINTS"
- note added: "ANALOG-OUT DAC"
- note added: "ANALOG-OUT OUTPUT DRIVERS"
- note added: "ANALOG-OUT TESTPOINTS"
- note added: "Choose R_ISOLATION = 68 Ω: 1. Stability with Capacitive Load: The combination of R_ISO and C_LOAD creates a low-pass filter. The cutoff frequency is: f_c = 1 / (2 * π * R_ISO * C_LOAD) For R_ISO = 68 Ω and C_LOAD = 20 nF: f_c = 1 / (2 * π * 68 * 20e-9) ≈ 117.2 kHz 2. Voltage Drop Across R_ISO: The voltage drop is: V_drop = I_load * R_ISO"
- note added: "DAC8568 Output Calculation: V_OUT = (1 + R_FB/R_G2 + R_FB/R_G1) * V_DAC - (R_FB/R_G2) * V_REF Given: Supply voltage: +/-12V Reference voltage (V_REF): 2.5V DAC resolution: 16 bits Desired output range: -12V to +12V 1. Determine the Gain (G): G = (V_OUT_max - V_OUT_min) / (V_DAC_max - V_DAC_min) G = (12 - (-12)) / (2.5 - 0) = 24 / 2.5 = 9.6 2. Solve for Resistor Ratios: G = 1 + R_FB/R_G2 + R_FB/R_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"
- note added: "DIGITAL IO - LOWER 16 BITS"
- note added: "DIGITAL IO - UPPER 16 BITS"
- note added: "DPHY1 JUMPERS"
- note added: "IN0+ AND IN1-"
- note added: "IN10+ AND IN11-"
- note added: "IN12+ AND IN13-"
- note added: "IN14+ AND IN15-"
- note added: "IN2+ AND IN3-"
- note added: "IN4+ AND IN5-"
- note added: "IN6+ AND IN7-"
- note added: "IN8+ AND IN9-"
- note added: "INPUT MULTIPLEXER"
- note added: "Negative Channel: - Known Values: - VBUF = 1.184 V - VOUTN = -12 V - R2N = 10 kΩ - Formula: R1N = -(VOUTN × R2N) / VBUF - Calculation: R1N = -(-12 × 10) / 1.184 R1N = (120 / 1.184) = 101.4 kΩ - Closest Resistor Value (0.1% Tolerance): R1N = 101 kΩ Final Resistor Values: - Negative Channel: - R1N = 101 kΩ - R2N = 10 kΩ - Calculated VOUTN ≈ -12.0 V Negative Channel: - Target VOUTN = -12 V, adjustme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"
- note added: "Negative Output (Vout_neg = -14V): - Given: - R1 = 1.3 MΩ - Calculated R2 ≈ 136.3 kΩ - Nearest E96 Standard Value: - R2 = 137 kΩ - Resulting Output Voltage: - Vout = 1.213 × (1 + R1 / R2) - Vout = 1.213 × (1 + 1300 / 137) ≈ 14.01 V - Final Pair: - R1 = 1.3 MΩ - R2 = 137 kΩ Negative Channel: - Target VOUTN = -14 V, adjustment range: -12.6 V to -15.4 V. - Configuration: - R2N = 137 kΩ (fixed). - R1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"
- note added: "PGA"
- note added: "Positive Channel: - Known Values: - VFBP = 1.184 V - VOUTP = 12 V - R2P = 10 kΩ - Formula: R1P = (VOUTP / VFBP - 1) × R2P - Calculation: R1P = (12 / 1.184 - 1) × 10 R1P = (10.14 - 1) × 10 = 91.4 kΩ - Closest Resistor Value (0.1% Tolerance): R1P = 91.5 kΩ Final Resistor Values: - Positive Channel: - R1P = 91.5 kΩ - R2P = 10 kΩ - Calculated VOUTP ≈ 12.0 V Positive Channel: - Target VOUTP = 12 V, ad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"
- note added: "Positive Output (Vout_pos = 14V): - Given: - R1 = 976 kΩ - Calculated R2 ≈ 102.3 kΩ - Nearest E96 Standard Value: - R2 = 102 kΩ - Resulting Output Voltage: - Vout = 1.213 × (1 + R1 / R2) - Vout = 1.213 × (1 + 976 / 102) ≈ 13.98 V - Final Pair: - R1 = 976 kΩ - R2 = 102 kΩ Positive Channel: - Target VOUTP = 14 V, adjustment range: 12.6 V to 15.4 V. - Configuration: - R2P = 102 kΩ (fixed). - R1P = 9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"
- note added: "TESTPOINTS POWER"
- note added: "X X 0 -"

Commit message: create PCB
Parts:
- removed C114, C116: 100nF, ds_passive:C0402
- removed C115, C117: 4.7uF, ds_passive:C0603
- removed IC20: MIC5504-3.3YM5-TR, ds_ic_vreg:MIC5504-3.3YM5-TR
- removed R81, R82: 0R, ds_passive:R0402
- removed TP100, TP101, TP102, TP103, TP104, TP105, TP106, TP17, TP18, TP19, TP20, TP21, TP22, TP23, TP24, TP25, TP26, TP27, TP28, TP29, TP30, TP31, TP32, TP33, TP34, TP35, TP36, TP37, TP38, TP39, TP40, TP46, TP47, TP48, TP49, TP50, TP51, TP53, TP54, TP55, TP56, TP57, TP80, TP81, TP82, TP83, TP84, TP85, TP89, TP90, TP91, TP92, TP93, TP94, TP95, TP96, TP97, TP98, TP99: PTR1B1,27, testpad:PTR1B1,27
- removed U$2: M.2, ds_con:M.2
- added 12VN, 12VP, 14VN, 14VP, BUF, CLR, DIO_CS, DIO_EN, DIO_GND, DIO_LS, DIO_RST, DIO_VREF, LDAC, REF/2, REFBY2, REFOUT, SPI1_CS0, SYNC, TP9, TPD0, TP_3V3, TP_BSW_G, TP_GND, TP_VFB_14VN, TP_VFB_14VP, TP_VREF_TPS, VCOMB, VFB12VN, VFB12VP, VOCMA, VREFR, VREF_DAC: TP, ds_passive:TP
- added C21: 100nF, ds_passive:C0603
- added C22, C25: 100nF, ds_passive:C0402
- added IC16: SN74LVC2G66, ds_ic_peripherals:SN74LVC2G66
- added IC17: 74LVC1G04, ds_ic_logic:74LVC1G04
- added J7: 2-5174225-5, Connector_D-Sub:2-5174225-5
- added JP4: POE, jumper:JP2Q
- added PCIE: M.2, ds_con:M.2
- added R25, R26, R27, R28, R29, R30, R31, R32, R33, R34, R35, R36, R37, R38, R39, R40, R41: 0R, ds_passive:R0603
- C110, C70: device ds_passive:C0805 -> ds_passive:C0603
- C111, C151, C152, C153, C154, C155, C156, C157, C158, C159, C160, C161, C162, C163, C164, C165, C166, C167, C168, C169, C170, C51, C53, C55, C57, C59, C61, C63, C65, C67, C69, C71: device ds_passive:C0603 -> ds_passive:C0402
- ETH1: value (none) -> G16LX-188S7-1G-GO-Y; device ds_con:MAGJACK -> ds_con:MAGJACK-POE
- IC38: value (none) -> SN74LVC2G66
- R17, R18: device ds_passive:R0402 -> ds_passive:R0603
- R24, R42, R43, R44, R45, R46, R47, R48: device ds_passive:R0603 -> ds_passive:R0402
- renumbered J3 to USB3, J4 to HDMI2, J5 to HDMI1, J6 to USBC, SV2 to GPIO, U$1 to SD1
Connections:
- removed net !CS1_ADC: IC10.!CS, R15.1, TP40.TP
- removed net !CS_ADA_A: IC7.!CS
- removed net !CS_ADA_B: IC9.!CS
- removed net DIO_CS1: IC36.!CS, TP104.TP
- removed net DIO_CS2: IC37.!CS
- removed net EEPROM_WP: JP2.4
- removed net MISO: IC36.SO, IC37.SO, IC7.SDO, IC9.SDO
- removed net MOSI: IC10.SDI, IC22.DIN, IC36.SI, IC37.SI, IC7.SDI, IC9.SDI
- removed net SCK: IC10.SCLK, IC22.SCLK, IC36.SCK, IC37.SCK, IC7.SCK, IC9.SCK
- removed net SDO_A_1: IC10.SDO-1/1A, R18.2
- removed net SDO_A_2: IC10.SDO-2/2A, R81.2
- removed net SDO_A_3: IC10.SDO-3/3A, R82.2
- removed net SDO_B_1: IC10.SDO-5/1B, R18.1
- removed net SDO_B_2: IC10.SDO-6/2B, R81.1
- removed net SDO_B_3: IC10.SDO-7/3B, R82.1
- removed net USBOTG: JP2.10
- removed net V+: C52.1, C53.1, C56.1, C57.1, C60.1, C61.1, C66.1, C67.1, IC6.V+, IC7.VDDH, IC8.V+, IC9.VDDH
- removed net V-: C54.1, C55.1, C58.1, C59.1, C62.1, C63.1, C68.1, C69.1, IC6.V-, IC7.PAD, IC7.VSSH, IC8.V-, IC9.PAD, IC9.VSSH
- new net !MISO_SEL: IC16.2C, IC17.OUT
- new net MISO_SEL: IC16.1C, IC17.IN
- new net SPI0_CS0: DIO_CS.P$1, IC36.!CS, R29.1
- new net SPI0_CS1: IC37.!CS, R30.1
- new net SPI0_MISO: IC36.SO, IC37.SO, R27.1
- new net SPI0_MOSI: IC22.DIN, IC36.SI, IC37.SI, R28.1
- new net SPI0_SCK: IC22.SCLK, IC36.SCK, IC37.SCK, R26.1
- new net SPI1_CS0: IC10.!CS, R15.1, R32.1, SPI1_CS0.P$1
- new net SPI1_CS1: IC7.!CS, R33.1
- new net SPI1_CS2: IC9.!CS, R34.1
- new net SPI1_MISO: IC16.1B, IC16.2B, IC7.SDO, IC9.SDO, R18.1
- new net SPI1_MOSI: IC10.SDI, IC7.SDI, IC9.SDI, R17.1
- new net SPI1_SCK: IC10.SCLK, IC7.SCK, IC9.SCK, R25.1
- new net TR0_TAP: ETH1.VC1, JP4.3
- new net TR1_TAP: ETH1.VC2, JP4.1
- new net TR2_TAP: ETH1.VC3, JP4.2
- new net TR3_TAP: ETH1.VC4, JP4.4
- net !ADC_RST: now also R38.1; no longer TP39.TP
- net +12V: now also 12VP.P$1, C52.1, C53.1, C56.1, C57.1, C60.1, C61.1, C66.1, C67.1, IC6.V+, IC7.VDDH, IC8.V+, IC9.VDDH; no longer TP53.TP
- net +14V: now also 14VP.P$1; no longer TP46.TP
- net +3V3: now also C21.1, C22.1, C25.1, ETH1.P18, ETH1.P20, IC16.VCC, IC17.V+, R86.5, TP_3V3.P$1; no longer C116.1, C117.1, ETH1.P11, ETH1.P14, IC20.VOUT
- net +3V3_EXT: now also J7.52, J7.67
- net +5V: now also J7.18, J7.33; no longer C114.1, C115.1, IC20.EN, IC20.VIN
- net -12V: now also 12VN.P$1, C54.1, C55.1, C58.1, C59.1, C62.1, C63.1, C68.1, C69.1, IC6.V-, IC7.PAD, IC7.VSSH, IC8.V-, IC9.PAD, IC9.VSSH; no longer TP54.TP
- net -14V: now also 14VN.P$1; no longer TP47.TP
- net ADC_AIN_N: no longer TP22.TP
- net ADC_AIN_P: no longer TP21.TP
- net ADC_BIN_N: no longer TP24.TP
- net ADC_BIN_P: no longer TP23.TP
- net ADC_IN0: no longer TP17.TP
- net ADC_IN1: no longer TP18.TP
- net ADC_IN2: no longer TP19.TP
- net ADC_IN3: no longer TP20.TP
- net ADC_RDY: now also R36.1; no longer TP28.TP
- net AO_0: now also J7.29
- net AO_1: now also J7.63
- net AO_2: now also J7.30
- net AO_3: now also J7.64
- net AO_4: now also J7.31
- net AO_5: now also J7.65
- net AO_6: now also J7.32
- net AO_7: now also J7.66
- net BSW_G: now also TP_BSW_G.P$1; no longer TP51.TP
- net BUF: now also BUF.P$1; no longer TP57.TP
- net DAC_!CLR: now also CLR.P$1, R37.1, R86.4; no longer R86.1, TP93.TP
- net DAC_!LDAC: now also LDAC.P$1, R35.1, R86.2; no longer R86.3, TP89.TP
- net DAC_!SYNC: now also R31.1, R86.3, SYNC.P$1; no longer R86.2, TP91.TP
- net DAC_0: now also TPD0.P$1; no longer TP90.TP
- net DAC_1: no longer TP92.TP
- net DAC_2: no longer TP94.TP
- net DAC_3: no longer TP96.TP
- net DAC_4: no longer TP97.TP
- net DAC_5: no longer TP98.TP
- net DAC_6: no longer TP99.TP
- net DAC_7: no longer TP100.TP
- net DIO_0: now also J7.2, R120.5; no longer R119.8
- net DIO_1: now also J7.3, R120.6; no longer R119.7
- net DIO_10: now also J7.12, R122.7; no longer R121.6
- net DIO_11: now also J7.13, R122.8; no longer R121.5
- net DIO_12: now also J7.14, R121.5; no longer R122.8
- net DIO_13: now also J7.15, R121.6; no longer R122.7
- net DIO_14: now also J7.16, R121.7; no longer R122.6
- net DIO_15: now also J7.17, R121.8; no longer R122.5
- net DIO_16: now also J7.36, R124.5; no longer R123.8
- net DIO_17: now also J7.37, R124.6; no longer R123.7
- net DIO_18: now also J7.38, R124.7; no longer R123.6
- net DIO_19: now also J7.39, R124.8; no longer R123.5
- net DIO_2: now also J7.4, R120.7; no longer R119.6
- net DIO_20: now also J7.40, R123.5; no longer R124.8
- net DIO_21: now also J7.41, R123.6; no longer R124.7
- net DIO_22: now also J7.42, R123.7; no longer R124.6
- net DIO_23: now also J7.43, R123.8; no longer R124.5
- net DIO_24: now also J7.44, R126.5; no longer R125.8
- net DIO_25: now also J7.45, R126.6; no longer R125.7
- net DIO_26: now also J7.46, R126.7; no longer R125.6
- net DIO_27: now also J7.47, R126.8; no longer R125.5
- net DIO_28: now also J7.48, R125.5; no longer R126.8
- net DIO_29: now also J7.49, R125.6; no longer R126.7
- net DIO_3: now also J7.5, R120.8; no longer R119.5
- net DIO_30: now also J7.50, R125.7; no longer R126.6
- net DIO_31: now also J7.51, R125.8; no longer R126.5
- net DIO_4: now also J7.6, R119.5; no longer R120.8
- net DIO_5: now also J7.7, R119.6; no longer R120.7
- net DIO_6: now also J7.8, R119.7; no longer R120.6
- net DIO_7: now also J7.9, R119.8; no longer R120.5
- net DIO_8: now also J7.10, R122.5; no longer R121.8
- net DIO_9: now also J7.11, R122.6; no longer R121.7
- net DIO_EN: now also DIO_EN.P$1, R41.1; no longer TP103.TP
- net DIO_LEVEL_SELECT: now also DIO_LS.P$1, R40.1; no longer TP101.TP, TP106.TP
- net DIO_RESET: now also DIO_RST.P$1, R39.1; no longer TP105.TP
- net EEPROM_NWP: now also JP2.4
- net GND: now also C21.2, C22.2, C25.2, DIO_GND.P$1, IC16.GND, IC17.V-, J7.1, J7.23, J7.28, J7.34, J7.35, J7.57, J7.62, J7.68, J7.MH1, J7.MH2, PCIE.GND1, PCIE.GND10, PCIE.GND11, PCIE.GND12, PCIE.GND13, PCIE.GND14, PCIE.GND2, PCIE.GND3, PCIE.GND4, PCIE.GND5, PCIE.GND6, PCIE.GND7, PCIE.GND8, PCIE.GND9, PCIE.S1, PCIE.S2, TP_GND.P$1; no longer C114.2, C115.2, C116.2, C117.2, IC20.GND, U$2.GND1, U$2.GND10, U$2.GND11, U$2.GND12, U$2.GND13, U$2.GND14, U$2.GND2, U$2.GND3, U$2.GND4, U$2.GND5, U$2.GND6, U$2.GND7, U$2.GND8, U$2.GND9, U$2.S1, U$2.S2
- net GPIO10: now also R28.2
- net GPIO11: now also R26.2
- net GPIO13: now also R40.2
- net GPIO16: now also R34.2
- net GPIO17: now also R33.2
- net GPIO18: now also R32.2
- net GPIO19: now also R18.2
- net GPIO20: now also R17.2
- net GPIO21: now also R25.2
- net GPIO23: now also R31.2
- net GPIO24: now also R36.2
- net GPIO25: now also R38.2
- net GPIO27: now also R35.2
- net GPIO4: now also R37.2
- net GPIO5: now also R41.2
- net GPIO6: now also R39.2
- net GPIO7: now also R30.2
- net GPIO8: now also R29.2
- net GPIO9: now also R27.2
- net IN0+: now also J7.19
- net IN1-: now also J7.53
- net IN10+: now also J7.25
- net IN11-: now also J7.59
- net IN12+: now also J7.26
- net IN13-: now also J7.60
- net IN14+: now also J7.27
- net IN15-: now also J7.61
- net IN2+: now also J7.20
- net IN3-: now also J7.54
- net IN4+: now also J7.21
- net IN5-: now also J7.55
- net IN6+: now also J7.22
- net IN7-: now also J7.56
- net IN8+: now also J7.24
- net IN9-: now also J7.58
- net M2_3V3: now also PCIE.VCC1, PCIE.VCC2, PCIE.VCC3, PCIE.VCC4, PCIE.VCC5, PCIE.VCC6, PCIE.VCC7, PCIE.VCC8, PCIE.VCC9; no longer U$2.VCC1, U$2.VCC2, U$2.VCC3, U$2.VCC4, U$2.VCC5, U$2.VCC6, U$2.VCC7, U$2.VCC8, U$2.VCC9
- net MUX_A_OUTA: no longer TP33.TP
- net MUX_A_OUTB: no longer TP34.TP
- net MUX_B_OUTA: no longer TP35.TP
- net MUX_B_OUTB: no longer TP36.TP
- net N$108: now also IC35.A6; no longer IC35.A3
- net N$109: now also IC35.A5; no longer IC35.A4
- net N$11: now also PCIE.SUSCLK; no longer U$2.SUSCLK
- net N$110: now also IC35.A4; no longer IC35.A5
- net N$111: now also IC35.A3; no longer IC35.A6
- net N$112: now also IC35.A2; no longer IC35.A7
- net N$113: now also IC35.A1; no longer IC35.A8
- net N$114: now also IC35.A7; no longer IC35.A2
- net N$115: now also IC35.A8; no longer IC35.A1
- net N$29: now also IC33.A7; no longer IC33.A2
- net N$4: now also ETH1.CT1, ETH1.CT2, ETH1.CT3, ETH1.CT4; no longer ETH1.P1, ETH1.P10
- net N$5: now also ETH1.P17; no longer ETH1.P13
- net N$6: now also PCIE.DA5/!DSS!/!LED1; no longer U$2.DA5/!DSS!/!LED1
- net N$61: now also IC32.A8; no longer IC32.A1
- net N$62: now also IC32.A7; no longer IC32.A2
- net N$63: now also IC32.A6; no longer IC32.A3
- net N$64: now also IC32.A5; no longer IC32.A4
- net N$65: now also IC32.A4; no longer IC32.A5
- net N$66: now also IC32.A3; no longer IC32.A6
- net N$67: now also IC32.A2; no longer IC32.A7
- net N$68: now also IC32.A1; no longer IC32.A8
- net N$77: now also IC33.A8; no longer IC33.A1
- net N$78: now also IC33.A6; no longer IC33.A3
- net N$79: now also IC33.A5; no longer IC33.A4
- net N$8: now also ETH1.P19; no longer ETH1.P12
- net N$80: now also IC33.A4; no longer IC33.A5
- net N$81: now also IC33.A3; no longer IC33.A6
- net N$82: now also IC33.A2; no longer IC33.A7
- net N$83: now also IC33.A1; no longer IC33.A8
- net N$92: now also IC34.A8; no longer IC34.A1
- net N$93: now also IC34.A7; no longer IC34.A2
- net N$94: now also IC34.A6; no longer IC34.A3
- net N$95: now also IC34.A5; no longer IC34.A4
- net N$96: now also IC34.A4; no longer IC34.A5
- net N$97: now also IC34.A3; no longer IC34.A6
- net N$98: now also IC34.A2; no longer IC34.A7
- net N$99: now also IC34.A1; no longer IC34.A8
- net PCIE_CLK_N: now also PCIE.REFCLK_N; no longer U$2.REFCLK_N
- net PCIE_CLK_P: now also PCIE.REFCLK_P; no longer U$2.REFCLK_P
- net PCIE_NCLKREQ: now also PCIE.!CLKREQ; no longer U$2.!CLKREQ
- net PCIE_NRST: now also PCIE.!PERST; no longer U$2.!PERST
- net PCIE_NWAKE: now also PCIE.!PEWAKE; no longer U$2.!PEWAKE
- net PCIE_RX_N: now also PCIE.PET_P0; no longer U$2.PET_P0
- net PCIE_RX_P: now also PCIE.PET_N0; no longer U$2.PET_N0
- net PCIE_TX_N: now also PCIE.PER_P0; no longer U$2.PER_P0
- net PCIE_TX_P: now also PCIE.PER_N0; no longer U$2.PER_N0
- net PGA_A_IN+: no longer TP29.TP
- net PGA_A_IN-: no longer TP30.TP
- net PGA_B_IN+: no longer TP31.TP
- net PGA_B_IN-: no longer TP32.TP
- net REFBY2: now also REFBY2.P$1; no longer TP85.TP
- net REFM_A: no longer TP81.TP
- net REFM_B: no longer TP83.TP
- net REFOUT: now also REFOUT.P$1; no longer TP84.TP
- net REFP_A: no longer TP80.TP
- net REFP_B: no longer TP82.TP
- net SDO_A_0: now also IC16.1A; no longer R17.2
- net SDO_B_0: now also IC16.2A; no longer R17.1
- net TRD0_N: now also ETH1.TD1-; no longer ETH1.P3
- net TRD0_P: now also ETH1.TD1+; no longer ETH1.P2
- net TRD1_N: now also ETH1.TD2-; no longer ETH1.P5
- net TRD1_P: now also ETH1.TD2+; no longer ETH1.P4
- net TRD2_N: now also D1.D2+, ETH1.TD3-; no longer D1.D1-, ETH1.P7
- net TRD2_P: now also D1.D2-, ETH1.TD3+; no longer D1.D1+, ETH1.P6
- net TRD3_N: now also D1.D1-, ETH1.TD4-; no longer D1.D2+, ETH1.P9
- net TRD3_P: now also D1.D1+, ETH1.TD4+; no longer D1.D2-, ETH1.P8
- net USBOTG_ID: now also JP2.10
- net VFB_12VN: now also VFB12VN.P$1; no longer TP56.TP
- net VFB_12VP: now also VFB12VP.P$1; no longer TP55.TP
- net VFB_14VN: now also TP_VFB_14VN.P$1; no longer TP49.TP
- net VFB_14VP: now also TP_VFB_14VP.P$1; no longer TP48.TP
- net VOCM_A: now also VOCMA.P$1; no longer TP37.TP
- net VOCM_B: now also VCOMB.P$1; no longer TP38.TP
- net VREF_ADC: now also TP9.P$1; no longer TP25.TP
- net VREF_ADC/2: now also REF/2.P$1; no longer TP27.TP
- net VREF_ADC_RAW: now also VREFR.P$1; no longer TP26.TP
- net VREF_DAC_OUT: now also VREF_DAC.P$1; no longer TP95.TP
- net VREF_TPS: now also TP_VREF_TPS.P$1; no longer TP50.TP
- net V_OUT_REF: now also DIO_VREF.P$1; no longer TP102.TP
Other:
- note added: "ADC ON SPI1"
- note added: "ADC_RDY"
- note added: "ADC_RST"
- note added: "DAC_CLR"
- note added: "DAC_LDAC"
- note added: "DAC_SYNC"
- note added: "DIO ON SPI0"
- note added: "DIO_EN"
- note added: "DIO_LS"
- note added: "DIO_RST"
- note added: "I2C"
- note added: "IO-GPIO JUMPERS"
- note added: "SPI0"
- note added: "SPI1"
- note added: "TEST CONNECTOR"
- note added: "UART_RX"
- note added: "UART_TX"
- note removed: "3.3V SYTEM LDO"
- moved on the sheet: 2230, 2242, 2260, 2280, C11, C12, D1, D2, LED2, R10, R8, R9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

Commit message: 3D render
Parts:
- removed C118, C119: 100uF, rcl:CPOL-EU153CLV-0605
- removed IC21: LD117ADT33TR, v-reg:LD117ADT33TR
- removed R77, R78: 20K, pot:TRIM_EU-3223G
- removed R79, R80: 250K, pot:TRIM_EU-3223G
- removed S1: (no value), adafruit:31-XX
- removed SV1: (no value), con-lstb:MA04-1
- removed X1: ASEK-32.768KHz-LRT, crystal-geyer_V1_0:KXO-PXO/XO-V96
- added C26, C27: 100uF 16V, ds_passive:CPOL
- added CON1: (no value), ds_con:CON-1X4
- added IC18: (no value), ds_ic_vreg:LDL1117S33R
- added R53, R54, R55, R56: (no value), ds_passive:R-TRIM
- added SW1: 1825027-8, ds_passive:1825027-8
- added X2: CRYSTAL, ds_passive:CRYSTAL
- C8: value 100uF -> 100uF 16V; device rcl:CPOL-EU153CLV-0505 -> ds_passive:CPOL
- GPIO: device con-lstb:MA20-2 -> ds_con:CON-2X20
- IC12: value REF3025 -> MCP1525T-I/TT; device maxim:MAX6520 -> ds_ic_vreg:MCP1525T-I/TT
- IC6, IC8: device ds_ic_peripherals:DG409 -> ds_ic_peripherals:DG409EUE+
- JP1, JP3, JP4: device jumper:JP2Q -> ds_con:CON-2X2
- JP2: device jumper:JP7Q -> ds_con:CON-2X7
- L1: value (none) -> L; device rcl:L-USL5038P -> ds_passive:L
- L3, L4: value B8246284-4.7uH -> SRR5228A-4R7Y; device inductor-coilcraft:MSS7341 -> ds_passive:L
- R49: value 20K -> (none); device pot:TRIM_EU-3223G -> ds_passive:R-TRIM
- SD1: value MICROSD -> (none); device adafruit:MICROSD -> ds_con:MICRO-SD
Connections:
- net +3V3: now also IC12.VIN; no longer IC12.IN
- net +3V3_EXT: now also C27.1, IC18.VOUT; no longer C119.+, IC21.OUT
- net +5V: now also C26.1, CON1.P$4, IC18.VIN; no longer C118.+, IC21.IN, SV1.4
- net GND: now also C26.2, C27.2, C8.2, CON1.P$2, IC18.GND, SD1.MT1, SD1.MT2, SD1.MT3, SD1.MT4, SW1.1, SW1.3, SW1.4, X2.VSS; no longer C118.-, C119.-, C8.-, IC21.ADJ, S1.S, SD1.GND, SD1.GND1, SV1.2, X1.GND
- net M2_3V3: now also X2.OUT, X2.VDD; no longer X1.TS, X1.VDD
- net N$11: now also X2.CON; no longer X1.OUT
- net N$19: now also R49.1; no longer R49.A
- net N$20: now also R49.2; no longer R49.S
- net N$38: now also R55.2, R55.3; no longer R77.E, R77.S
- net N$42: now also R56.2, R56.3; no longer R78.E, R78.S
- net N$43: now also R53.2, R53.3; no longer R79.E, R79.S
- net N$44: now also R54.2, R54.3; no longer R80.E, R80.S
- net PWM: now also CON1.P$3; no longer SV1.3
- net PWR_BUT: now also SW1.2; no longer S1.P
- net SD_CLK: now also SD1.CLK; no longer SD1.SCLK
- net SD_CMD: now also SD1.CMD; no longer SD1.DATA_IN
- net SD_DAT0: now also SD1.DAT0; no longer SD1.DATA_OUT
- net SD_DAT3: now also SD1.CD/DAT3; no longer SD1.CS
- net TACHO: now also CON1.P$1; no longer SV1.1
- net VBUS: now also C8.1; no longer C8.+
- net VFB_12VN: now also R56.1; no longer R78.A
- net VFB_12VP: now also R55.1; no longer R77.A
- net VFB_14VN: now also R54.1; no longer R80.A
- net VFB_14VP: now also R53.1; no longer R79.A
- net VREF_ADC: now also R49.3; no longer R49.E
- net VREF_ADC_RAW: now also IC12.VREF; no longer IC12.OUT
Other:
- moved on the sheet: C12, C46, C48, C49, GPIO, IC13
