File: src/HardwareDesign/Dataforge-Pi.brd (EAGLE design)
At the start: 180 x 100 mm, 364 parts, among them IC1 RT9742GGJ, IC10 ADS9234RIRHBR, IC11 MCP6001RT, IC12 MCP1525T-I/TT, IC13 MCP6001RT, IC14 TPS65131, IC15 TPS7A39, IC16 SN74LVC2G66, IC17 74LVC1G04, IC2 AP22653W6, IC22 DAC8568, IC23 MCP6001RT, IC24 MCP6001RT, IC25 MCP6001RT, IC26 MCP6001RT, IC27 MCP6001RT, IC28 MCP6001RT, IC29 MCP6001RT, IC3 74LVC1G07, IC30 MCP6001RT, IC31 MCP6001RT, IC32 LSF0108, IC33 LSF0108, IC34 LSF0108, IC35 LSF0108, IC36 MCP23S18, IC38 SN74LVC2G66, IC39 74LVC1G04, IC4 RT9742NGV, IC5 AP3441SHE-7B, IC6 DG409, IC7 ADA4254ACPZ, IC8 DG409, IC9 ADA4254ACPZ, J1 10164227-1001A1RLF, J2 10164227-1001A1RLF, J3 FH12-22S-0.5SVA, J4 FH12-22S-0.5SH(55), J7 2-5174225-5, SW1 1825027-8, T2 IRLML5203, X2 CRYSTAL

Commit message: Baseboard design ready
Parts:
- removed 12VN, 12VP, 14VN, 14VP, BUF, CLR, DIO_CS, DIO_EN, DIO_GND, DIO_LS, DIO_RST, DIO_VREF, LDAC, REF/2, REFBY2, REFOUT, SPI1_CS0, SYNC, TP-VBAT, TP9, TPD0, TP_3V3, TP_BSW_G, TP_GND, TP_VFB_14VN, TP_VFB_14VP, TP_VREF_TPS, VCOMB, VFB12VN, VFB12VP, VOCMA, VREFR, VREF_DAC: TP, ds_passive:TP
- removed BT1: 79523141, Battery Holder:79523141
- removed C100, C101: 10pF, ds_passive:0402
- removed C102, C104: 10uF, ds_passive:1206
- removed C103, C106, C107: 10nF, ds_passive:0402
- removed C105, C99: 220nF, ds_passive:0402
- removed C108, C109, C93, C94, C95, C96, C97, C98: 22uF, ds_passive:1206
- removed C110, C70: 10uF, ds_passive:0603
- removed C111, C120, C121, C125, C126, C128, C129, C131, C132, C134, C135, C137, C138, C140, C141, C143, C144, C146, C147, C149, C150, C152, C154, C156, C158, C160, C162, C164, C166, C168, C170, C22, C25, C45, C46, C49, C51, C53, C55, C57, C59, C61, C63, C65, C67, C69, C71, C75, C76: 100nF, ds_passive:0402
- removed C122, C124, C50, C52, C54, C56, C58, C60, C62, C64, C66, C68, C72: 1uF, ds_passive:0603
- removed C123, C171, C73: 100nF, ds_passive:0603
- removed C127, C130, C133, C136, C139, C142, C145, C148: 20nF, ds_passive:0402
- removed C151, C153, C155, C157, C159, C161, C163, C165, C167, C169: 1uF, ds_passive:0402
- removed C23, C24, C42, C43: 270pF, ds_passive:0402
- removed C26, C27: 100uF 16V, ds_passive:100UF-16V
- removed C41, C44: 680pF, ds_passive:0402
- removed C47, C90: 10uF, ds_passive:0805
- removed C48, C74: (no value), ds_passive:0805
- removed C85: 4.7uF, ds_passive:0805
- removed C86: 100nF, ds_passive:0805
- removed C91: 10nF, ds_passive:0805
- removed C92: 4.7nF, ds_passive:0805
- removed CON1: (no value), ds_con:1X4
- removed D3, D4: SS12, Diodes:SMA
- removed IC10: ADS9234RIRHBR, ds_ic_peripherals:VQFN32-5X5
- removed IC11, IC13, IC23, IC24, IC25, IC26, IC27, IC28, IC29, IC30, IC31: MCP6001RT, ds_ic_opa:SOT23-5
- removed IC12: MCP1525T-I/TT, ds_ic_vreg:SOT23
- removed IC14: TPS65131, ds_ic_vreg:VQFN24-4X4-THERMAL2.5X2.5
- removed IC15: TPS7A39, ds_ic_vreg:WSON10-3X3
- removed IC16, IC38: SN74LVC2G66, ds_ic_peripherals:SOP50P310X90-8N
- removed IC17, IC39: 74LVC1G04, ds_ic_logic:SOT95P280X145-5N
- removed IC18: (no value), ds_ic_vreg:SOT230
- removed IC22: DAC8568, ds_ic_peripherals:TSSOP16
- removed IC32, IC33, IC34, IC35: LSF0108, ds_ic_peripherals:VQFN20
- removed IC36: MCP23S18, ds_ic_peripherals:QFN50P400X400X100-25T265
- removed IC37: (no value), ds_ic_peripherals:QFN50P400X400X100-25T265
- removed IC6, IC8: DG409, ds_ic_peripherals:TSSOP2
- removed IC7, IC9: ADA4254ACPZ, ds_ic_opa:QFN50P500X500X75-29T314N
- removed J7: 2-5174225-5, Connector_D-Sub:2-5174225-5
- removed JP1: (no value), ds_con:2X2
- removed JP4: POE, ds_con:2X2
- removed L3, L4: SRR5228A-4R7Y, ds_passive:SRR5228A
- removed R100, R103, R104, R107, R108, R111, R112, R115, R116, R73, R76, R87, R88, R91, R92, R95, R96, R99: 10K 0.1%, ds_passive:0402
- removed R101, R105, R109, R113, R117, R89, R93, R97: 43K 0.1%, ds_passive:0402
- removed R102, R106, R110, R114, R118, R90, R94, R98: 68R 1%, ds_passive:0402
- removed R119, R120, R121, R122, R123, R124, R125, R126: YC164-JR-0733RL, Resistor Array:YC164-JR-0733RL
- removed R127, R128, R129, R130: 200K, ds_passive:0402
- removed R14: 100R, ds_passive:1206
- removed R15, R24, R42, R43, R44, R45, R46, R47, R48: 0R, ds_passive:0402
- removed R16: 10K, ds_passive:0402
- removed R17, R18, R25, R26, R27, R28, R29, R30, R31, R32, R33, R34, R35, R36, R37, R38, R39, R40, R41, R51, R52: 0R, ds_passive:0603
- removed R19: 950K 0.1%, ds_passive:0402
- removed R20, R21, R22, R23: 200R, ds_passive:0402
- removed R49, R53, R54, R55, R56: (no value), ds_passive:TC33X
- removed R50: 100R, ds_passive:0402
- removed R57: 102K 0.1%, ds_passive:0402
- removed R58: 1.2M 0.1%, ds_passive:0402
- removed R59: 137K 0.1%, ds_passive:0402
- removed R60: 75K 0.1%, ds_passive:0402
- removed R74: 90K 0.1%, ds_passive:0402
- removed R86: CRA034RF100RP05Z, Resistor Array:YC164-JR-0733RL
- removed T2: IRLML5203, transistor-power:MICRO3
- removed USB3: 692141030100, Wurth_Connectors_WR-USB:692141030100
- added CON2, CON3: (no value), ds_con:2X20
- added FAN: (no value), ds_con:1X4
- added ID: (no value), ds_con:2X2
- added PI1: (no value), ds_ic_peripherals:CM5
- added POE: POE, ds_con:2X2
- added X1, X3: CON-VG_MAB642, ds_con:CON-VG-MAB64-RECEPTACLE
- C21: value 100nF -> 100uF 16V; device ds_passive:0603 -> ds_passive:100UF-16V
- J1, J2: value 10164227-1001A1RLF -> 692121030100; device ds_con:AMPHENOL_10164227-1001A1RLF -> Wurth_Connectors_WR-USB:692121030100
- J4: value FH12-22S-0.5SH(55) -> FH12-22S-0.5SVA; device ds_con:CONN_FH12-22S-0.5SH(55)_HIR -> ds_con:FH12-22S-0.5SH
- moved C2 174.4 mm to (180.2, 88.7), turned to 0 degrees
- moved USBC 167.4 mm to (177.4, 97.3)
- moved R1 165.9 mm to (180.2, 89.9)
- moved C21 160.3 mm to (186.6, 90.2), turned to 90 degrees
- moved C1 159.5 mm to (173.8, 90.0), turned to 180 degrees
- moved TP_5VP 113.9 mm to (123.5, 10.2)
- moved J2 90.2 mm to (65.8, -6.30), turned to 0 degrees
- moved C10 84.0 mm to (131.3, 2.25), turned to 90 degrees
- moved IC1 82.0 mm to (128.5, 2.74), turned to 90 degrees
- moved J1 82.0 mm to (84.4, -6.36), turned to 0 degrees
- moved SD1 81.3 mm to (129.5, -7.62)
- moved TP-VSD 79.1 mm to (132.8, 5.37), turned to 0 degrees
- moved TP-BTN 71.2 mm to (148.0, 88.9), turned to 90 degrees
- moved TP-5VP 62.1 mm to (158.1, 79.6), turned to 0 degrees
- moved C3 58.6 mm to (75.5, 98.2), turned to 0 degrees
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Connections:
- removed net !DIO_LEVEL_SELECT: IC38.3, IC39.4
- removed net !MISO_SEL: IC16.3, IC17.4
- removed net +12V: 12VP.TP, C107.2, C108.1, C52.1, C53.1, C56.1, C57.1, C60.1, C61.1, C66.1, C67.1, IC15.10, IC6.14, IC7.26, IC8.14, IC9.26, R60.1
- removed net +14V: 14VP.TP, C100.1, C104.1, C93.1, C94.1, C95.1, D3.C, IC14.23, IC15.1, IC15.2, R19.1
- removed net +3V3_EXT: C121.1, C27.1, IC18.2, IC18.4, J7.52, J7.67
- removed net -12V: 12VN.TP, C106.1, C109.1, C54.1, C55.1, C58.1, C59.1, C62.1, C63.1, C68.1, C69.1, IC15.6, IC6.3, IC7.27, IC7.29, IC8.3, IC9.27, IC9.29, R76.2
- removed net -14V: 14VN.TP, C101.1, C102.1, C96.1, C97.1, C98.1, D4.A, IC14.15, IC15.5, R59.2
- removed net ADA_A_IO0: IC6.1, IC7.18
- removed net ADA_A_IO1: IC6.16, IC7.17
- removed net ADA_A_IO2: IC6.2, IC7.16
- removed net ADA_B_IO0: IC8.1, IC9.18
- removed net ADA_B_IO1: IC8.16, IC9.17
- removed net ADA_B_IO2: IC8.2, IC9.16
- removed net ADC_AIN_N: C24.2, C41.2, R21.1, R46.1
- removed net ADC_AIN_P: C23.1, C41.1, R20.1, R45.2
- removed net ADC_BIN_N: C43.2, C44.2, R23.1, R48.2
- removed net ADC_BIN_P: C42.1, C44.1, R22.1, R47.1
- removed net ADC_IN0: IC10.1, R45.1
- removed net ADC_IN1: IC10.2, R46.2
- removed net ADC_IN2: IC10.8, R48.1
- removed net ADC_IN3: IC10.7, R47.2
- removed net AO_0: C127.1, J7.29, R89.2, R90.2
- removed net AO_1: C130.1, J7.63, R93.2, R94.2
- removed net AO_2: C133.1, J7.30, R97.2, R98.2
- removed net AO_3: C136.1, J7.64, R101.2, R102.2
- removed net AO_4: C139.1, J7.31, R105.2, R106.2
- removed net AO_5: C142.1, J7.65, R109.2, R110.2
- removed net AO_6: C145.1, J7.32, R113.2, R114.2
- removed net AO_7: C148.1, J7.66, R117.2, R118.2
- removed net BSW_G: IC14.7, T2.1, TP_BSW_G.TP
- removed net BUF: BUF.TP, C105.2, IC15.8, R74.1
- removed net DAC_!SYNC: IC22.2, R31.1, R86.3, SYNC.TP
- removed net DAC_0: IC22.4, IC24.3, TPD0.TP
- removed net DAC_1: IC22.13, IC25.3
- removed net DAC_2: IC22.5, IC26.3
- removed net DAC_3: IC22.12, IC27.3
- removed net DAC_4: IC22.6, IC28.3
- removed net DAC_5: IC22.11, IC29.3
- removed net DAC_6: IC22.7, IC30.3
- removed net DAC_7: IC22.10, IC31.3
- removed net DIO_0: J7.2, R120.5
- removed net DIO_1: J7.3, R120.6
- removed net DIO_10: J7.12, R122.7
- removed net DIO_11: J7.13, R122.8
- removed net DIO_12: J7.14, R121.5
- removed net DIO_13: J7.15, R121.6
- removed net DIO_14: J7.16, R121.7
- removed net DIO_15: J7.17, R121.8
- removed net DIO_16: J7.36, R124.5
- removed net DIO_17: J7.37, R124.6
- removed net DIO_18: J7.38, R124.7
- removed net DIO_19: J7.39, R124.8
- removed net DIO_2: J7.4, R120.7
- removed net DIO_20: J7.40, R123.5
- removed net DIO_21: J7.41, R123.6
- removed net DIO_22: J7.42, R123.7
- removed net DIO_23: J7.43, R123.8
- removed net DIO_24: J7.44, R126.5
- removed net DIO_25: J7.45, R126.6
- removed net DIO_26: J7.46, R126.7
- removed net DIO_27: J7.47, R126.8
- removed net DIO_28: J7.48, R125.5
- removed net DIO_29: J7.49, R125.6
- removed net DIO_3: J7.5, R120.8
- removed net DIO_30: J7.50, R125.7
- removed net DIO_31: J7.51, R125.8
- removed net DIO_4: J7.6, R119.5
- removed net DIO_5: J7.7, R119.6
- removed net DIO_6: J7.8, R119.7
- removed net DIO_7: J7.9, R119.8
- removed net DIO_8: J7.10, R122.5
- removed net DIO_9: J7.11, R122.6
- removed net IN0+: IC6.4, J7.19
- removed net IN1-: IC6.13, J7.53
- removed net IN10+: IC8.5, J7.25
- removed net IN11-: IC8.12, J7.59
- removed net IN12+: IC8.6, J7.26
- removed net IN13-: IC8.11, J7.60
- removed net IN14+: IC8.7, J7.27
- removed net IN15-: IC8.10, J7.61
- removed net IN2+: IC6.5, J7.20
- removed net IN3-: IC6.12, J7.54
- removed net IN4+: IC6.6, J7.21
- removed net IN5-: IC6.11, J7.55
- removed net IN6+: IC6.7, J7.22
- removed net IN7-: IC6.10, J7.56
- removed net IN8+: IC8.4, J7.24
- removed net IN9-: IC8.13, J7.58
- removed net MUX_A_OUTA: IC6.8, R43.2
- removed net MUX_A_OUTB: IC6.9, R44.1
- removed net MUX_B_OUTA: IC8.8, R24.2
- removed net MUX_B_OUTB: IC8.9, R42.1
- removed net N$100: IC34.18, R123.1
- removed net N$101: IC34.17, R123.2
- removed net N$102: IC34.16, R123.3
- removed net N$103: IC34.15, R123.4
- removed net N$104: IC34.14, R124.1
- removed net N$105: IC34.13, R124.2
- removed net N$106: IC34.12, R124.3
- removed net N$107: IC34.11, R124.4
- removed net N$108: IC35.8, IC37.2
- removed net N$109: IC35.7, IC37.3
- removed net N$110: IC35.6, IC37.4
- removed net N$111: IC35.5, IC37.5
- removed net N$112: IC35.4, IC37.6
- removed net N$113: IC35.3, IC37.7
- removed net N$114: IC35.9, IC37.1
- removed net N$115: IC35.10, IC37.24
- removed net N$116: IC35.18, R125.1
- removed net N$117: IC35.17, R125.2
- removed net N$118: IC35.16, R125.3
- removed net N$119: IC35.15, R125.4
- removed net N$12: IC7.19, R20.2
- removed net N$120: IC35.14, R126.1
- removed net N$121: IC35.13, R126.2
- removed net N$122: IC35.12, R126.3
- removed net N$123: IC35.11, R126.4
- removed net N$124: IC32.19, R127.1
- removed net N$125: IC33.19, R128.1
- removed net N$126: IC35.19, R129.1
- removed net N$127: IC34.19, R130.1
- removed net N$13: IC7.20, R21.2
- removed net N$14: C129.2, IC24.1, R90.1
- removed net N$15: IC9.19, R22.2
- removed net N$16: IC9.20, R23.2
- removed net N$17: C129.1, IC24.4, R87.2, R88.2, R89.1
- removed net N$18: IC10.13, R15.2
- removed net N$19: C72.2, C73.2, R49.1
- removed net N$20: C74.1, R49.2, R50.1
- removed net N$21: IC11.3, R50.2
- removed net N$22: C132.1, IC25.4, R91.2, R92.2, R93.1
- removed net N$23: C132.2, IC25.1, R94.1
- removed net N$24: D3.A, IC14.1, IC14.24, L3.2
- removed net N$25: C135.1, IC26.4, R95.2, R96.2, R97.1
- removed net N$26: C135.2, IC26.1, R98.1
- removed net N$27: C138.1, IC27.4, R100.2, R101.1, R99.2
- removed net N$28: C138.2, IC27.1, R102.1
- removed net N$29: IC33.9, IC36.1
- removed net N$30: C90.1, L3.1, T2.3
- removed net N$31: C141.1, IC28.4, R103.2, R104.2, R105.1
- removed net N$32: C86.1, IC14.10, IC14.11, IC14.4, IC14.8, IC14.9, R14.1
- removed net N$33: C141.2, IC28.1, R106.1
- removed net N$34: C144.1, IC29.4, R107.2, R108.2, R109.1
- removed net N$35: C91.1, IC14.21
- removed net N$36: C92.1, IC14.18
- removed net N$37: D4.C, IC14.13, IC14.14, L4.2
- removed net N$38: R55.2, R55.3, R60.2
- removed net N$39: C103.1, IC15.3
- removed net N$40: C144.2, IC29.1, R110.1
- removed net N$41: C147.1, IC30.4, R111.2, R112.2, R113.1
- removed net N$42: R56.2, R56.3, R74.2
- removed net N$43: R19.2, R53.2, R53.3
- removed net N$44: R54.2, R54.3, R58.2
- removed net N$58: C147.2, IC30.1, R114.1
- removed net N$59: C150.1, IC31.4, R115.2, R116.2, R117.1
- removed net N$60: C150.2, IC31.1, R118.1
- removed net N$61: IC32.10, IC36.15
- removed net N$62: IC32.9, IC36.16
- removed net N$63: IC32.8, IC36.17
- removed net N$64: IC32.7, IC36.18
- removed net N$65: IC32.6, IC36.19
- removed net N$66: IC32.5, IC36.20
- removed net N$67: IC32.4, IC36.21
- removed net N$68: IC32.3, IC36.22
- removed net N$69: IC32.18, R119.1
- removed net N$70: IC32.17, R119.2
- removed net N$71: IC32.16, R119.3
- removed net N$72: IC32.15, R119.4
- removed net N$73: IC32.14, R120.1
- removed net N$74: IC32.13, R120.2
- removed net N$75: IC32.12, R120.3
- removed net N$76: IC32.11, R120.4
- removed net N$77: IC33.10, IC36.24
- removed net N$78: IC33.8, IC36.2
- removed net N$79: IC33.7, IC36.3
- removed net N$80: IC33.6, IC36.4
- removed net N$81: IC33.5, IC36.5
- removed net N$82: IC33.4, IC36.6
- removed net N$83: IC33.3, IC36.7
- removed net N$84: IC33.18, R121.1
- removed net N$85: IC33.17, R121.2
- removed net N$86: IC33.16, R121.3
- removed net N$87: IC33.15, R121.4
- removed net N$88: IC33.14, R122.1
- removed net N$89: IC33.13, R122.2
- removed net N$90: IC33.12, R122.3
- removed net N$91: IC33.11, R122.4
- removed net N$92: IC34.10, IC37.15
- removed net N$93: IC34.9, IC37.16
- removed net N$94: IC34.8, IC37.17
- removed net N$95: IC34.7, IC37.18
- removed net N$96: IC34.6, IC37.19
- removed net N$97: IC34.5, IC37.20
- removed net N$98: IC34.4, IC37.21
- removed net N$99: IC34.3, IC37.22
- removed net PGA_A_IN+: IC7.1, R43.1
- removed net PGA_A_IN-: IC7.2, IC7.3, R44.2
- removed net PGA_B_IN+: IC9.1, R24.1
- removed net PGA_B_IN-: IC9.2, IC9.3, R42.2
- removed net REFBY2: C71.1, IC10.3, REFBY2.TP
- removed net REFM_A: C70.2, IC10.32
- removed net REFM_B: C110.2, IC10.9
- removed net REFOUT: C111.1, IC10.5, REFOUT.TP
- removed net REFP_A: C70.1, IC10.31
- removed net REFP_B: C110.1, IC10.10
- removed net SPI0_CS0: DIO_CS.TP, IC36.9, R29.1
- removed net SPI0_CS1: IC37.9, R30.1
- removed net SPI0_MISO: IC36.12, IC37.12, R27.1
- removed net SPI0_MOSI: IC22.15, IC36.11, IC37.11, R28.1
- removed net SPI0_SCK: IC22.16, IC36.10, IC37.10, R26.1
- removed net SPI1_CS0: IC10.14, R15.1, R32.1, SPI1_CS0.TP
- removed net SPI1_CS1: IC7.11, R33.1
- removed net SPI1_CS2: IC9.11, R34.1
- removed net SPI1_MISO: IC16.2, IC16.6, IC7.8, IC9.8, R18.1
- removed net SPI1_MOSI: IC10.15, IC7.9, IC9.9, R17.1
- removed net SPI1_SCK: IC10.16, IC7.10, IC9.10, R25.1
- removed net VFB_12VN: C106.2, IC15.7, R56.1, R76.1, VFB12VN.TP
- removed net VFB_12VP: C107.1, IC15.9, R55.1, R73.1, VFB12VP.TP
- removed net VFB_14VN: C101.2, IC14.16, R54.1, R59.1, TP_VFB_14VN.TP
- removed net VFB_14VP: C100.2, IC14.22, R53.1, R57.1, TP_VFB_14VP.TP
- removed net VOCM_A: IC7.21, R51.2, VOCMA.TP
- removed net VOCM_B: IC9.21, R52.1, VCOMB.TP
- removed net VREF_ADC: C46.1, C72.1, C73.1, IC13.1, IC13.4, IC7.23, IC9.23, R49.3, TP9.TP
- removed net VREF_ADC/2: C75.1, IC11.1, IC11.4, R51.1, R52.2, REF/2.TP
- removed net VREF_ADC_RAW: C48.1, IC12.2, IC13.3, VREFR.TP
- removed net VREF_DAC: C125.1, IC23.1, IC23.4, R100.1, R104.1, R108.1, R112.1, R116.1, R88.1, R92.1, R96.1
- removed net VREF_DAC_OUT: C124.1, IC22.8, IC23.3, VREF_DAC.TP
- removed net VREF_TPS: C99.2, IC14.17, R58.1, TP_VREF_TPS.TP
- removed net V_OUT_REF: C153.1, C154.1, C157.1, C158.1, C161.1, C162.1, C165.1, C166.1, DIO_VREF.TP, IC38.2, IC38.6, R127.2, R128.2, R129.2, R130.2
- new net RP2040_RST0: CON3.23, X1.B18
- new net RP2040_RST1: CON3.21, X3.B18
- new net SDO_A_1: CON2.13, X1.A18
- new net SDO_A_2: CON2.11, X1.A19
- new net SDO_A_3: CON2.9, X1.A20
- new net SDO_B_1: CON2.5, X1.A22
- new net SDO_B_2: CON2.3, X1.A23
- new net SDO_B_3: CON2.1, X1.A24
- new net SPI_ADC_CS: CON2.39, X1.A2
- new net SPI_AIOMODULE_CS0: CON3.5, X1.A29, X1.B29
- new net SPI_AIOMODULE_MISO: CON3.11, X1.A26, X1.B26
- new net SPI_AIOMODULE_MOSI: CON3.9, X1.A27, X1.B27
- new net SPI_AIOMODULE_SCK: CON3.7, X1.A28, X1.B28
- new net SPI_DAC_CS: CON2.21, X1.B2
- new net SPI_DIOMODULE_CS1: CON3.3, X3.A29, X3.B29
- new net SPI_DIOMODULE_MISO: X3.A26, X3.B26
- new net SPI_DIOMODULE_MOSI: X3.A27, X3.B27
- new net SPI_DIOMODULE_SCK: X3.A28, X3.B28
- new net SPI_DIO_CS0: CON3.33, X3.A2
- new net SPI_DIO_CS1: CON3.31, X3.A3
- new net SPI_MISO: CON2.29, X1.A7, X1.B7, X3.A7, X3.B7
- new net SPI_MOSI: CON2.31, X1.A6, X1.B6, X3.A6, X3.B6
- new net SPI_PGA_CS0: CON2.37, X1.A3
- new net SPI_PGA_CS1: CON2.35, X1.A4
- new net SPI_SCK: CON2.33, X1.A5, X1.B5, X3.A5, X3.B5
- new net SWCLK: CON3.15, X1.B23, X3.B23
- new net SWDIO: CON3.13, X1.B24, X3.B24
- new net UART0_RX: CON3.19, X1.B20, X3.B20
- new net UART0_TX: CON3.17, X1.B21, X3.B21
- net !ADC_RST: now also CON2.25, X1.A12; no longer IC10.26, R16.2, R38.1
- net +1V8: now also PI1.87, PI1.89; no longer J2.88, J2.90
- net +3V3: now also PI1.83, PI1.85, X1.A1, X1.B1, X3.A1, X3.B1; no longer C122.1, C123.1, C126.1, C128.1, C131.1, C134.1, C137.1, C140.1, C143.1, C146.1, C149.1, C151.1, C152.1, C155.1, C156.1, C159.1, C160.1, C163.1, C164.1, C167.1, C168.1, C169.1, C170.1, C171.1, C21.1, C22.1, C25.1, C45.1, C47.1, C49.1, C50.1, C51.1, C64.1, C65.1, C76.1, IC10.12, IC10.28, IC10.29, IC11.2, IC12.1, IC13.2, IC16.8, IC17.5, IC22.3, IC23.2, IC24.2, IC25.2, IC26.2, IC27.2, IC28.2, IC29.2, IC30.2, IC31.2, IC32.2, IC33.2, IC34.2, IC35.2, IC36.8, IC37.8, IC38.1, IC38.8, IC39.5, IC7.7, IC9.7, J2.84, J2.86, R16.1, R86.5, R86.6, R86.7, R86.8, TP_3V3.TP
- net +5V: now also C21.1, CON3.1, CON3.2, FAN.4, PI1.78, PI1.80, PI1.82, PI1.84, PI1.86, PI1.88, X1.A8, X1.A9, X1.B8, X1.B9, X3.A8, X3.A9, X3.B8, X3.B9; no longer C120.1, C26.1, C85.1, CON1.4, IC14.5, IC14.6, IC18.3, IC38.5, J2.77, J2.79, J2.81, J2.83, J2.85, J2.87, J7.18, J7.33, R14.2, T2.2
- net ADC_RDY: now also CON2.27, X1.A11; no longer IC10.25, R36.1
- net BT_NDIS: now also PI1.92; no longer J2.91
- net CAM_GPIO0: now also PI1.98; no longer J2.97
- net CAM_GPIO1: now also PI1.99; no longer J2.100
- net CC1: now also PI1.93; no longer J2.94
- net CC2: now also PI1.95; no longer J2.96
- net DAC_!CLR: now also CON2.17, X1.B13; no longer CLR.TP, IC22.9, R37.1, R86.4
- net DAC_!LDAC: now also CON2.19, X1.B12; no longer IC22.1, LDAC.TP, R35.1, R86.2
- net DIO_EN: now also CON3.29, X3.A11; no longer DIO_EN.TP, IC32.20, IC33.20, IC34.20, IC35.20, R41.1
- net DIO_LEVEL_SELECT: now also CON3.25, X3.A13; no longer DIO_LS.TP, IC38.7, IC39.2, R40.1
- net DIO_RESET: now also CON3.27, X3.A12; no longer DIO_RST.TP, IC36.13, IC37.13, R39.1
- net DPHY0_C_N: now also PI1.128; no longer J1.27
- net DPHY0_C_P: now also PI1.130; no longer J1.29
- net DPHY0_D0_N: now also PI1.116; no longer J1.15
- net DPHY0_D0_P: now also PI1.118; no longer J1.17
- net DPHY0_D1_N: now also PI1.122; no longer J1.21
- net DPHY0_D1_P: now also PI1.124; no longer J1.23
- net DPHY0_D2_N: now also PI1.134; no longer J1.33
- net DPHY0_D2_P: now also PI1.136; no longer J1.35
- net DPHY0_D3_N: now also PI1.140; no longer J1.39
- net DPHY0_D3_P: now also PI1.142; no longer J1.41
- net DPHY1_C_N: now also PI1.188; no longer J1.87
- net DPHY1_C_P: now also PI1.190; no longer J1.89
- net DPHY1_D0_N: now also PI1.176; no longer J1.75
- net DPHY1_D0_P: now also PI1.178; no longer J1.77
- net DPHY1_D1_N: now also PI1.182; no longer J1.81
- net DPHY1_D1_P: now also PI1.184; no longer J1.83
- net DPHY1_D2_N: now also PI1.194; no longer J1.93
- net DPHY1_D2_P: now also PI1.196; no longer J1.95
- net DPHY1_D3_N: now also PI1.193; no longer J1.94
- net DPHY1_D3_P: now also PI1.195; no longer J1.96
- net EEPROM_NWP: now also PI1.19; no longer J2.20
- net ETH_LEDG: now also PI1.18; no longer J2.17
- net ETH_LEDY: now also PI1.16; no longer J2.15
- net GND: now also FAN.2, J1.4, J1.S1, J1.S2, J2.4, J2.S1, J2.S2, J4.25, J4.26, PI1.1, PI1.107, PI1.108, PI1.113, PI1.114, PI1.119, PI1.120, PI1.125, PI1.126, PI1.13, PI1.131, PI1.132, PI1.137, PI1.138, PI1.14, PI1.143, PI1.149, PI1.155, PI1.156, PI1.161, PI1.162, PI1.167, PI1.168, PI1.173, PI1.174, PI1.179, PI1.180, PI1.185, PI1.186, PI1.191, PI1.192, PI1.197, PI1.198, PI1.2, PI1.21, PI1.24, PI1.31, PI1.34, PI1.41, PI1.44, PI1.51, PI1.54, PI1.59, PI1.60, PI1.65, PI1.66, PI1.7, PI1.72, PI1.73, PI1.8, PI1.97, X1.A10, X1.A14, X1.A15, X1.A16, X1.A25, X1.A30, X1.A31, X1.A32, X1.B10, X1.B14, X1.B15, X1.B16, X1.B19, X1.B22, X1.B25, X1.B30, X1.B31, X1.B32, X3.A10, X3.A14, X3.A15, X3.A16, X3.A25, X3.A30, X3.A31, X3.A32, X3.B10, X3.B14, X3.B15, X3.B16, X3.B19, X3.B22, X3.B25, X3.B30, X3.B31, X3.B32; no longer BT1.N, C102.2, C103.2, C104.2, C105.1, C108.2, C109.2, C111.2, C120.2, C121.2, C122.2, C123.2, C124.2, C125.2, C126.2, C127.2, C128.2, C130.2, C131.2, C133.2, C134.2, C136.2, C137.2, C139.2, C140.2, C142.2, C143.2, C145.2, C146.2, C148.2, C149.2, C151.2, C152.2, C153.2, C154.2, C155.2, C156.2, C157.2, C158.2, C159.2, C160.2, C161.2, C162.2, C163.2, C164.2, C165.2, C166.2, C167.2, C168.2, C169.2, C170.2, C171.2, C22.2, C23.2, C24.1, C25.2, C26.2, C27.2, C42.2, C43.1, C45.2, C46.2, C47.2, C48.2, C49.2, C50.2, C51.2, C52.2, C53.2, C54.2, C55.2, C56.2, C57.2, C58.2, C59.2, C60.2, C61.2, C62.2, C63.2, C64.2, C65.2, C66.2, C67.2, C68.2, C69.2, C71.2, C74.2, C75.2, C76.2, C85.2, C86.2, C90.2, C91.2, C92.2, C93.2, C94.2, C95.2, C96.2, C97.2, C98.2, C99.1, CON1.2, DIO_GND.TP, IC10.11, IC10.27, IC10.30, IC10.33, IC10.4, IC11.5, IC12.3, IC13.5, IC14.19, IC14.2, IC14.25, IC14.3, IC15.4, IC15.PAD, IC15.PAD1, IC15.PAD2, IC15.PAD3, IC15.PAD4, IC16.4, IC17.3, IC18.1, IC22.14, IC23.5, IC24.5, IC25.5, IC26.5, IC27.5, IC28.5, IC29.5, IC30.5, IC31.5, IC32.1, IC32.PAD, IC33.1, IC33.PAD, IC34.1, IC34.PAD, IC35.1, IC35.PAD, IC36.23, IC36.25, IC37.23, IC37.25, IC38.4, IC39.3, IC6.15, IC7.22, IC7.24, IC7.25, IC7.4, IC7.6, IC8.15, IC9.22, IC9.24, IC9.25, IC9.4, IC9.6, J1.13, J1.14, J1.19, J1.20, J1.25, J1.26, J1.31, J1.32, J1.37, J1.38, J1.44, J1.50, J1.55, J1.56, J1.61, J1.62, J1.67, J1.68, J1.73, J1.74, J1.79, J1.8, J1.80, J1.85, J1.86, J1.91, J1.92, J1.97, J1.98, J2.1, J2.13, J2.14, J2.2, J2.22, J2.23, J2.32, J2.33, J2.42, J2.43, J2.52, J2.53, J2.59, J2.60, J2.65, J2.66, J2.71, J2.74, J2.8, J2.98, J7.1, J7.23, J7.28, J7.34, J7.35, J7.57, J7.62, J7.68, J7.MH1, J7.MH2, L4.1, R103.1, R107.1, R111.1, R115.1, R57.2, R73.2, R87.1, R91.1, R95.1, R99.1, TP_GND.TP, USB3.13, USB3.16, USB3.4, USB3.7, USB3.S1, USB3.S2, USB3.S3, USB3.S4
- net GPIO10: now also CON3.10, PI1.43; no longer J2.44, R28.2
- net GPIO11: now also CON3.8, PI1.37; no longer J2.38, R26.2
- net GPIO12: now also CON2.18, PI1.32; no longer J2.31
- net GPIO13: now also CON2.24, PI1.27; no longer J2.28, R40.2
- net GPIO14: now also CON3.18, PI1.56; no longer J2.55
- net GPIO15: now also CON3.20, PI1.52; no longer J2.51
- net GPIO16: now also CON2.36, PI1.30; no longer J2.29, R34.2
- net GPIO17: now also CON2.38, PI1.49; no longer J2.50, R33.2
- net GPIO18: now also CON2.40, PI1.50; no longer J2.49, R32.2
- net GPIO19: now also CON2.30, PI1.25; no longer J2.26, R18.2
- net GPIO2: now also CON3.24, PI1.57; no longer J2.58
- net GPIO20: now also CON2.32, PI1.28; no longer J2.27, R17.2
- net GPIO21: now also CON2.34, PI1.26; no longer J2.25, R25.2
- net GPIO22: now also CON3.32, PI1.45; no longer J2.46
- net GPIO23: now also PI1.48; no longer J2.47, R31.2
- net GPIO24: now also CON3.14, PI1.46; no longer J2.45, R36.2
- net GPIO25: now also CON3.16, PI1.42; no longer J2.41, R38.2
- net GPIO26: now also CON2.20, PI1.23; no longer J2.24
- net GPIO27: now also CON3.34, PI1.47; no longer J2.48, R35.2
- net GPIO3: now also CON3.22, PI1.55; no longer J2.56
- net GPIO4: now also CON2.28, PI1.53; no longer J2.54, R37.2
- net GPIO5: now also CON2.22, PI1.33; no longer J2.34, R41.2
- net GPIO6: now also CON2.26, CON3.30, PI1.29; no longer J2.30, R39.2
- net GPIO7: now also CON3.4, PI1.38; no longer J2.37, R30.2
- net GPIO8: now also CON3.6, PI1.40; no longer J2.39, R29.2
- net GPIO9: now also CON3.12, PI1.39; no longer J2.40, R27.2
- net GPIO_VREF: now also PI1.77; no longer J2.78
- net HDMI0_CEC: now also PI1.152; no longer J1.51
- net HDMI0_CK_N: now also PI1.189; no longer J1.90
- net HDMI0_CK_P: now also PI1.187; no longer J1.88
- net HDMI0_D0_N: now also PI1.183; no longer J1.84
- net HDMI0_D0_P: now also PI1.181; no longer J1.82
- net HDMI0_D1_N: now also PI1.177; no longer J1.78
- net HDMI0_D1_P: now also PI1.175; no longer J1.76
- net HDMI0_D2_N: now also PI1.171; no longer J1.72
- net HDMI0_D2_P: now also PI1.169; no longer J1.70
- net HDMI0_HOTPLUG: now also PI1.154; no longer J1.53
- net HDMI0_SCL: now also PI1.199; no longer J1.100
- net HDMI0_SDA: now also PI1.200; no longer J1.99
- net HDMI1_CEC: now also PI1.150; no longer J1.49
- net HDMI1_CK_N: now also PI1.165; no longer J1.66
- net HDMI1_CK_P: now also PI1.163; no longer J1.64
- net HDMI1_D0_N: now also PI1.159; no longer J1.60
- net HDMI1_D0_P: now also PI1.157; no longer J1.58
- net HDMI1_D1_N: now also PI1.153; no longer J1.54
- net HDMI1_D1_P: now also PI1.151; no longer J1.52
- net HDMI1_D2_N: now also PI1.147; no longer J1.48
- net HDMI1_D2_P: now also PI1.145; no longer J1.46
- net HDMI1_HOTPLUG: now also PI1.144; no longer J1.43
- net HDMI1_SCL: now also PI1.148; no longer J1.47
- net HDMI1_SDA: now also PI1.146; no longer J1.45
- net ID_SC: now also ID.1, PI1.36; no longer J2.35, JP1.1
- net ID_SD: now also ID.3, PI1.35; no longer J2.36, JP1.3
- net LED_NACT: now also PI1.22; no longer J2.21
- net MISO_SEL: now also CON2.23, X1.A13; no longer IC16.7, IC17.2
- net NPWR_LED: now also PI1.96; no longer J2.95
- net NRPIBOOT: now also PI1.94; no longer J2.93
- net PCIE_CLK_N: now also PI1.111; no longer J1.12
- net PCIE_CLK_P: now also PI1.109; no longer J1.10
- net PCIE_NCLKREQ: now also PI1.101; no longer J1.2
- net PCIE_NRST: now also PI1.110; no longer J1.9
- net PCIE_NWAKE: now also PI1.103; no longer J1.4
- net PCIE_PWR_EN: now also PI1.105; no longer J1.6
- net PCIE_RX_N: now also PI1.117; no longer J1.18
- net PCIE_RX_P: now also PI1.115; no longer J1.16
- net PCIE_TX_N: now also PI1.123; no longer J1.24
- net PCIE_TX_P: now also PI1.121; no longer J1.22
- net PMIC_ENABLE: now also PI1.100; no longer J2.99
- net PWM: now also FAN.3, PI1.20; no longer CON1.3, J2.19
- net PWR_BUT: now also PI1.91; no longer J2.92
- net SCL0: now also PI1.79; no longer J2.80
- net SCL1: now also ID.2; no longer JP1.2
- net SDA0: now also PI1.81; no longer J2.82
- net SDA1: now also ID.4; no longer JP1.4
- net SDO_A_0: now also CON2.15, X1.A17; no longer IC10.24, IC16.1
- net SDO_B_0: now also CON2.7, X1.A21; no longer IC10.20, IC16.5
- net SD_CLK: now also PI1.58; no longer J2.57
- net SD_CMD: now also PI1.61; no longer J2.62
- net SD_DAT0: now also PI1.64; no longer J2.63
- net SD_DAT1: now also PI1.68; no longer J2.67
- net SD_DAT2: now also PI1.70; no longer J2.69
- net SD_DAT3: now also PI1.62; no longer J2.61
- net SD_PWR_ON: now also PI1.76; no longer J2.75
- net SYNC_OUT: now also PI1.17; no longer J2.18
- net TACHO: now also FAN.1, PI1.15; no longer CON1.1, J2.16
- net TR0_TAP: now also POE.3; no longer JP4.3
- net TR1_TAP: now also POE.1; no longer JP4.1
- net TR2_TAP: now also POE.2; no longer JP4.2
- net TR3_TAP: now also POE.4; no longer JP4.4
- net TRD0_N: now also PI1.9; no longer J2.10
- net TRD0_P: now also PI1.11; no longer J2.12
- net TRD1_N: now also PI1.5; no longer J2.6
- net TRD1_P: now also PI1.3; no longer J2.4
- net TRD2_N: now also PI1.10; no longer J2.9
- net TRD2_P: now also PI1.12; no longer J2.11
- net TRD3_N: now also PI1.6; no longer J2.5
- net TRD3_P: now also PI1.4; no longer J2.3
- net USB2_N: now also PI1.104; no longer J1.3
- net USB2_P: now also PI1.106; no longer J1.5
- net USB3-0-D_N: now also J1.2, PI1.135; no longer J1.36, USB3.2
- net USB3-0-D_P: now also J1.3, PI1.133; no longer J1.34, USB3.3
- net USB3-0-RX_N: now also J1.5, PI1.127; no longer J1.28, USB3.5
- net USB3-0-RX_P: now also J1.6, PI1.129; no longer J1.30, USB3.6
- net USB3-0-TX_N: now also J1.8, PI1.139; no longer J1.40, USB3.8
- net USB3-0-TX_P: now also J1.9, PI1.141; no longer J1.42, USB3.9
- net USB3-1-D_N: now also J2.2, PI1.166; no longer J1.65, USB3.11
- net USB3-1-D_P: now also J2.3, PI1.164; no longer J1.63, USB3.12
- net USB3-1-RX_N: now also J2.5, PI1.158; no longer J1.57, USB3.14
- net USB3-1-RX_P: now also J2.6, PI1.160; no longer J1.59, USB3.15
- net USB3-1-TX_N: now also J2.8, PI1.170; no longer J1.69, USB3.17
- net USB3-1-TX_P: now also J2.9, PI1.172; no longer J1.71, USB3.18
- net USBOTG_ID: now also PI1.102; no longer J1.1
- net VBAT: now also PI1.75; no longer BT1.P1, BT1.P2, J2.76, TP-VBAT.TP
- net VBUS: now also J1.1, J2.1; no longer USB3.1, USB3.10
- net VBUS_EN: now also PI1.112; no longer J1.11
- net WL_NDIS: now also PI1.90; no longer J2.89
Routing:
- net GND: track 2181.6 -> 582.8 mm, vias 288 -> 60
- net +3V3: track 793.3 -> 408.4 mm, vias 37 -> 6
- net +5V: track 777.7 -> 589.2 mm, vias 34 -> 43
- net +14V: track 171.8 -> 0.00 mm
- net VBAT: track 169.2 -> 0.00 mm, vias 1 -> 0
- net -14V: track 148.0 -> 0.00 mm
- net -12V: track 136.5 -> 0.00 mm, vias 9 -> 0
- net +12V: track 135.8 -> 0.00 mm, vias 7 -> 0
- net SPI1_CS1: track 125.9 -> 0.00 mm, vias 4 -> 0
- net DIO_31: track 114.6 -> 0.00 mm, vias 1 -> 0
- net VREF_ADC: track 111.3 -> 0.00 mm, vias 4 -> 0
- net DIO_30: track 111.1 -> 0.00 mm, vias 1 -> 0
- net DIO_29: track 110.1 -> 0.00 mm, vias 1 -> 0
- net SPI1_MISO: track 107.2 -> 0.00 mm, vias 8 -> 0
- net DIO_28: track 104.4 -> 0.00 mm, vias 1 -> 0
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- added copper zone on layer 1, net +5V
- added copper zone on layer 1, net M2_3V3
- added copper zone on layer 1, net N$10
- added copper zone on layer 1, net N$9
- added copper zone on layer 1, net VBUS
Other:
- board size 180 x 100 mm -> 195.6 x 114 mm
- board text added: "+5V"
- board text added: "ADC_RDY"
- board text added: "ADC_RST"
- board text added: "CS_ADC"
- board text added: "CS_DAC"
- board text added: "CS_PGA0"
- board text added: "CS_PGA1"
- board text added: "DAC_CLR"
- board text added: "DAC_LDAC"
- board text added: "DIO_EN"
- board text added: "DIO_LS"
- board text added: "DIO_RES"
- board text added: "DISABLE BT"
- board text added: "DISABLE WiFi"
- board text added: "EEPROM WP"
- board text added: "GND"
- board text added: "GPIO10"
- board text added: "GPIO11"
- board text added: "GPIO12"
- board text added: "GPIO13"
- board text added: "GPIO14"
- board text added: "GPIO15"
- board text added: "GPIO16"
- board text added: "GPIO17"
- board text added: "GPIO18"
- board text added: "GPIO19"
- board text added: "GPIO2"
- board text added: "GPIO20"
- board text added: "GPIO21"
- board text added: "GPIO22"
- board text added: "GPIO24"
- board text added: "GPIO25"
- board text added: "GPIO26"
- board text added: "GPIO27"
- board text added: "GPIO3"
- board text added: "GPIO5"
- board text added: "GPIO6"
- board text added: "GPIO7"
- board text added: "GPIO8"
- board text added: "GPIO9"
- board text added: "MISO_SEL"
- board text added: "Module - Baseboard, Rev 1.0"
- board text added: "NC"
- board text added: "NRPBOOT"
- board text added: "PMIC ENABLE"
- board text added: "PWM"
- board text added: "PWR BUTTON"
- board text added: "RP_RES0"
- board text added: "RP_RES1"
- board text added: "SD0_A0"
- board text added: "SD0_A1"
- board text added: "SD0_A2"
- board text added: "SD0_A3"
- board text added: "SD0_B0"
- board text added: "SD0_B1"
- board text added: "SD0_B2"
- board text added: "SD0_B3"
- board text added: "SN-192776090225"
- board text added: "SPI_CS0"
- board text added: "SPI_CS1"
- board text added: "SPI_MISO"
- board text added: "SPI_MOSI"
- board text added: "SPI_SCK"
- board text added: "SWCLK"
- board text added: "SWDIO"
- board text added: "SYNC OUT"
- board text added: "TACHO"
- board text added: "UART_RX"
- board text added: "UART_TX"
- board text added: "USBOTG"
- board text added: "XSPI_CS0"
- board text added: "XSPI_CS1"
- board text added: "XSPI_MI"
- board text added: "XSPI_MO"
- board text added: "XSPI_SCK"
- board text added: "github.com/DvidMakesThings/HW_10-In-Rack_DAQ"
- board text removed: "BT_DIS WL_DIS"
- board text removed: "DataForge-PI"
- board text removed: "DataForge-Pi Rev 1.0"
- board text removed: "David Sipos - 2025 Wien"
- board text removed: "ID_SD ID_SC"
- board text removed: "PWRBU PMICEN OTG SYNC EEWP NRBT"
