File: src/HardwareDesign/Dataforge-Pi.sch (EAGLE design)
At the start: 364 parts, among them IC1 RT9742GGJ, IC10 ADS9234RIRHBR, IC11 MCP6001RT, IC12 MCP1525T-I/TT, IC13 MCP6001RT, IC14 TPS65131, IC15 TPS7A39, IC16 SN74LVC2G66, IC17 74LVC1G04, IC2 AP22653W6, IC22 DAC8568, IC23 MCP6001RT, IC24 MCP6001RT, IC25 MCP6001RT, IC26 MCP6001RT, IC27 MCP6001RT, IC28 MCP6001RT, IC29 MCP6001RT, IC3 74LVC1G07, IC30 MCP6001RT, IC31 MCP6001RT, IC32 LSF0108, IC33 LSF0108, IC34 LSF0108, IC35 LSF0108, IC36 MCP23S18, IC38 SN74LVC2G66, IC39 74LVC1G04, IC4 RT9742NGV, IC5 AP3441SHE-7B, IC6 DG409, IC7 ADA4254ACPZ, IC8 DG409, IC9 ADA4254ACPZ, J1 10164227-1001A1RLF, J2 10164227-1001A1RLF, J3 FH12-22S-0.5SVA, J4 FH12-22S-0.5SH(55), J7 2-5174225-5, SW1 1825027-8, T2 IRLML5203, X2 CRYSTAL

Commit message: Baseboard design ready
Parts:
- removed 12VN, 12VP, 14VN, 14VP, BUF, CLR, DIO_CS, DIO_EN, DIO_GND, DIO_LS, DIO_RST, DIO_VREF, LDAC, REF/2, REFBY2, REFOUT, SPI1_CS0, SYNC, TP-VBAT, TP9, TPD0, TP_3V3, TP_BSW_G, TP_GND, TP_VFB_14VN, TP_VFB_14VP, TP_VREF_TPS, VCOMB, VFB12VN, VFB12VP, VOCMA, VREFR, VREF_DAC: TP, ds_passive:TP
- removed BT1: 79523141, Battery Holder:79523141
- removed C100, C101: 10pF, ds_passive:C0402
- removed C102, C104: 10uF, ds_passive:C1206
- removed C103, C106, C107: 10nF, ds_passive:C0402
- removed C105, C99: 220nF, ds_passive:C0402
- removed C108, C109, C93, C94, C95, C96, C97, C98: 22uF, ds_passive:C1206
- removed C110, C70: 10uF, ds_passive:C0603
- removed C111, C120, C121, C125, C126, C128, C129, C131, C132, C134, C135, C137, C138, C140, C141, C143, C144, C146, C147, C149, C150, C152, C154, C156, C158, C160, C162, C164, C166, C168, C170, C22, C25, C45, C46, C49, C51, C53, C55, C57, C59, C61, C63, C65, C67, C69, C71, C75, C76: 100nF, ds_passive:C0402
- removed C122, C124, C50, C52, C54, C56, C58, C60, C62, C64, C66, C68, C72: 1uF, ds_passive:C0603
- removed C123, C171, C73: 100nF, ds_passive:C0603
- removed C127, C130, C133, C136, C139, C142, C145, C148: 20nF, ds_passive:C0402
- removed C151, C153, C155, C157, C159, C161, C163, C165, C167, C169: 1uF, ds_passive:C0402
- removed C23, C24, C42, C43: 270pF, ds_passive:C0402
- removed C26, C27: 100uF 16V, ds_passive:CPOL
- removed C41, C44: 680pF, ds_passive:C0402
- removed C47, C90: 10uF, ds_passive:C0805
- removed C48, C74: (no value), ds_passive:C0805
- removed C85: 4.7uF, ds_passive:C0805
- removed C86: 100nF, ds_passive:C0805
- removed C91: 10nF, ds_passive:C0805
- removed C92: 4.7nF, ds_passive:C0805
- removed D3, D4: SS12, Diodes:SS12
- removed IC10: ADS9234RIRHBR, ds_ic_peripherals:ADS9234RIRHBR
- removed IC11, IC13, IC23, IC24, IC25, IC26, IC27, IC28, IC29, IC30, IC31: MCP6001RT, ds_ic_opa:MCP6001RT
- removed IC12: MCP1525T-I/TT, ds_ic_vreg:MCP1525T-I/TT
- removed IC14: TPS65131, ds_ic_vreg:TPS65131TRGERQ1
- removed IC15: TPS7A39, ds_ic_vreg:TPS7A3901DSCR
- removed IC16, IC38: SN74LVC2G66, ds_ic_peripherals:SN74LVC2G66
- removed IC17, IC39: 74LVC1G04, ds_ic_logic:74LVC1G04
- removed IC18: (no value), ds_ic_vreg:LDL1117S33R
- removed IC22: DAC8568, ds_ic_peripherals:DAC8568
- removed IC32, IC33, IC34, IC35: LSF0108, ds_ic_peripherals:LSF0108-Q1
- removed IC36: MCP23S18, ds_ic_peripherals:MCP23S18
- removed IC37: (no value), ds_ic_peripherals:MCP23S18
- removed IC6, IC8: DG409, ds_ic_peripherals:DG409EUE+
- removed IC7, IC9: ADA4254ACPZ, ds_ic_opa:ADA4254ACPZ
- removed J7: 2-5174225-5, Connector_D-Sub:2-5174225-5
- removed L3, L4: SRR5228A-4R7Y, ds_passive:L
- removed R100, R103, R104, R107, R108, R111, R112, R115, R116, R73, R76, R87, R88, R91, R92, R95, R96, R99: 10K 0.1%, ds_passive:R0402
- removed R101, R105, R109, R113, R117, R89, R93, R97: 43K 0.1%, ds_passive:R0402
- removed R102, R106, R110, R114, R118, R90, R94, R98: 68R 1%, ds_passive:R0402
- removed R119, R120, R121, R122, R123, R124, R125, R126: YC164-JR-0733RL, Resistor Array:YC164-JR-0733RL
- removed R127, R128, R129, R130: 200K, ds_passive:R0402
- removed R14: 100R, ds_passive:R1206
- removed R15, R24, R42, R43, R44, R45, R46, R47, R48: 0R, ds_passive:R0402
- removed R16: 10K, ds_passive:R0402
- removed R17, R18, R25, R26, R27, R28, R29, R30, R31, R32, R33, R34, R35, R36, R37, R38, R39, R40, R41, R51, R52: 0R, ds_passive:R0603
- removed R19: 950K 0.1%, ds_passive:R0402
- removed R20, R21, R22, R23: 200R, ds_passive:R0402
- removed R49, R53, R54, R55, R56: (no value), ds_passive:R-TRIM
- removed R50: 100R, ds_passive:R0402
- removed R57: 102K 0.1%, ds_passive:R0402
- removed R58: 1.2M 0.1%, ds_passive:R0402
- removed R59: 137K 0.1%, ds_passive:R0402
- removed R60: 75K 0.1%, ds_passive:R0402
- removed R74: 90K 0.1%, ds_passive:R0402
- removed R86: CRA034RF100RP05Z, Resistor Array:YC164-JR-0733RL
- removed T2: IRLML5203, transistor-power:IRLML5203
- removed USB3: 692141030100, Wurth_Connectors_WR-USB:692141030100
- added CON2, CON3: (no value), ds_con:CON-2X20
- added PI1: (no value), ds_ic_peripherals:RASPBERRY_CM5
- added X1, X3: CON-VG_MAB642, ds_con:CON-VG_MAB642
- C21: value 100nF -> 100uF 16V; device ds_passive:C0603 -> ds_passive:CPOL
- J1, J2: value 10164227-1001A1RLF -> 692121030100; device ds_con:10164227-1001A1RLF -> Wurth_Connectors_WR-USB:692121030100
- J4: value FH12-22S-0.5SH(55) -> FH12-22S-0.5SVA; device ds_con:FH12-22S-0.5SH(55) -> ds_con:FH12-22S-0.5SVA
- renumbered CON1 to FAN, JP1 to ID, JP4 to POE
Connections:
- removed net !DIO_LEVEL_SELECT: IC38.2C, IC39.OUT
- removed net !MISO_SEL: IC16.2C, IC17.OUT
- removed net +12V: 12VP.P$1, C107.2, C108.1, C52.1, C53.1, C56.1, C57.1, C60.1, C61.1, C66.1, C67.1, IC15.OUTP, IC6.V+, IC7.VDDH, IC8.V+, IC9.VDDH, R60.1
- removed net +14V: 14VP.P$1, C100.1, C104.1, C93.1, C94.1, C95.1, D3.C, IC14.VPOS, IC15.EN, IC15.INP, R19.1
- removed net +3V3_EXT: C121.1, C27.1, IC18.VOUT, J7.52, J7.67
- removed net -12V: 12VN.P$1, C106.1, C109.1, C54.1, C55.1, C58.1, C59.1, C62.1, C63.1, C68.1, C69.1, IC15.OUTN, IC6.V-, IC7.PAD, IC7.VSSH, IC8.V-, IC9.PAD, IC9.VSSH, R76.2
- removed net -14V: 14VN.P$1, C101.1, C102.1, C96.1, C97.1, C98.1, D4.A, IC14.VNEG, IC15.INN, R59.2
- removed net ADA_A_IO0: IC6.A0, IC7.GPIO0
- removed net ADA_A_IO1: IC6.A1, IC7.GPIO1
- removed net ADA_A_IO2: IC6.EN, IC7.GPIO2
- removed net ADA_B_IO0: IC8.A0, IC9.GPIO0
- removed net ADA_B_IO1: IC8.A1, IC9.GPIO1
- removed net ADA_B_IO2: IC8.EN, IC9.GPIO2
- removed net ADC_AIN_N: C24.2, C41.2, R21.1, R46.1
- removed net ADC_AIN_P: C23.1, C41.1, R20.1, R45.2
- removed net ADC_BIN_N: C43.2, C44.2, R23.1, R48.2
- removed net ADC_BIN_P: C42.1, C44.1, R22.1, R47.1
- removed net ADC_IN0: IC10.AINP_A, R45.1
- removed net ADC_IN1: IC10.AINM_A, R46.2
- removed net ADC_IN2: IC10.AINP_B, R48.1
- removed net ADC_IN3: IC10.AINM_B, R47.2
- removed net AO_0: C127.1, J7.29, R89.2, R90.2
- removed net AO_1: C130.1, J7.63, R93.2, R94.2
- removed net AO_2: C133.1, J7.30, R97.2, R98.2
- removed net AO_3: C136.1, J7.64, R101.2, R102.2
- removed net AO_4: C139.1, J7.31, R105.2, R106.2
- removed net AO_5: C142.1, J7.65, R109.2, R110.2
- removed net AO_6: C145.1, J7.32, R113.2, R114.2
- removed net AO_7: C148.1, J7.66, R117.2, R118.2
- removed net BSW_G: IC14.BSW, T2.G, TP_BSW_G.P$1
- removed net BUF: BUF.P$1, C105.2, IC15.BUF, R74.1
- removed net DAC_!SYNC: IC22.!SYNC, R31.1, R86.3, SYNC.P$1
- removed net DAC_0: IC22.VOUT_A, IC24.+IN, TPD0.P$1
- removed net DAC_1: IC22.VOUT_B, IC25.+IN
- removed net DAC_2: IC22.VOUT_C, IC26.+IN
- removed net DAC_3: IC22.VOUT_D, IC27.+IN
- removed net DAC_4: IC22.VOUT_E, IC28.+IN
- removed net DAC_5: IC22.VOUT_F, IC29.+IN
- removed net DAC_6: IC22.VOUT_G, IC30.+IN
- removed net DAC_7: IC22.VOUT_H, IC31.+IN
- removed net DIO_0: J7.2, R120.5
- removed net DIO_1: J7.3, R120.6
- removed net DIO_10: J7.12, R122.7
- removed net DIO_11: J7.13, R122.8
- removed net DIO_12: J7.14, R121.5
- removed net DIO_13: J7.15, R121.6
- removed net DIO_14: J7.16, R121.7
- removed net DIO_15: J7.17, R121.8
- removed net DIO_16: J7.36, R124.5
- removed net DIO_17: J7.37, R124.6
- removed net DIO_18: J7.38, R124.7
- removed net DIO_19: J7.39, R124.8
- removed net DIO_2: J7.4, R120.7
- removed net DIO_20: J7.40, R123.5
- removed net DIO_21: J7.41, R123.6
- removed net DIO_22: J7.42, R123.7
- removed net DIO_23: J7.43, R123.8
- removed net DIO_24: J7.44, R126.5
- removed net DIO_25: J7.45, R126.6
- removed net DIO_26: J7.46, R126.7
- removed net DIO_27: J7.47, R126.8
- removed net DIO_28: J7.48, R125.5
- removed net DIO_29: J7.49, R125.6
- removed net DIO_3: J7.5, R120.8
- removed net DIO_30: J7.50, R125.7
- removed net DIO_31: J7.51, R125.8
- removed net DIO_4: J7.6, R119.5
- removed net DIO_5: J7.7, R119.6
- removed net DIO_6: J7.8, R119.7
- removed net DIO_7: J7.9, R119.8
- removed net DIO_8: J7.10, R122.5
- removed net DIO_9: J7.11, R122.6
- removed net IN0+: IC6.IN_A_0, J7.19
- removed net IN1-: IC6.IN_B_0, J7.53
- removed net IN10+: IC8.IN_A_1, J7.25
- removed net IN11-: IC8.IN_B_1, J7.59
- removed net IN12+: IC8.IN_A_2, J7.26
- removed net IN13-: IC8.IN_B_2, J7.60
- removed net IN14+: IC8.IN_A_3, J7.27
- removed net IN15-: IC8.IN_B_3, J7.61
- removed net IN2+: IC6.IN_A_1, J7.20
- removed net IN3-: IC6.IN_B_1, J7.54
- removed net IN4+: IC6.IN_A_2, J7.21
- removed net IN5-: IC6.IN_B_2, J7.55
- removed net IN6+: IC6.IN_A_3, J7.22
- removed net IN7-: IC6.IN_B_3, J7.56
- removed net IN8+: IC8.IN_A_0, J7.24
- removed net IN9-: IC8.IN_B_0, J7.58
- removed net MUX_A_OUTA: IC6.OUT_A, R43.2
- removed net MUX_A_OUTB: IC6.OUT_B, R44.1
- removed net MUX_B_OUTA: IC8.OUT_A, R24.2
- removed net MUX_B_OUTB: IC8.OUT_B, R42.1
- removed net N$100: IC34.B1, R123.1
- removed net N$101: IC34.B2, R123.2
- removed net N$102: IC34.B3, R123.3
- removed net N$103: IC34.B4, R123.4
- removed net N$104: IC34.B5, R124.1
- removed net N$105: IC34.B6, R124.2
- removed net N$106: IC34.B7, R124.3
- removed net N$107: IC34.B8, R124.4
- removed net N$108: IC35.A6, IC37.GPB2
- removed net N$109: IC35.A5, IC37.GPB3
- removed net N$110: IC35.A4, IC37.GPB4
- removed net N$111: IC35.A3, IC37.GPB5
- removed net N$112: IC35.A2, IC37.GPB6
- removed net N$113: IC35.A1, IC37.GPB7
- removed net N$114: IC35.A7, IC37.GPB1
- removed net N$115: IC35.A8, IC37.GPB0
- removed net N$116: IC35.B1, R125.1
- removed net N$117: IC35.B2, R125.2
- removed net N$118: IC35.B3, R125.3
- removed net N$119: IC35.B4, R125.4
- removed net N$12: IC7.OUT+, R20.2
- removed net N$120: IC35.B5, R126.1
- removed net N$121: IC35.B6, R126.2
- removed net N$122: IC35.B7, R126.3
- removed net N$123: IC35.B8, R126.4
- removed net N$124: IC32.VREF_B, R127.1
- removed net N$125: IC33.VREF_B, R128.1
- removed net N$126: IC35.VREF_B, R129.1
- removed net N$127: IC34.VREF_B, R130.1
- removed net N$13: IC7.OUT-, R21.2
- removed net N$14: C129.2, IC24.OUT, R90.1
- removed net N$15: IC9.OUT+, R22.2
- removed net N$16: IC9.OUT-, R23.2
- removed net N$17: C129.1, IC24.-IN, R87.2, R88.2, R89.1
- removed net N$18: IC10.CONVST, R15.2
- removed net N$19: C72.2, C73.2, R49.1
- removed net N$20: C74.1, R49.2, R50.1
- removed net N$21: IC11.+IN, R50.2
- removed net N$22: C132.1, IC25.-IN, R91.2, R92.2, R93.1
- removed net N$23: C132.2, IC25.OUT, R94.1
- removed net N$24: D3.A, IC14.INP, L3.2
- removed net N$25: C135.1, IC26.-IN, R95.2, R96.2, R97.1
- removed net N$26: C135.2, IC26.OUT, R98.1
- removed net N$27: C138.1, IC27.-IN, R100.2, R101.1, R99.2
- removed net N$28: C138.2, IC27.OUT, R102.1
- removed net N$29: IC33.A7, IC36.GPB1
- removed net N$30: C90.1, L3.1, T2.D
- removed net N$31: C141.1, IC28.-IN, R103.2, R104.2, R105.1
- removed net N$32: C86.1, IC14.ENN, IC14.ENP, IC14.PSN, IC14.PSP, IC14.VIN, R14.1
- removed net N$33: C141.2, IC28.OUT, R106.1
- removed net N$34: C144.1, IC29.-IN, R107.2, R108.2, R109.1
- removed net N$35: C91.1, IC14.CP
- removed net N$36: C92.1, IC14.CN
- removed net N$37: D4.C, IC14.OUTN, L4.2
- removed net N$38: R55.2, R55.3, R60.2
- removed net N$39: C103.1, IC15.NR/SS
- removed net N$40: C144.2, IC29.OUT, R110.1
- removed net N$41: C147.1, IC30.-IN, R111.2, R112.2, R113.1
- removed net N$42: R56.2, R56.3, R74.2
- removed net N$43: R19.2, R53.2, R53.3
- removed net N$44: R54.2, R54.3, R58.2
- removed net N$58: C147.2, IC30.OUT, R114.1
- removed net N$59: C150.1, IC31.-IN, R115.2, R116.2, R117.1
- removed net N$60: C150.2, IC31.OUT, R118.1
- removed net N$61: IC32.A8, IC36.GPA0
- removed net N$62: IC32.A7, IC36.GPA1
- removed net N$63: IC32.A6, IC36.GPA2
- removed net N$64: IC32.A5, IC36.GPA3
- removed net N$65: IC32.A4, IC36.GPA4
- removed net N$66: IC32.A3, IC36.GPA5
- removed net N$67: IC32.A2, IC36.GPA6
- removed net N$68: IC32.A1, IC36.GPA7
- removed net N$69: IC32.B1, R119.1
- removed net N$70: IC32.B2, R119.2
- removed net N$71: IC32.B3, R119.3
- removed net N$72: IC32.B4, R119.4
- removed net N$73: IC32.B5, R120.1
- removed net N$74: IC32.B6, R120.2
- removed net N$75: IC32.B7, R120.3
- removed net N$76: IC32.B8, R120.4
- removed net N$77: IC33.A8, IC36.GPB0
- removed net N$78: IC33.A6, IC36.GPB2
- removed net N$79: IC33.A5, IC36.GPB3
- removed net N$80: IC33.A4, IC36.GPB4
- removed net N$81: IC33.A3, IC36.GPB5
- removed net N$82: IC33.A2, IC36.GPB6
- removed net N$83: IC33.A1, IC36.GPB7
- removed net N$84: IC33.B1, R121.1
- removed net N$85: IC33.B2, R121.2
- removed net N$86: IC33.B3, R121.3
- removed net N$87: IC33.B4, R121.4
- removed net N$88: IC33.B5, R122.1
- removed net N$89: IC33.B6, R122.2
- removed net N$90: IC33.B7, R122.3
- removed net N$91: IC33.B8, R122.4
- removed net N$92: IC34.A8, IC37.GPA0
- removed net N$93: IC34.A7, IC37.GPA1
- removed net N$94: IC34.A6, IC37.GPA2
- removed net N$95: IC34.A5, IC37.GPA3
- removed net N$96: IC34.A4, IC37.GPA4
- removed net N$97: IC34.A3, IC37.GPA5
- removed net N$98: IC34.A2, IC37.GPA6
- removed net N$99: IC34.A1, IC37.GPA7
- removed net PGA_A_IN+: IC7.IN1+, R43.1
- removed net PGA_A_IN-: IC7.IN1-, IC7.IN2+, R44.2
- removed net PGA_B_IN+: IC9.IN1+, R24.1
- removed net PGA_B_IN-: IC9.IN1-, IC9.IN2+, R42.2
- removed net REFBY2: C71.1, IC10.REFBY2, REFBY2.P$1
- removed net REFM_A: C70.2, IC10.REFM_A
- removed net REFM_B: C110.2, IC10.REFM_B
- removed net REFOUT: C111.1, IC10.REFOUT, REFOUT.P$1
- removed net REFP_A: C70.1, IC10.REFP_A
- removed net REFP_B: C110.1, IC10.REFP_B
- removed net SPI0_CS0: DIO_CS.P$1, IC36.!CS, R29.1
- removed net SPI0_CS1: IC37.!CS, R30.1
- removed net SPI0_MISO: IC36.SO, IC37.SO, R27.1
- removed net SPI0_MOSI: IC22.DIN, IC36.SI, IC37.SI, R28.1
- removed net SPI0_SCK: IC22.SCLK, IC36.SCK, IC37.SCK, R26.1
- removed net SPI1_CS0: IC10.!CS, R15.1, R32.1, SPI1_CS0.P$1
- removed net SPI1_CS1: IC7.!CS, R33.1
- removed net SPI1_CS2: IC9.!CS, R34.1
- removed net SPI1_MISO: IC16.1B, IC16.2B, IC7.SDO, IC9.SDO, R18.1
- removed net SPI1_MOSI: IC10.SDI, IC7.SDI, IC9.SDI, R17.1
- removed net SPI1_SCK: IC10.SCLK, IC7.SCK, IC9.SCK, R25.1
- removed net VFB_12VN: C106.2, IC15.FBN, R56.1, R76.1, VFB12VN.P$1
- removed net VFB_12VP: C107.1, IC15.FBP, R55.1, R73.1, VFB12VP.P$1
- removed net VFB_14VN: C101.2, IC14.FBN, R54.1, R59.1, TP_VFB_14VN.P$1
- removed net VFB_14VP: C100.2, IC14.FBP, R53.1, R57.1, TP_VFB_14VP.P$1
- removed net VOCM_A: IC7.VOCM, R51.2, VOCMA.P$1
- removed net VOCM_B: IC9.VOCM, R52.1, VCOMB.P$1
- removed net VREF_ADC: C46.1, C72.1, C73.1, IC13.-IN, IC13.OUT, IC7.AVDD, IC9.AVDD, R49.3, TP9.P$1
- removed net VREF_ADC/2: C75.1, IC11.-IN, IC11.OUT, R51.1, R52.2, REF/2.P$1
- removed net VREF_ADC_RAW: C48.1, IC12.VREF, IC13.+IN, VREFR.P$1
- removed net VREF_DAC: C125.1, IC23.-IN, IC23.OUT, R100.1, R104.1, R108.1, R112.1, R116.1, R88.1, R92.1, R96.1
- removed net VREF_DAC_OUT: C124.1, IC22.VREF_IO, IC23.+IN, VREF_DAC.P$1
- removed net VREF_TPS: C99.2, IC14.VREF, R58.1, TP_VREF_TPS.P$1
- removed net V_OUT_REF: C153.1, C154.1, C157.1, C158.1, C161.1, C162.1, C165.1, C166.1, DIO_VREF.P$1, IC38.1B, IC38.2B, R127.2, R128.2, R129.2, R130.2
- new net RP2040_RST0: CON3.23, X1B.18
- new net RP2040_RST1: CON3.21, X3B.18
- new net SDO_A_1: CON2.13, X1A.18
- new net SDO_A_2: CON2.11, X1A.19
- new net SDO_A_3: CON2.9, X1A.20
- new net SDO_B_1: CON2.5, X1A.22
- new net SDO_B_2: CON2.3, X1A.23
- new net SDO_B_3: CON2.1, X1A.24
- new net SPI_ADC_CS: CON2.39, X1A.2
- new net SPI_AIOMODULE_CS0: CON3.5, X1A.29, X1B.29
- new net SPI_AIOMODULE_MISO: CON3.11, X1A.26, X1B.26
- new net SPI_AIOMODULE_MOSI: CON3.9, X1A.27, X1B.27
- new net SPI_AIOMODULE_SCK: CON3.7, X1A.28, X1B.28
- new net SPI_DAC_CS: CON2.21, X1B.2
- new net SPI_DIOMODULE_CS1: CON3.3, X3A.29, X3B.29
- new net SPI_DIOMODULE_MISO: X3A.26, X3B.26
- new net SPI_DIOMODULE_MOSI: X3A.27, X3B.27
- new net SPI_DIOMODULE_SCK: X3A.28, X3B.28
- new net SPI_DIO_CS0: CON3.33, X3A.2
- new net SPI_DIO_CS1: CON3.31, X3A.3
- new net SPI_MISO: CON2.29, X1A.7, X1B.7, X3A.7, X3B.7
- new net SPI_MOSI: CON2.31, X1A.6, X1B.6, X3A.6, X3B.6
- new net SPI_PGA_CS0: CON2.37, X1A.3
- new net SPI_PGA_CS1: CON2.35, X1A.4
- new net SPI_SCK: CON2.33, X1A.5, X1B.5, X3A.5, X3B.5
- new net SWCLK: CON3.15, X1B.23, X3B.23
- new net SWDIO: CON3.13, X1B.24, X3B.24
- new net UART0_RX: CON3.19, X1B.20, X3B.20
- new net UART0_TX: CON3.17, X1B.21, X3B.21
- net !ADC_RST: now also CON2.25, X1A.12; no longer IC10.!PD!/!RST, R16.2, R38.1
- net +1V8: now also PI1GPIO.87, PI1GPIO.89; no longer J2.88, J2.90
- net +3V3: now also PI1GPIO.83, PI1GPIO.85, X1A.1, X1B.1, X3A.1, X3B.1; no longer C122.1, C123.1, C126.1, C128.1, C131.1, C134.1, C137.1, C140.1, C143.1, C146.1, C149.1, C151.1, C152.1, C155.1, C156.1, C159.1, C160.1, C163.1, C164.1, C167.1, C168.1, C169.1, C170.1, C171.1, C21.1, C22.1, C25.1, C45.1, C47.1, C49.1, C50.1, C51.1, C64.1, C65.1, C76.1, IC10.AVDD, IC10.DVDD, IC11.V+, IC12.VIN, IC13.V+, IC16.VCC, IC17.V+, IC22.AVDD, IC23.V+, IC24.V+, IC25.V+, IC26.V+, IC27.V+, IC28.V+, IC29.V+, IC30.V+, IC31.V+, IC32.VREF_A, IC33.VREF_A, IC34.VREF_A, IC35.VREF_A, IC36.VDD, IC37.VDD, IC38.1A, IC38.VCC, IC39.V+, IC7.DVDD, IC9.DVDD, J2.84, J2.86, R16.1, R86.5, R86.6, R86.7, R86.8, TP_3V3.P$1
- net +5V: now also C21.1, CON3.1, CON3.2, PI1GPIO.78, PI1GPIO.80, PI1GPIO.82, PI1GPIO.84, PI1GPIO.86, PI1GPIO.88, X1A.8, X1A.9, X1B.8, X1B.9, X3A.8, X3A.9, X3B.8, X3B.9; no longer C120.1, C26.1, C85.1, IC14.INN, IC18.VIN, IC38.2A, J2.77, J2.79, J2.81, J2.83, J2.85, J2.87, J7.18, J7.33, R14.2, T2.S
- net ADC_RDY: now also CON2.27, X1A.11; no longer IC10.READY/STROBE, R36.1
- net BT_NDIS: now also PI1GPIO.92; no longer J2.91
- net CAM_GPIO0: now also PI1GPIO.98; no longer J2.97
- net CAM_GPIO1: now also PI1GPIO.99; no longer J2.100
- net CC1: now also PI1GPIO.93; no longer J2.94
- net CC2: now also PI1GPIO.95; no longer J2.96
- net DAC_!CLR: now also CON2.17, X1B.13; no longer CLR.P$1, IC22.!CLR, R37.1, R86.4
- net DAC_!LDAC: now also CON2.19, X1B.12; no longer IC22.!LDAC, LDAC.P$1, R35.1, R86.2
- net DIO_EN: now also CON3.29, X3A.11; no longer DIO_EN.P$1, IC32.EN, IC33.EN, IC34.EN, IC35.EN, R41.1
- net DIO_LEVEL_SELECT: now also CON3.25, X3A.13; no longer DIO_LS.P$1, IC38.1C, IC39.IN, R40.1
- net DIO_RESET: now also CON3.27, X3A.12; no longer DIO_RST.P$1, IC36.!RESET, IC37.!RESET, R39.1
- net DPHY0_C_N: now also PI1HISPEED.28; no longer J1.27
- net DPHY0_C_P: now also PI1HISPEED.30; no longer J1.29
- net DPHY0_D0_N: now also PI1HISPEED.16; no longer J1.15
- net DPHY0_D0_P: now also PI1HISPEED.18; no longer J1.17
- net DPHY0_D1_N: now also PI1HISPEED.22; no longer J1.21
- net DPHY0_D1_P: now also PI1HISPEED.24; no longer J1.23
- net DPHY0_D2_N: now also PI1HISPEED.34; no longer J1.33
- net DPHY0_D2_P: now also PI1HISPEED.36; no longer J1.35
- net DPHY0_D3_N: now also PI1HISPEED.40; no longer J1.39
- net DPHY0_D3_P: now also PI1HISPEED.42; no longer J1.41
- net DPHY1_C_N: now also PI1HISPEED.88; no longer J1.87
- net DPHY1_C_P: now also PI1HISPEED.90; no longer J1.89
- net DPHY1_D0_N: now also PI1HISPEED.76; no longer J1.75
- net DPHY1_D0_P: now also PI1HISPEED.78; no longer J1.77
- net DPHY1_D1_N: now also PI1HISPEED.82; no longer J1.81
- net DPHY1_D1_P: now also PI1HISPEED.84; no longer J1.83
- net DPHY1_D2_N: now also PI1HISPEED.94; no longer J1.93
- net DPHY1_D2_P: now also PI1HISPEED.96; no longer J1.95
- net DPHY1_D3_N: now also PI1HISPEED.93; no longer J1.94
- net DPHY1_D3_P: now also PI1HISPEED.95; no longer J1.96
- net EEPROM_NWP: now also PI1GPIO.19; no longer J2.20
- net ETH_LEDG: now also PI1GPIO.18; no longer J2.17
- net ETH_LEDY: now also PI1GPIO.16; no longer J2.15
- net GND: now also J1.GND, J1.GND_DRAIN, J1.SHIELD, J2.GND, J2.GND_DRAIN, J2.SHIELD, PI1GPIO.1, PI1GPIO.13, PI1GPIO.14, PI1GPIO.2, PI1GPIO.21, PI1GPIO.24, PI1GPIO.31, PI1GPIO.34, PI1GPIO.41, PI1GPIO.44, PI1GPIO.51, PI1GPIO.54, PI1GPIO.59, PI1GPIO.60, PI1GPIO.65, PI1GPIO.66, PI1GPIO.7, PI1GPIO.72, PI1GPIO.73, PI1GPIO.8, PI1GPIO.97, PI1HISPEED.13, PI1HISPEED.14, PI1HISPEED.19, PI1HISPEED.20, PI1HISPEED.25, PI1HISPEED.26, PI1HISPEED.31, PI1HISPEED.32, PI1HISPEED.37, PI1HISPEED.38, PI1HISPEED.43, PI1HISPEED.49, PI1HISPEED.55, PI1HISPEED.56, PI1HISPEED.61, PI1HISPEED.62, PI1HISPEED.67, PI1HISPEED.68, PI1HISPEED.7, PI1HISPEED.73, PI1HISPEED.74, PI1HISPEED.79, PI1HISPEED.8, PI1HISPEED.80, PI1HISPEED.85, PI1HISPEED.86, PI1HISPEED.91, PI1HISPEED.92, PI1HISPEED.97, PI1HISPEED.98, X1A.10, X1A.14, X1A.15, X1A.16, X1A.25, X1A.30, X1A.31, X1A.32, X1B.10, X1B.14, X1B.15, X1B.16, X1B.19, X1B.22, X1B.25, X1B.30, X1B.31, X1B.32, X3A.10, X3A.14, X3A.15, X3A.16, X3A.25, X3A.30, X3A.31, X3A.32, X3B.10, X3B.14, X3B.15, X3B.16, X3B.19, X3B.22, X3B.25, X3B.30, X3B.31, X3B.32; no longer BT1.-, C102.2, C103.2, C104.2, C105.1, C108.2, C109.2, C111.2, C120.2, C121.2, C122.2, C123.2, C124.2, C125.2, C126.2, C127.2, C128.2, C130.2, C131.2, C133.2, C134.2, C136.2, C137.2, C139.2, C140.2, C142.2, C143.2, C145.2, C146.2, C148.2, C149.2, C151.2, C152.2, C153.2, C154.2, C155.2, C156.2, C157.2, C158.2, C159.2, C160.2, C161.2, C162.2, C163.2, C164.2, C165.2, C166.2, C167.2, C168.2, C169.2, C170.2, C171.2, C22.2, C23.2, C24.1, C25.2, C26.2, C27.2, C42.2, C43.1, C45.2, C46.2, C47.2, C48.2, C49.2, C50.2, C51.2, C52.2, C53.2, C54.2, C55.2, C56.2, C57.2, C58.2, C59.2, C60.2, C61.2, C62.2, C63.2, C64.2, C65.2, C66.2, C67.2, C68.2, C69.2, C71.2, C74.2, C75.2, C76.2, C85.2, C86.2, C90.2, C91.2, C92.2, C93.2, C94.2, C95.2, C96.2, C97.2, C98.2, C99.1, DIO_GND.P$1, IC10.GND, IC10.PAD, IC11.V-, IC12.GND, IC13.V-, IC14.AGND, IC14.PGND, IC15.GND, IC15.PAD, IC16.GND, IC17.V-, IC18.GND, IC22.GND, IC23.V-, IC24.V-, IC25.V-, IC26.V-, IC27.V-, IC28.V-, IC29.V-, IC30.V-, IC31.V-, IC32.GND, IC33.GND, IC34.GND, IC35.GND, IC36.VSS, IC37.VSS, IC38.GND, IC39.V-, IC6.GND, IC7.AVSS, IC7.DVSS, IC7.IN2-, IC7.IOUT_HV, IC7.IOUT_LV, IC8.GND, IC9.AVSS, IC9.DVSS, IC9.IN2-, IC9.IOUT_HV, IC9.IOUT_LV, J1.13, J1.14, J1.19, J1.20, J1.25, J1.26, J1.31, J1.32, J1.37, J1.38, J1.44, J1.50, J1.55, J1.56, J1.61, J1.62, J1.67, J1.68, J1.7, J1.73, J1.74, J1.79, J1.8, J1.80, J1.85, J1.86, J1.91, J1.92, J1.97, J1.98, J2.1, J2.13, J2.14, J2.2, J2.22, J2.23, J2.32, J2.33, J2.42, J2.43, J2.52, J2.53, J2.59, J2.60, J2.65, J2.66, J2.7, J2.71, J2.74, J2.8, J2.98, J7.1, J7.23, J7.28, J7.34, J7.35, J7.57, J7.62, J7.68, J7.MH1, J7.MH2, L4.1, R103.1, R107.1, R111.1, R115.1, R57.2, R73.2, R87.1, R91.1, R95.1, R99.1, TP_GND.P$1, USB3USBA.GND, USB3USBA.GND_DRAIN, USB3USBA.SHIELD, USB3USBB.GND, USB3USBB.GND_DRAIN, USB3USBB.SHIELD
- net GPIO10: now also CON3.10, PI1GPIO.43; no longer J2.44, R28.2
- net GPIO11: now also CON3.8, PI1GPIO.37; no longer J2.38, R26.2
- net GPIO12: now also CON2.18, PI1GPIO.32; no longer J2.31
- net GPIO13: now also CON2.24, PI1GPIO.27; no longer J2.28, R40.2
- net GPIO14: now also CON3.18, PI1GPIO.56; no longer J2.55
- net GPIO15: now also CON3.20, PI1GPIO.52; no longer J2.51
- net GPIO16: now also CON2.36, PI1GPIO.30; no longer J2.29, R34.2
- net GPIO17: now also CON2.38, PI1GPIO.49; no longer J2.50, R33.2
- net GPIO18: now also CON2.40, PI1GPIO.50; no longer J2.49, R32.2
- net GPIO19: now also CON2.30, PI1GPIO.25; no longer J2.26, R18.2
- net GPIO2: now also CON3.24, PI1GPIO.57; no longer J2.58
- net GPIO20: now also CON2.32, PI1GPIO.28; no longer J2.27, R17.2
- net GPIO21: now also CON2.34, PI1GPIO.26; no longer J2.25, R25.2
- net GPIO22: now also CON3.32, PI1GPIO.45; no longer J2.46
- net GPIO23: now also PI1GPIO.48; no longer J2.47, R31.2
- net GPIO24: now also CON3.14, PI1GPIO.46; no longer J2.45, R36.2
- net GPIO25: now also CON3.16, PI1GPIO.42; no longer J2.41, R38.2
- net GPIO26: now also CON2.20, PI1GPIO.23; no longer J2.24
- net GPIO27: now also CON3.34, PI1GPIO.47; no longer J2.48, R35.2
- net GPIO3: now also CON3.22, PI1GPIO.55; no longer J2.56
- net GPIO4: now also CON2.28, PI1GPIO.53; no longer J2.54, R37.2
- net GPIO5: now also CON2.22, PI1GPIO.33; no longer J2.34, R41.2
- net GPIO6: now also CON2.26, CON3.30, PI1GPIO.29; no longer J2.30, R39.2
- net GPIO7: now also CON3.4, PI1GPIO.38; no longer J2.37, R30.2
- net GPIO8: now also CON3.6, PI1GPIO.40; no longer J2.39, R29.2
- net GPIO9: now also CON3.12, PI1GPIO.39; no longer J2.40, R27.2
- net GPIO_VREF: now also PI1GPIO.77; no longer J2.78
- net HDMI0_CEC: now also PI1HISPEED.52; no longer J1.51
- net HDMI0_CK_N: now also PI1HISPEED.89; no longer J1.90
- net HDMI0_CK_P: now also PI1HISPEED.87; no longer J1.88
- net HDMI0_D0_N: now also PI1HISPEED.83; no longer J1.84
- net HDMI0_D0_P: now also PI1HISPEED.81; no longer J1.82
- net HDMI0_D1_N: now also PI1HISPEED.77; no longer J1.78
- net HDMI0_D1_P: now also PI1HISPEED.75; no longer J1.76
- net HDMI0_D2_N: now also PI1HISPEED.71; no longer J1.72
- net HDMI0_D2_P: now also PI1HISPEED.69; no longer J1.70
- net HDMI0_HOTPLUG: now also PI1HISPEED.54; no longer J1.53
- net HDMI0_SCL: now also PI1HISPEED.99; no longer J1.100
- net HDMI0_SDA: now also PI1HISPEED.100; no longer J1.99
- net HDMI1_CEC: now also PI1HISPEED.50; no longer J1.49
- net HDMI1_CK_N: now also PI1HISPEED.65; no longer J1.66
- net HDMI1_CK_P: now also PI1HISPEED.63; no longer J1.64
- net HDMI1_D0_N: now also PI1HISPEED.59; no longer J1.60
- net HDMI1_D0_P: now also PI1HISPEED.57; no longer J1.58
- net HDMI1_D1_N: now also PI1HISPEED.53; no longer J1.54
- net HDMI1_D1_P: now also PI1HISPEED.51; no longer J1.52
- net HDMI1_D2_N: now also PI1HISPEED.47; no longer J1.48
- net HDMI1_D2_P: now also PI1HISPEED.45; no longer J1.46
- net HDMI1_HOTPLUG: now also PI1HISPEED.44; no longer J1.43
- net HDMI1_SCL: now also PI1HISPEED.48; no longer J1.47
- net HDMI1_SDA: now also PI1HISPEED.46; no longer J1.45
- net ID_SC: now also PI1GPIO.36; no longer J2.35
- net ID_SD: now also PI1GPIO.35; no longer J2.36
- net LED_NACT: now also PI1GPIO.22; no longer J2.21
- net MISO_SEL: now also CON2.23, X1A.13; no longer IC16.1C, IC17.IN
- net NPWR_LED: now also PI1GPIO.96; no longer J2.95
- net NRPIBOOT: now also PI1GPIO.94; no longer J2.93
- net PCIE_CLK_N: now also PI1HISPEED.11; no longer J1.12
- net PCIE_CLK_P: now also PI1HISPEED.9; no longer J1.10
- net PCIE_NCLKREQ: now also PI1HISPEED.1; no longer J1.2
- net PCIE_NRST: now also PI1HISPEED.10; no longer J1.9
- net PCIE_NWAKE: now also PI1HISPEED.3; no longer J1.4
- net PCIE_PWR_EN: now also PI1HISPEED.5; no longer J1.6
- net PCIE_RX_N: now also PI1HISPEED.17; no longer J1.18
- net PCIE_RX_P: now also PI1HISPEED.15; no longer J1.16
- net PCIE_TX_N: now also PI1HISPEED.23; no longer J1.24
- net PCIE_TX_P: now also PI1HISPEED.21; no longer J1.22
- net PMIC_ENABLE: now also PI1GPIO.100; no longer J2.99
- net PWM: now also PI1GPIO.20; no longer J2.19
- net PWR_BUT: now also PI1GPIO.91; no longer J2.92
- net SCL0: now also PI1GPIO.79; no longer J2.80
- net SDA0: now also PI1GPIO.81; no longer J2.82
- net SDO_A_0: now also CON2.15, X1A.17; no longer IC10.SDO-0/0A, IC16.1A
- net SDO_B_0: now also CON2.7, X1A.21; no longer IC10.SDO-4/0B, IC16.2A
- net SD_CLK: now also PI1GPIO.58; no longer J2.57
- net SD_CMD: now also PI1GPIO.61; no longer J2.62
- net SD_DAT0: now also PI1GPIO.64; no longer J2.63
- net SD_DAT1: now also PI1GPIO.68; no longer J2.67
- net SD_DAT2: now also PI1GPIO.70; no longer J2.69
- net SD_DAT3: now also PI1GPIO.62; no longer J2.61
- net SD_PWR_ON: now also PI1GPIO.76; no longer J2.75
- net SYNC_OUT: now also PI1GPIO.17; no longer J2.18
- net TACHO: now also PI1GPIO.15; no longer J2.16
- net TRD0_N: now also PI1GPIO.9; no longer J2.10
- net TRD0_P: now also PI1GPIO.11; no longer J2.12
- net TRD1_N: now also PI1GPIO.5; no longer J2.6
- net TRD1_P: now also PI1GPIO.3; no longer J2.4
- net TRD2_N: now also PI1GPIO.10; no longer J2.9
- net TRD2_P: now also PI1GPIO.12; no longer J2.11
- net TRD3_N: now also PI1GPIO.6; no longer J2.5
- net TRD3_P: now also PI1GPIO.4; no longer J2.3
- net USB2_N: now also PI1HISPEED.4; no longer J1.3
- net USB2_P: now also PI1HISPEED.6; no longer J1.5
- net USB3-0-D_N: now also J1.D-, PI1HISPEED.35; no longer J1.36, USB3USBA.D-
- net USB3-0-D_P: now also J1.D+, PI1HISPEED.33; no longer J1.34, USB3USBA.D+
- net USB3-0-RX_N: now also J1.STDA_SSRX-, PI1HISPEED.27; no longer J1.28, USB3USBA.STDA_SSRX-
- net USB3-0-RX_P: now also J1.STDA_SSRX+, PI1HISPEED.29; no longer J1.30, USB3USBA.STDA_SSRX+
- net USB3-0-TX_N: now also J1.STDA_SSTX-, PI1HISPEED.39; no longer J1.40, USB3USBA.STDA_SSTX-
- net USB3-0-TX_P: now also J1.STDA_SSTX+, PI1HISPEED.41; no longer J1.42, USB3USBA.STDA_SSTX+
- net USB3-1-D_N: now also J2.D-, PI1HISPEED.66; no longer J1.65, USB3USBB.D-
- net USB3-1-D_P: now also J2.D+, PI1HISPEED.64; no longer J1.63, USB3USBB.D+
- net USB3-1-RX_N: now also J2.STDA_SSRX-, PI1HISPEED.58; no longer J1.57, USB3USBB.STDA_SSRX-
- net USB3-1-RX_P: now also J2.STDA_SSRX+, PI1HISPEED.60; no longer J1.59, USB3USBB.STDA_SSRX+
- net USB3-1-TX_N: now also J2.STDA_SSTX-, PI1HISPEED.70; no longer J1.69, USB3USBB.STDA_SSTX-
- net USB3-1-TX_P: now also J2.STDA_SSTX+, PI1HISPEED.72; no longer J1.71, USB3USBB.STDA_SSTX+
- net USBOTG_ID: now also PI1HISPEED.2; no longer J1.1
- net VBAT: now also PI1GPIO.75; no longer BT1.+, J2.76, TP-VBAT.P$1
- net VBUS: now also J1.VBUS, J2.VBUS; no longer USB3USBA.VBUS, USB3USBB.VBUS
- net VBUS_EN: now also PI1HISPEED.12; no longer J1.11
- net WL_NDIS: now also PI1GPIO.90; no longer J2.89
Other:
- note added: "AIO BOARD CONNECTOR"
- note added: "BOARD JUMPERS"
- note added: "DIO BOARD CONNECTOR"
- note added: "Enable SWD Debugging on Raspberry Pi: Install OpenOCD (sudo apt install openocd) Configure /boot/config.txt to enable GPIO-based debugging. SWDIO - GPIO24 SWCLK - GPIO25"
- note added: "GPIO12"
- note added: "GPIO13"
- note added: "GPIO16"
- note added: "GPIO2"
- note added: "GPIO22"
- note added: "GPIO26"
- note added: "GPIO27"
- note added: "GPIO3"
- note added: "GPIO4"
- note added: "GPIO5"
- note added: "GPIO6"
- note added: "NOT NEEDED"
- note added: "SPI0-CE0"
- note added: "SPI0-CE1"
- note added: "SPI0-MISO"
- note added: "SPI0-MOSI"
- note added: "SPI0-SCLK"
- note added: "SPI1-CE0"
- note added: "SPI1-CE1"
- note added: "SPI1-CE2"
- note added: "SPI1-MISO"
- note added: "SPI1-MOSI"
- note added: "SPI1-SCLK"
- note added: "TCK - ALT4"
- note added: "TDO - ALT4"
- note added: "UART0 -RX"
- note added: "UART0 -TX"
- note removed: "+/-14V to +/12V LDO"
- note removed: "0 0 1 OUT0"
- note removed: "0 1 1 OUT1"
- note removed: "1 0 1 OUT2"
- note removed: "1 1 1 OUT3"
- note removed: "2.5V VREF"
- note removed: "3.3V TARGET LDO"
- note removed: "5V to +/-14V BOOST CONVERTER"
- note removed: "A1 A0 EN ON"
- note removed: "ADC ON SPI1"
- note removed: "ADS9234R ADC"
- note removed: "ANALOG-IN TESTPOINTS"
- note removed: "ANALOG-OUT DAC"
- note removed: "ANALOG-OUT OUTPUT DRIVERS"
- note removed: "ANALOG-OUT TESTPOINTS"
- note removed: "Choose R_ISOLATION = 68 Ω: 1. Stability with Capacitive Load: The combination of R_ISO and C_LOAD creates a low-pass filter. The cutoff frequency is: f_c = 1 / (2 * π * R_ISO * C_LOAD) For R_ISO = 68 Ω and C_LOAD = 20 nF: f_c = 1 / (2 * π * 68 * 20e-9) ≈ 117.2 kHz 2. Voltage Drop Across R_ISO: The voltage drop is: V_drop = I_load * R_ISO"
- note removed: "DAC8568 Output Calculation: V_OUT = (1 + R_FB/R_G2 + R_FB/R_G1) * V_DAC - (R_FB/R_G2) * V_REF Given: Supply voltage: +/-12V Reference voltage (V_REF): 2.5V DAC resolution: 16 bits Desired output range: -12V to +12V 1. Determine the Gain (G): G = (V_OUT_max - V_OUT_min) / (V_DAC_max - V_DAC_min) G = (12 - (-12)) / (2.5 - 0) = 24 / 2.5 = 9.6 2. Solve for Resistor Ratios: G = 1 + R_FB/R_G2 + R_FB/R_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"
- note removed: "DIGITAL IO - LOWER 16 BITS"
- note removed: "DIGITAL IO - UPPER 16 BITS"
- note removed: "DIO ON SPI0"
- note removed: "IN0+ AND IN1-"
- note removed: "IN10+ AND IN11-"
- note removed: "IN12+ AND IN13-"
- note removed: "IN14+ AND IN15-"
- note removed: "IN2+ AND IN3-"
- note removed: "IN4+ AND IN5-"
- note removed: "IN6+ AND IN7-"
- note removed: "IN8+ AND IN9-"
- note removed: "INPUT MULTIPLEXER"
- note removed: "IO-GPIO JUMPERS"
- note removed: "Negative Channel: - Known Values: - VBUF = 1.184 V - VOUTN = -12 V - R2N = 10 kΩ - Formula: R1N = -(VOUTN × R2N) / VBUF - Calculation: R1N = -(-12 × 10) / 1.184 R1N = (120 / 1.184) = 101.4 kΩ - Closest Resistor Value (0.1% Tolerance): R1N = 101 kΩ Final Resistor Values: - Negative Channel: - R1N = 101 kΩ - R2N = 10 kΩ - Calculated VOUTN ≈ -12.0 V Negative Channel: - Target VOUTN = -12 V, adjustme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"
- note removed: "Negative Output (Vout_neg = -14V): - Given: - R1 = 1.3 MΩ - Calculated R2 ≈ 136.3 kΩ - Nearest E96 Standard Value: - R2 = 137 kΩ - Resulting Output Voltage: - Vout = 1.213 × (1 + R1 / R2) - Vout = 1.213 × (1 + 1300 / 137) ≈ 14.01 V - Final Pair: - R1 = 1.3 MΩ - R2 = 137 kΩ Negative Channel: - Target VOUTN = -14 V, adjustment range: -12.6 V to -15.4 V. - Configuration: - R2N = 137 kΩ (fixed). - R1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"
- note removed: "PGA"
- note removed: "Positive Channel: - Known Values: - VFBP = 1.184 V - VOUTP = 12 V - R2P = 10 kΩ - Formula: R1P = (VOUTP / VFBP - 1) × R2P - Calculation: R1P = (12 / 1.184 - 1) × 10 R1P = (10.14 - 1) × 10 = 91.4 kΩ - Closest Resistor Value (0.1% Tolerance): R1P = 91.5 kΩ Final Resistor Values: - Positive Channel: - R1P = 91.5 kΩ - R2P = 10 kΩ - Calculated VOUTP ≈ 12.0 V Positive Channel: - Target VOUTP = 12 V, ad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"
- note removed: "Positive Output (Vout_pos = 14V): - Given: - R1 = 976 kΩ - Calculated R2 ≈ 102.3 kΩ - Nearest E96 Standard Value: - R2 = 102 kΩ - Resulting Output Voltage: - Vout = 1.213 × (1 + R1 / R2) - Vout = 1.213 × (1 + 976 / 102) ≈ 13.98 V - Final Pair: - R1 = 976 kΩ - R2 = 102 kΩ Positive Channel: - Target VOUTP = 14 V, adjustment range: 12.6 V to 15.4 V. - Configuration: - R2P = 102 kΩ (fixed). - R1P = 9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"
- note removed: "SPI0"
- note removed: "SPI1"
- note removed: "TEST CONNECTOR"
- note removed: "TESTPOINTS POWER"
- note removed: "X X 0 -"
