File: src/HardwareDesign/Module_DIO.sch (EAGLE design)
At the start: 364 parts, among them IC1 RT9742GGJ, IC10 ADS9234RIRHBR, IC11 MCP6001RT, IC12 MCP1525T-I/TT, IC13 MCP6001RT, IC14 TPS65131, IC15 TPS7A39, IC16 SN74LVC2G66, IC17 74LVC1G04, IC2 AP22653W6, IC22 DAC8568, IC23 MCP6001RT, IC24 MCP6001RT, IC25 MCP6001RT, IC26 MCP6001RT, IC27 MCP6001RT, IC28 MCP6001RT, IC29 MCP6001RT, IC3 74LVC1G07, IC30 MCP6001RT, IC31 MCP6001RT, IC32 LSF0108, IC33 LSF0108, IC34 LSF0108, IC35 LSF0108, IC36 MCP23S18, IC38 SN74LVC2G66, IC39 74LVC1G04, IC4 RT9742NGV, IC5 AP3441SHE-7B, IC6 DG409, IC7 ADA4254ACPZ, IC8 DG409, IC9 ADA4254ACPZ, J1 10164227-1001A1RLF, J2 10164227-1001A1RLF, J3 FH12-22S-0.5SVA, J4 FH12-22S-0.5SH(55), J7 2-5174225-5, SW1 1825027-8, T2 IRLML5203, X2 CRYSTAL

Commit message: finish DIO card desing
Parts:
- removed 12VN, 12VP, 14VN, 14VP, BUF, CLR, DIO_CS, LDAC, REF/2, REFBY2, REFOUT, SPI1_CS0, SYNC, TP-5VHD, TP-5VP, TP-BTN, TP-GREF, TP-LED, TP-LX, TP-M2CLK, TP-M2FB, TP-VBAT, TP-VBUS, TP-VM2, TP-VSD, TP9, TPD0, TP_3V3, TP_5VP, TP_BSW_G, TP_GND, TP_VFB_14VN, TP_VFB_14VP, TP_VREF_TPS, VCOMB, VFB12VN, VFB12VP, VOCMA, VREFR, VREF_DAC: TP, ds_passive:TP
- removed 2230, 2242, 2260, 2280: M2 x 1mm, Wurth_Assembly_WA-SMSI:WA-SMSI_9774XXX243_9774010243
- removed BT1: 79523141, Battery Holder:79523141
- removed C10, C11, C111, C12, C125, C126, C128, C129, C131, C132, C134, C135, C137, C138, C140, C141, C143, C144, C146, C147, C149, C150, C20, C22, C25, C45, C46, C49, C51, C53, C55, C57, C59, C61, C63, C65, C67, C69, C71, C75, C76, C9: 100nF, ds_passive:C0402
- removed C100, C101: 10pF, ds_passive:C0402
- removed C102, C104: 10uF, ds_passive:C1206
- removed C103, C106, C107: 10nF, ds_passive:C0402
- removed C105, C99: 220nF, ds_passive:C0402
- removed C108, C109, C93, C94, C95, C96, C97, C98: 22uF, ds_passive:C1206
- removed C110, C70: 10uF, ds_passive:C0603
- removed C122, C124, C50, C52, C54, C56, C58, C60, C62, C64, C66, C68, C72: 1uF, ds_passive:C0603
- removed C123, C21, C73: 100nF, ds_passive:C0603
- removed C127, C130, C133, C136, C139, C142, C145, C148: 20nF, ds_passive:C0402
- removed C13: 4.7nF, ds_passive:C0402
- removed C14, C15, C16, C17, C18, C19, C47, C7, C90: 10uF, ds_passive:C0805
- removed C23, C24, C42, C43: 270pF, ds_passive:C0402
- removed C41, C44: 680pF, ds_passive:C0402
- removed C48, C74: (no value), ds_passive:C0805
- removed C8: 100uF 16V, ds_passive:CPOL
- removed C85: 4.7uF, ds_passive:C0805
- removed C86: 100nF, ds_passive:C0805
- removed C91: 10nF, ds_passive:C0805
- removed C92: 4.7nF, ds_passive:C0805
- removed CON1: (no value), ds_con:CON-1X4
- removed D2: TPD4EUSB30, ds_ic_peripherals:TPD4EUSB30
- removed D3, D4: SS12, Diodes:SS12
- removed ETH1: G16LX-188S7-1G-GO-Y, ds_con:MAGJACK-POE
- removed GPIO: (no value), ds_con:CON-2X20
- removed HDMI1, HDMI2: 685119136923, Wurth_Connectors_WR-HDMI:685119136923
- removed IC10: ADS9234RIRHBR, ds_ic_peripherals:ADS9234RIRHBR
- removed IC11, IC13, IC23, IC24, IC25, IC26, IC27, IC28, IC29, IC30, IC31: MCP6001RT, ds_ic_opa:MCP6001RT
- removed IC12: MCP1525T-I/TT, ds_ic_vreg:MCP1525T-I/TT
- removed IC14: TPS65131, ds_ic_vreg:TPS65131TRGERQ1
- removed IC15: TPS7A39, ds_ic_vreg:TPS7A3901DSCR
- removed IC16: SN74LVC2G66, ds_ic_peripherals:SN74LVC2G66
- removed IC17: 74LVC1G04, ds_ic_logic:74LVC1G04
- removed IC18: (no value), ds_ic_vreg:LDL1117S33R
- removed IC22: DAC8568, ds_ic_peripherals:DAC8568
- removed IC5: AP3441SHE-7B, ds_ic_vreg:AP3441SHE-7B
- removed IC6, IC8: DG409, ds_ic_peripherals:DG409EUE+
- removed IC7, IC9: ADA4254ACPZ, ds_ic_opa:ADA4254ACPZ
- removed J2: 10164227-1001A1RLF, ds_con:10164227-1001A1RLF
- removed J3: FH12-22S-0.5SVA, ds_con:FH12-22S-0.5SVA
- removed J4: FH12-22S-0.5SH(55), ds_con:FH12-22S-0.5SH(55)
- removed J7: 2-5174225-5, Connector_D-Sub:2-5174225-5
- removed JP1, JP3: (no value), ds_con:CON-2X2
- removed JP2: (no value), ds_con:CON-2X7
- removed JP4: POE, ds_con:CON-2X2
- removed L1: L, ds_passive:L
- removed L3, L4: SRR5228A-4R7Y, ds_passive:L
- removed LED1: Green, led:LEDCHIPLED_0805
- removed LED2: (no value), led:LEDCHIPLED_0805
- removed PCIE: M.2, ds_con:M.2
- removed R100, R103, R104, R107, R108, R111, R112, R115, R116, R73, R76, R87, R88, R91, R92, R95, R96, R99: 10K 0.1%, ds_passive:R0402
- removed R101, R105, R109, R113, R117, R89, R93, R97: 43K 0.1%, ds_passive:R0402
- removed R102, R106, R110, R114, R118, R90, R94, R98: 68R 1%, ds_passive:R0402
- removed R12: 10K 1%, ds_passive:R0402
- removed R128, R129, R130: 200K, ds_passive:R0402
- removed R13: 2.2K 1%, ds_passive:R0402
- removed R14: 100R, ds_passive:R1206
- removed R15, R24, R42, R43, R44, R45, R46, R47, R48: 0R, ds_passive:R0402
- removed R16: 10K, ds_passive:R0402
- removed R17, R18, R25, R26, R27, R28, R29, R30, R31, R32, R33, R34, R35, R36, R37, R38, R39, R40, R41, R51, R52: 0R, ds_passive:R0603
- removed R19: 950K 0.1%, ds_passive:R0402
- removed R20, R21: 200R, ds_passive:R0402
- removed R49, R53, R54, R55, R56: (no value), ds_passive:R-TRIM
- removed R50: 100R, ds_passive:R0402
- removed R57: 102K 0.1%, ds_passive:R0402
- removed R58: 1.2M 0.1%, ds_passive:R0402
- removed R59: 137K 0.1%, ds_passive:R0402
- removed R60: 75K 0.1%, ds_passive:R0402
- removed R74: 90K 0.1%, ds_passive:R0402
- removed R86: CRA034RF100RP05Z, Resistor Array:YC164-JR-0733RL
- removed SD1: (no value), ds_con:MICRO-SD
- removed SW1: 1825027-8, ds_passive:1825027-8
- removed T2: IRLML5203, transistor-power:IRLML5203
- removed USB3: 692141030100, Wurth_Connectors_WR-USB:692141030100
- removed X2: CRYSTAL, ds_passive:CRYSTAL
- added AVDD, CS0, CS1, DVDD, IOVDD, MISO, MOSI, SCK, VBUS, VREF1: TP, ds_passive:TP
- added C112, C113, C114, C116, C77, C80, C81, C82, C83, C84, C87, C88, C89: 100nF, ds_passive:C-0402
- added C115: 4.7nF, ds_passive:C0402
- added C78: 10uF, ds_passive:C0805
- added C79: 100nF, ds_passive:C0402
- added DBG1, DBG2: (no value), ds_con:CON-1X4
- added ESD1: SP0503BAHTG-ES, ds_ic_peripherals:SP0503BAHT
- added JP-3V3-1, JP-3V3-2, JP-EXT-1, JP-EXT-2: 0R, ds_passive:R0603
- added R62: 5.1K, ds_passive:R0402
- added R63, R64, R72, R75, R77: 10K, ds_passive:R0402
- added R68: 1M, ds_passive:R0402
- added REF1: LM4040BXX, ds_ic_vreg:LM4040BXX
- added RESET, USB_BOOT: B3U-1000P-B, 52101-101-REV-A_v16:SWITCH-OMRON_B3U-1000P
- added X1: K5A1200015304P, ds_passive:CRYSTAL
- added X3: CON-VG_MAB64, ds_con:CON-VG_MAB64
- C1, C2: value (none) -> 15pF; device ds_passive:C0402 -> ds_passive:C-0402
- C120, C121, C151, C152, C153, C154, C155, C156, C157, C158, C159, C160, C161, C162, C163, C164, C165, C166, C167, C168, C169, C170, C4, C5: device ds_passive:C0402 -> ds_passive:C-0402
- C171: device ds_passive:C0603 -> ds_passive:C-0603
- C3: value 100nF -> 1uF; device ds_passive:C0402 -> ds_passive:C-0402
- C6: value 10uF -> 100nF; device ds_passive:C0805 -> ds_passive:C-0402
- D1: value TPD4EUSB30 -> SS12; device ds_ic_peripherals:TPD4EUSB30 -> Diodes:SS12
- IC1: value RT9742GGJ -> MIC5504-3.3YM5-TR; device ds_ic_peripherals:RT9742GGJ5 -> ds_ic_vreg:MIC5504-3.3YM5-TR
- IC2: value AP22653W6 -> RP2040; device ds_ic_peripherals:AP22653W6 -> ds_ic_mcu:RP2040
- IC3: value 74LVC1G07 -> MCP6001AIDBVRG; device ds_ic_logic:74LVC1G07 -> ds_ic_opa:MCP6001RT
- IC37: value (none) -> MCP23S18
- IC4: value RT9742NGV -> W25Q128JVPIQ; device ds_ic_peripherals:RT9742NGV -> MCU:W25Q128JVP
- J1: value 10164227-1001A1RLF -> (none); device ds_con:10164227-1001A1RLF -> ds_con:N10236-52B3PC
- R1, R4: value 2.2K 1% -> 1K
- R10: value (none) -> 200K
- R11: value 100K 1% -> 200K
- R2: value 15K 1% -> 4.7K
- R22, R23: value 200R -> 10K
- R3: value 2.2K 1% -> DNI
- R5: value 1K -> 2.2K 1%
- R6: value 0R -> 27R
- R61: value 2.2K 1% -> 5.1K
- R7: value DNI -> 27R
- R8: value 470R -> 200K
- R9: value 470R -> 0R
- USBC: value 629722000214 -> USB-TYPE-C-018
Connections:
- removed net !ADC_RST: IC10.!PD!/!RST, R16.2, R38.1
- removed net !MISO_SEL: IC16.2C, IC17.OUT
- removed net +12V: 12VP.P$1, C107.2, C108.1, C52.1, C53.1, C56.1, C57.1, C60.1, C61.1, C66.1, C67.1, IC15.OUTP, IC6.V+, IC7.VDDH, IC8.V+, IC9.VDDH, R60.1
- removed net +14V: 14VP.P$1, C100.1, C104.1, C93.1, C94.1, C95.1, D3.C, IC14.VPOS, IC15.EN, IC15.INP, R19.1
- removed net +1V8: J2.88, J2.90, R7.1
- removed net +3V3_EXT: C121.1, C27.1, IC18.VOUT, J7.52, J7.67
- removed net -12V: 12VN.P$1, C106.1, C109.1, C54.1, C55.1, C58.1, C59.1, C62.1, C63.1, C68.1, C69.1, IC15.OUTN, IC6.V-, IC7.PAD, IC7.VSSH, IC8.V-, IC9.PAD, IC9.VSSH, R76.2
- removed net -14V: 14VN.P$1, C101.1, C102.1, C96.1, C97.1, C98.1, D4.A, IC14.VNEG, IC15.INN, R59.2
- removed net ADA_A_IO0: IC6.A0, IC7.GPIO0
- removed net ADA_A_IO1: IC6.A1, IC7.GPIO1
- removed net ADA_A_IO2: IC6.EN, IC7.GPIO2
- removed net ADA_B_IO0: IC8.A0, IC9.GPIO0
- removed net ADA_B_IO1: IC8.A1, IC9.GPIO1
- removed net ADA_B_IO2: IC8.EN, IC9.GPIO2
- removed net ADC_AIN_N: C24.2, C41.2, R21.1, R46.1
- removed net ADC_AIN_P: C23.1, C41.1, R20.1, R45.2
- removed net ADC_BIN_N: C43.2, C44.2, R23.1, R48.2
- removed net ADC_BIN_P: C42.1, C44.1, R22.1, R47.1
- removed net ADC_IN0: IC10.AINP_A, R45.1
- removed net ADC_IN1: IC10.AINM_A, R46.2
- removed net ADC_IN2: IC10.AINP_B, R48.1
- removed net ADC_IN3: IC10.AINM_B, R47.2
- removed net ADC_RDY: IC10.READY/STROBE, R36.1
- removed net AO_0: C127.1, J7.29, R89.2, R90.2
- removed net AO_1: C130.1, J7.63, R93.2, R94.2
- removed net AO_2: C133.1, J7.30, R97.2, R98.2
- removed net AO_3: C136.1, J7.64, R101.2, R102.2
- removed net AO_4: C139.1, J7.31, R105.2, R106.2
- removed net AO_5: C142.1, J7.65, R109.2, R110.2
- removed net AO_6: C145.1, J7.32, R113.2, R114.2
- removed net AO_7: C148.1, J7.66, R117.2, R118.2
- removed net BSW_G: IC14.BSW, T2.G, TP_BSW_G.P$1
- removed net BT_NDIS: J2.91, JP3.3
- removed net BUF: BUF.P$1, C105.2, IC15.BUF, R74.1
- removed net CAM_GPIO0: J2.97, J3.17
- removed net CAM_GPIO1: J2.100, J3.18
- removed net DAC_!CLR: CLR.P$1, IC22.!CLR, R37.1, R86.4
- removed net DAC_!LDAC: IC22.!LDAC, LDAC.P$1, R35.1, R86.2
- removed net DAC_!SYNC: IC22.!SYNC, R31.1, R86.3, SYNC.P$1
- removed net DAC_0: IC22.VOUT_A, IC24.+IN, TPD0.P$1
- removed net DAC_1: IC22.VOUT_B, IC25.+IN
- removed net DAC_2: IC22.VOUT_C, IC26.+IN
- removed net DAC_3: IC22.VOUT_D, IC27.+IN
- removed net DAC_4: IC22.VOUT_E, IC28.+IN
- removed net DAC_5: IC22.VOUT_F, IC29.+IN
- removed net DAC_6: IC22.VOUT_G, IC30.+IN
- removed net DAC_7: IC22.VOUT_H, IC31.+IN
- removed net DPHY0_C_N: J1.27, J3.8
- removed net DPHY0_C_P: J1.29, J3.9
- removed net DPHY0_D0_N: J1.15, J3.2
- removed net DPHY0_D0_P: J1.17, J3.3
- removed net DPHY0_D1_N: J1.21, J3.5
- removed net DPHY0_D1_P: J1.23, J3.6
- removed net DPHY0_D2_N: J1.33, J3.11
- removed net DPHY0_D2_P: J1.35, J3.12
- removed net DPHY0_D3_N: J1.39, J3.14
- removed net DPHY0_D3_P: J1.41, J3.15
- removed net DPHY1_C_N: J1.87, J4.8
- removed net DPHY1_C_P: J1.89, J4.9
- removed net DPHY1_D0_N: J1.75, J4.2
- removed net DPHY1_D0_P: J1.77, J4.3
- removed net DPHY1_D1_N: J1.81, J4.5
- removed net DPHY1_D1_P: J1.83, J4.6
- removed net DPHY1_D2_N: J1.93, J4.11
- removed net DPHY1_D2_P: J1.95, J4.12
- removed net DPHY1_D3_N: J1.94, J4.14
- removed net DPHY1_D3_P: J1.96, J4.15
- removed net EEPROM_NWP: J2.20, JP2.4
- removed net ETH_LEDG: J2.17, R8.1
- removed net ETH_LEDY: J2.15, R9.2
- removed net GPIO10: GPIO.19, J2.44, R28.2
- removed net GPIO11: GPIO.23, J2.38, R26.2
- removed net GPIO12: GPIO.32, J2.31
- removed net GPIO13: GPIO.33, J2.28, R40.2
- removed net GPIO14: GPIO.8, J2.55
- removed net GPIO15: GPIO.10, J2.51
- removed net GPIO16: GPIO.36, J2.29, R34.2
- removed net GPIO17: GPIO.11, J2.50, R33.2
- removed net GPIO18: GPIO.12, J2.49, R32.2
- removed net GPIO19: GPIO.35, J2.26, R18.2
- removed net GPIO2: GPIO.3, J2.58
- removed net GPIO20: GPIO.38, J2.27, R17.2
- removed net GPIO21: GPIO.40, J2.25, R25.2
- removed net GPIO22: GPIO.15, J2.46
- removed net GPIO23: GPIO.16, J2.47, R31.2
- removed net GPIO24: GPIO.18, J2.45, R36.2
- removed net GPIO25: GPIO.22, J2.41, R38.2
- removed net GPIO26: GPIO.37, J2.24
- removed net GPIO27: GPIO.13, J2.48, R35.2
- removed net GPIO3: GPIO.5, J2.56
- removed net GPIO4: GPIO.7, J2.54, R37.2
- removed net GPIO5: GPIO.29, J2.34, R41.2
- removed net GPIO6: GPIO.31, J2.30, R39.2
- removed net GPIO7: GPIO.26, J2.37, R30.2
- removed net GPIO8: GPIO.24, J2.39, R29.2
- removed net GPIO9: GPIO.21, J2.40, R27.2
- removed net GPIO_VREF: J2.78, R3.1, R4.1, R6.2, R7.2, TP-GREF.P$1
- removed net HDMI0_CEC: HDMI2.GROUND, J1.51
- removed net HDMI0_CK_N: HDMI2.TMDSCLOCK-, J1.90
- removed net HDMI0_CK_P: HDMI2.TMDSCLOCKSHIELD, J1.88
- removed net HDMI0_D0_N: HDMI2.TMDS0-, J1.84
- removed net HDMI0_D0_P: HDMI2.TMDS0SHIELD, J1.82
- removed net HDMI0_D1_N: HDMI2.TMDS1-, J1.78
- removed net HDMI0_D1_P: HDMI2.TMDS1SHIELD, J1.76
- removed net HDMI0_D2_N: HDMI2.TMDS2-, J1.72
- removed net HDMI0_D2_P: HDMI2.TMDS2SHIELD, J1.70
- removed net HDMI0_HOTPLUG: HDMI2.HOTPLUG/HEC+, J1.53
- removed net HDMI0_SCL: HDMI2.SCL, J1.100
- removed net HDMI0_SDA: HDMI2.SDA, J1.99
- removed net HDMI1_CEC: HDMI1.GROUND, J1.49
- removed net HDMI1_CK_N: HDMI1.TMDSCLOCK-, J1.66
- removed net HDMI1_CK_P: HDMI1.TMDSCLOCKSHIELD, J1.64
- removed net HDMI1_D0_N: HDMI1.TMDS0-, J1.60
- removed net HDMI1_D0_P: HDMI1.TMDS0SHIELD, J1.58
- removed net HDMI1_D1_N: HDMI1.TMDS1-, J1.54
- removed net HDMI1_D1_P: HDMI1.TMDS1SHIELD, J1.52
- removed net HDMI1_D2_N: HDMI1.TMDS2-, J1.48
- removed net HDMI1_D2_P: HDMI1.TMDS2SHIELD, J1.46
- removed net HDMI1_HOTPLUG: HDMI1.HOTPLUG/HEC+, J1.43
- removed net HDMI1_SCL: HDMI1.SCL, J1.47
- removed net HDMI1_SDA: HDMI1.SDA, J1.45
- removed net HDMI_5V: C4.1, HDMI1.POWER, HDMI2.POWER, IC4.OUT, TP-5VHD.P$1
- removed net ID_SC: GPIO.28, J2.35, JP1.1
- removed net ID_SD: GPIO.27, J2.36, JP1.3
- removed net IN0+: IC6.IN_A_0, J7.19
- removed net IN1-: IC6.IN_B_0, J7.53
- removed net IN10+: IC8.IN_A_1, J7.25
- removed net IN11-: IC8.IN_B_1, J7.59
- removed net IN12+: IC8.IN_A_2, J7.26
- removed net IN13-: IC8.IN_B_2, J7.60
- removed net IN14+: IC8.IN_A_3, J7.27
- removed net IN15-: IC8.IN_B_3, J7.61
- removed net IN2+: IC6.IN_A_1, J7.20
- removed net IN3-: IC6.IN_B_1, J7.54
- removed net IN4+: IC6.IN_A_2, J7.21
- removed net IN5-: IC6.IN_B_2, J7.55
- removed net IN6+: IC6.IN_A_3, J7.22
- removed net IN7-: IC6.IN_B_3, J7.56
- removed net IN8+: IC8.IN_A_0, J7.24
- removed net IN9-: IC8.IN_B_0, J7.58
- removed net LED_NACT: J2.21
- removed net M2_3V3: C12.1, C13.1, C14.1, C15.1, C16.1, C17.1, L1.2, PCIE.VCC1, PCIE.VCC2, PCIE.VCC3, PCIE.VCC4, PCIE.VCC5, PCIE.VCC6, PCIE.VCC7, PCIE.VCC8, PCIE.VCC9, R12.1, TP-VM2.P$1, X2.OUT, X2.VDD
- removed net MISO_SEL: IC16.1C, IC17.IN
- removed net MUX_A_OUTA: IC6.OUT_A, R43.2
- removed net MUX_A_OUTB: IC6.OUT_B, R44.1
- removed net MUX_B_OUTA: IC8.OUT_A, R24.2
- removed net MUX_B_OUTB: IC8.OUT_B, R42.1
- removed net N$10: C13.2, IC5.FB, R12.2, R13.1, TP-M2FB.P$1
- removed net N$11: PCIE.SUSCLK, TP-M2CLK.P$1, X2.CON
- removed net N$12: IC7.OUT+, R20.2
- removed net N$124: IC32.VREF_B, R127.1
- removed net N$125: IC33.VREF_B, R128.1
- removed net N$126: IC35.VREF_B, R129.1
- removed net N$127: IC34.VREF_B, R130.1
- removed net N$13: IC7.OUT-, R21.2
- removed net N$14: C129.2, IC24.OUT, R90.1
- removed net N$15: IC9.OUT+, R22.2
- removed net N$16: IC9.OUT-, R23.2
- removed net N$17: C129.1, IC24.-IN, R87.2, R88.2, R89.1
- removed net N$18: IC10.CONVST, R15.2
- removed net N$19: C72.2, C73.2, R49.1
- removed net N$20: C74.1, R49.2, R50.1
- removed net N$21: IC11.+IN, R50.2
- removed net N$22: C132.1, IC25.-IN, R91.2, R92.2, R93.1
- removed net N$23: C132.2, IC25.OUT, R94.1
- removed net N$24: D3.A, IC14.INP, L3.2
- removed net N$25: C135.1, IC26.-IN, R95.2, R96.2, R97.1
- removed net N$26: C135.2, IC26.OUT, R98.1
- removed net N$27: C138.1, IC27.-IN, R100.2, R101.1, R99.2
- removed net N$28: C138.2, IC27.OUT, R102.1
- removed net N$3: IC3.Y, R5.2
- removed net N$30: C90.1, L3.1, T2.D
- removed net N$31: C141.1, IC28.-IN, R103.2, R104.2, R105.1
- removed net N$32: C86.1, IC14.ENN, IC14.ENP, IC14.PSN, IC14.PSP, IC14.VIN, R14.1
- removed net N$33: C141.2, IC28.OUT, R106.1
- removed net N$34: C144.1, IC29.-IN, R107.2, R108.2, R109.1
- removed net N$35: C91.1, IC14.CP
- removed net N$36: C92.1, IC14.CN
- removed net N$37: D4.C, IC14.OUTN, L4.2
- removed net N$38: R55.2, R55.3, R60.2
- removed net N$39: C103.1, IC15.NR/SS
- removed net N$40: C144.2, IC29.OUT, R110.1
- removed net N$41: C147.1, IC30.-IN, R111.2, R112.2, R113.1
- removed net N$42: R56.2, R56.3, R74.2
- removed net N$43: R19.2, R53.2, R53.3
- removed net N$44: R54.2, R54.3, R58.2
- removed net N$45: J4.17, R61.1
- removed net N$5: ETH1.P17, R9.1
- removed net N$58: C147.2, IC30.OUT, R114.1
- removed net N$59: C150.1, IC31.-IN, R115.2, R116.2, R117.1
- removed net N$6: PCIE.DA5/!DSS!/!LED1, R10.2
- removed net N$60: C150.2, IC31.OUT, R118.1
- removed net N$7: LED2.C, R10.1
- removed net N$8: ETH1.P19, R8.2
- removed net N$9: IC5.LX, L1.1, TP-LX.P$1
- removed net NPWR_LED: IC3.A, J2.95, TP-LED.P$1
- removed net NRPIBOOT: J2.93, JP2.2
- removed net PCIE_CLK_N: J1.12, PCIE.REFCLK_N
- removed net PCIE_CLK_P: J1.10, PCIE.REFCLK_P
- removed net PCIE_NCLKREQ: J1.2, PCIE.!CLKREQ
- removed net PCIE_NRST: J1.9, PCIE.!PERST
- removed net PCIE_NWAKE: J1.4, PCIE.!PEWAKE
- removed net PCIE_PWR_EN: IC5.EN, J1.6, R11.1
- removed net PCIE_RX_N: J1.18, PCIE.PET_P0
- removed net PCIE_RX_P: J1.16, PCIE.PET_N0
- removed net PCIE_TX_N: J1.24, PCIE.PER_P0
- removed net PCIE_TX_P: J1.22, PCIE.PER_N0
- removed net PGA_A_IN+: IC7.IN1+, R43.1
- removed net PGA_A_IN-: IC7.IN1-, IC7.IN2+, R44.2
- removed net PGA_B_IN+: IC9.IN1+, R24.1
- removed net PGA_B_IN-: IC9.IN1-, IC9.IN2+, R42.2
- removed net PMIC_ENABLE: J2.99, JP2.12
- removed net PWM: CON1.P$3, J2.19
- removed net PWR_BUT: J2.92, JP2.14, SW1.2, TP-BTN.P$1
- removed net REFBY2: C71.1, IC10.REFBY2, REFBY2.P$1
- removed net REFM_A: C70.2, IC10.REFM_A
- removed net REFM_B: C110.2, IC10.REFM_B
- removed net REFOUT: C111.1, IC10.REFOUT, REFOUT.P$1
- removed net REFP_A: C70.1, IC10.REFP_A
- removed net REFP_B: C110.1, IC10.REFP_B
- removed net SCL0: J2.80, J3.20
- removed net SCL1: J4.20, JP1.2, R4.2
- removed net SDA0: J2.82, J3.21
- removed net SDA1: J4.21, JP1.4, R3.2
- removed net SDO_A_0: IC10.SDO-0/0A, IC16.1A
- removed net SDO_B_0: IC10.SDO-4/0B, IC16.2A
- removed net SD_CLK: J2.57, SD1.CLK
- removed net SD_CMD: J2.62, SD1.CMD
- removed net SD_DAT0: J2.63, SD1.DAT0
- removed net SD_DAT1: J2.67, SD1.DAT1
- removed net SD_DAT2: J2.69, SD1.DAT2
- removed net SD_DAT3: J2.61, SD1.CD/DAT3
- removed net SD_PWR: C10.1, IC1.OUT, SD1.VDD, TP-VSD.P$1
- removed net SD_PWR_ON: IC1.EN, J2.75
- removed net SPI1_CS0: IC10.!CS, R15.1, R32.1, SPI1_CS0.P$1
- removed net SPI1_CS1: IC7.!CS, R33.1
- removed net SPI1_CS2: IC9.!CS, R34.1
- removed net SYNC_OUT: J2.18, JP2.6
- removed net TACHO: CON1.P$1, J2.16
- removed net TR0_TAP: ETH1.VC1, JP4.3
- removed net TR1_TAP: ETH1.VC2, JP4.1
- removed net TR2_TAP: ETH1.VC3, JP4.2
- removed net TR3_TAP: ETH1.VC4, JP4.4
- removed net TRD0_N: D2.D1-, ETH1.TD1-, J2.10
- removed net TRD0_P: D2.D1+, ETH1.TD1+, J2.12
- removed net TRD1_N: D2.D2+, ETH1.TD2-, J2.6
- removed net TRD1_P: D2.D2-, ETH1.TD2+, J2.4
- removed net TRD2_N: D1.D2+, ETH1.TD3-, J2.9
- removed net TRD2_P: D1.D2-, ETH1.TD3+, J2.11
- removed net TRD3_N: D1.D1-, ETH1.TD4-, J2.5
- removed net TRD3_P: D1.D1+, ETH1.TD4+, J2.3
- removed net USB2_N: J1.3, USBC.D-1, USBC.D-2
- removed net USB2_P: J1.5, USBC.D+1, USBC.D+2
- removed net USB3-0-D_N: J1.36, USB3USBA.D-
- removed net USB3-0-D_P: J1.34, USB3USBA.D+
- removed net USB3-0-RX_N: J1.28, USB3USBA.STDA_SSRX-
- removed net USB3-0-RX_P: J1.30, USB3USBA.STDA_SSRX+
- removed net USB3-0-TX_N: J1.40, USB3USBA.STDA_SSTX-
- removed net USB3-0-TX_P: J1.42, USB3USBA.STDA_SSTX+
- removed net USB3-1-D_N: J1.65, USB3USBB.D-
- removed net USB3-1-D_P: J1.63, USB3USBB.D+
- removed net USB3-1-RX_N: J1.57, USB3USBB.STDA_SSRX-
- removed net USB3-1-RX_P: J1.59, USB3USBB.STDA_SSRX+
- removed net USB3-1-TX_N: J1.69, USB3USBB.STDA_SSTX-
- removed net USB3-1-TX_P: J1.71, USB3USBB.STDA_SSTX+
- removed net USBOTG_ID: J1.1, JP2.10
- removed net VBAT: BT1.+, J2.76, TP-VBAT.P$1
- removed net VBUS_EN: IC2.EN, J1.11
- removed net VFB_12VN: C106.2, IC15.FBN, R56.1, R76.1, VFB12VN.P$1
- removed net VFB_12VP: C107.1, IC15.FBP, R55.1, R73.1, VFB12VP.P$1
- removed net VFB_14VN: C101.2, IC14.FBN, R54.1, R59.1, TP_VFB_14VN.P$1
- removed net VFB_14VP: C100.2, IC14.FBP, R53.1, R57.1, TP_VFB_14VP.P$1
- removed net VOCM_A: IC7.VOCM, R51.2, VOCMA.P$1
- removed net VOCM_B: IC9.VOCM, R52.1, VCOMB.P$1
- removed net VREF_ADC: C46.1, C72.1, C73.1, IC13.-IN, IC13.OUT, IC7.AVDD, IC9.AVDD, R49.3, TP9.P$1
- removed net VREF_ADC/2: C75.1, IC11.-IN, IC11.OUT, R51.1, R52.2, REF/2.P$1
- removed net VREF_ADC_RAW: C48.1, IC12.VREF, IC13.+IN, VREFR.P$1
- removed net VREF_DAC: C125.1, IC23.-IN, IC23.OUT, R100.1, R104.1, R108.1, R112.1, R116.1, R88.1, R92.1, R96.1
- removed net VREF_DAC_OUT: C124.1, IC22.VREF_IO, IC23.+IN, VREF_DAC.P$1
- removed net VREF_TPS: C99.2, IC14.VREF, R58.1, TP_VREF_TPS.P$1
- removed net WL_NDIS: J2.89, JP3.1
- new net !QSPI_SS: IC2.QSPI_SS_N, IC4.!CS, R3.1, R4.2
- new net +1V1: C112.1, C113.1, C114.1, DVDD.P$1, IC2.DVDD, IC2.VREG_VOUT
- new net 5VFB_EXT: IC2.GPIO27/ADC1
- new net ADC_5VP: IC2.GPIO29/ADC3, R72.1, R77.2
- new net ADC_VOUT_REF: IC2.GPIO28/ADC2, R22.2, R23.1
- new net ADC_VUSB: IC2.GPIO26/ADC0, R63.2, R64.1
- new net AVDD: AVDD.P$1, C5.1, C89.1, IC2.ADC_AVDD, IC3.-IN, IC3.OUT
- new net EXT: J1.1, J1.20, JP-EXT-1.2, JP-EXT-2.2
- new net QSPI_SCLK: IC2.QSPI_SCLK, IC4.CLK
- new net QSPI_SD0: IC2.QSPI_SD0, IC4.DI/IO0
- new net QSPI_SD1: IC2.QSPI_SD1, IC4.DO/IO1
- new net QSPI_SD2: IC2.QSPI_SD2, IC4.!WP!/IO2
- new net QSPI_SD3: IC2.QSPI_SD3, IC4.!HOLD!/IO3
- new net RP2040_RST: IC2.RUN, R75.2, RESET.P, X3B.18
- new net RP_USBD_N: IC2.USB_DM, R6.2
- new net RP_USBD_P: IC2.USB_DP, R7.2
- new net RP_XI: C1.1, IC2.XIN, R9.1, X1.CON
- new net RP_XO: IC2.XOUT, R1.2
- new net SPI1_CS: IC2.GPIO13, X3A.29, X3B.29
- new net SWCLK: DBG2.P$1, IC2.SWCLK, X3B.23
- new net SWDIO: DBG2.P$3, IC2.SWDIO, X3B.24
- new net UART0_RX: DBG1.P$1, IC2.GPIO0, X3B.20
- new net UART0_TX: DBG1.P$3, IC2.GPIO1, X3B.21
- new net USBD_N: ESD1.C2, R6.1, USBC.D-1, USBC.D-2
- new net USBD_P: ESD1.C1, R7.1, USBC.D+1, USBC.D+2
- new net USB_BOOT: R4.1, USB_BOOT.P
- new net USB_SHIELD: C115.1, R68.1, USBC.SHIELD
- new net VREF: C3.1, C4.1, IC3.+IN, R2.1, REF1.C, VREF1.P$1
- net +3V3: now also C116.1, C121.1, C27.1, C6.1, C77.1, C80.1, C81.1, C82.1, C83.1, C84.1, C87.1, C88.1, IC1.VOUT, IC2.IOVDD, IC2.USB_VDD, IC2.VREG_VIN, IC3.V+, IC4.VCC, IOVDD.P$1, JP-3V3-1.1, JP-3V3-2.1, R2.2, R3.2, R75.1; no longer C122.1, C123.1, C126.1, C128.1, C131.1, C134.1, C137.1, C140.1, C143.1, C146.1, C149.1, C21.1, C22.1, C25.1, C45.1, C47.1, C49.1, C50.1, C51.1, C64.1, C65.1, C76.1, C9.1, ETH1.P18, ETH1.P20, GPIO.1, GPIO.17, IC1.IN, IC10.AVDD, IC10.DVDD, IC11.V+, IC12.VIN, IC13.V+, IC16.VCC, IC17.V+, IC22.AVDD, IC23.V+, IC24.V+, IC25.V+, IC26.V+, IC27.V+, IC28.V+, IC29.V+, IC3.VCC, IC30.V+, IC31.V+, IC7.DVDD, IC9.DVDD, J2.84, J2.86, J3.22, J4.22, LED1.A, LED2.A, R16.1, R6.1, R61.2, R86.5, R86.6, R86.7, R86.8, TP_3V3.P$1
- net +5V: now also D1.C, IC1.EN, IC1.VIN, JP-EXT-1.1, JP-EXT-2.1, R72.2, X3A.8, X3A.9, X3B.8, X3B.9; no longer C1.1, C18.1, C19.1, C2.1, C20.1, C3.1, C5.1, C85.1, CON1.P$4, GPIO.2, GPIO.4, IC14.INN, IC18.VIN, IC2.IN, IC4.IN, IC5.VIN, J2.77, J2.79, J2.81, J2.83, J2.85, J2.87, J7.18, J7.33, R1.1, R14.2, T2.S, TP-5VP.P$1, TP_5VP.P$1, USBC.VBUS, USBC.VBUS1, USBC.VBUS2, USBC.VBUS3
- net CC1: now also R62.1; no longer J2.94
- net CC2: now also R61.1; no longer J2.96
- net DIO_0: now also J1.2; no longer J7.2
- net DIO_1: now also J1.21; no longer J7.3
- net DIO_10: now also J1.7; no longer J7.12
- net DIO_11: now also J1.26; no longer J7.13
- net DIO_12: now also J1.8; no longer J7.14
- net DIO_13: now also J1.27; no longer J7.15
- net DIO_14: now also J1.9; no longer J7.16
- net DIO_15: now also J1.28; no longer J7.17
- net DIO_16: now also J1.10; no longer J7.36
- net DIO_17: now also J1.29; no longer J7.37
- net DIO_18: now also J1.11; no longer J7.38
- net DIO_19: now also J1.30; no longer J7.39
- net DIO_2: now also J1.3; no longer J7.4
- net DIO_20: now also J1.12; no longer J7.40
- net DIO_21: now also J1.31; no longer J7.41
- net DIO_22: now also J1.13; no longer J7.42
- net DIO_23: now also J1.32; no longer J7.43
- net DIO_24: now also J1.14; no longer J7.44
- net DIO_25: now also J1.33; no longer J7.45
- net DIO_26: now also J1.15; no longer J7.46
- net DIO_27: now also J1.34; no longer J7.47
- net DIO_28: now also J1.16; no longer J7.48
- net DIO_29: now also J1.35; no longer J7.49
- net DIO_3: now also J1.22; no longer J7.5
- net DIO_30: now also J1.17; no longer J7.50
- net DIO_31: now also J1.36; no longer J7.51
- net DIO_4: now also J1.4; no longer J7.6
- net DIO_5: now also J1.23; no longer J7.7
- net DIO_6: now also J1.5; no longer J7.8
- net DIO_7: now also J1.24; no longer J7.9
- net DIO_8: now also J1.6; no longer J7.10
- net DIO_9: now also J1.25; no longer J7.11
- net DIO_EN: now also IC2.GPIO9, R10.2, R11.2, R127.2, R8.2, X3A.11; no longer R41.1
- net DIO_LEVEL_SELECT: now also IC2.GPIO7, X3A.13; no longer R40.1
- net DIO_RESET: now also IC2.GPIO8, X3A.12; no longer R39.1
- net GND: now also C112.2, C113.2, C114.2, C115.2, C116.2, C77.2, C78.2, C79.2, C80.2, C81.2, C82.2, C83.2, C84.2, C87.2, C88.2, C89.2, DBG1.P$2, DBG1.P$4, DBG2.P$2, DBG2.P$4, ESD1.A, IC2.TESTEN, IC3.V-, J1.18, J1.MH1, J1.MH2, R23.2, R5.2, R61.2, R62.2, R64.2, R68.2, R77.1, REF1.A, RESET.S, USB_BOOT.S, X1.VDD, X1.VSS, X3A.10, X3A.14, X3A.15, X3A.16, X3A.25, X3A.30, X3A.31, X3A.32, X3B.10, X3B.14, X3B.15, X3B.16, X3B.19, X3B.22, X3B.25, X3B.30, X3B.31, X3B.32; no longer 2230.1, 2242.1, 2260.1, 2280.1, BT1.-, C10.2, C102.2, C103.2, C104.2, C105.1, C108.2, C109.2, C11.2, C111.2, C12.2, C122.2, C123.2, C124.2, C125.2, C126.2, C127.2, C128.2, C130.2, C131.2, C133.2, C134.2, C136.2, C137.2, C139.2, C14.2, C140.2, C142.2, C143.2, C145.2, C146.2, C148.2, C149.2, C15.2, C16.2, C17.2, C18.2, C19.2, C20.2, C21.2, C22.2, C23.2, C24.1, C25.2, C42.2, C43.1, C45.2, C46.2, C47.2, C48.2, C49.2, C50.2, C51.2, C52.2, C53.2, C54.2, C55.2, C56.2, C57.2, C58.2, C59.2, C60.2, C61.2, C62.2, C63.2, C64.2, C65.2, C66.2, C67.2, C68.2, C69.2, C7.2, C71.2, C74.2, C75.2, C76.2, C8.2, C85.2, C86.2, C9.2, C90.2, C91.2, C92.2, C93.2, C94.2, C95.2, C96.2, C97.2, C98.2, C99.1, CON1.P$2, D1.GND, D2.GND, ETH1.SHIELD, GPIO.14, GPIO.20, GPIO.25, GPIO.30, GPIO.34, GPIO.39, GPIO.6, GPIO.9, HDMI1.SHIELD, HDMI1.TMDS0+, HDMI1.TMDS2+, HDMI1.TMDSCLOCK+, HDMI1.TMDSDATA1+, HDMI1.UTILITY/HEAC+, HDMI2.SHIELD, HDMI2.TMDS0+, HDMI2.TMDS2+, HDMI2.TMDSCLOCK+, HDMI2.TMDSDATA1+, HDMI2.UTILITY/HEAC+, IC10.GND, IC10.PAD, IC11.V-, IC12.GND, IC13.V-, IC14.AGND, IC14.PGND, IC15.GND, IC15.PAD, IC16.GND, IC17.V-, IC18.GND, IC22.GND, IC23.V-, IC24.V-, IC25.V-, IC26.V-, IC27.V-, IC28.V-, IC29.V-, IC3.GND, IC30.V-, IC31.V-, IC5.PGND, IC5.SGND, IC6.GND, IC7.AVSS, IC7.DVSS, IC7.IN2-, IC7.IOUT_HV, IC7.IOUT_LV, IC8.GND, IC9.AVSS, IC9.DVSS, IC9.IN2-, IC9.IOUT_HV, IC9.IOUT_LV, J1.13, J1.14, J1.20, J1.25, J1.26, J1.31, J1.32, J1.37, J1.38, J1.44, J1.50, J1.55, J1.56, J1.61, J1.62, J1.67, J1.68, J1.7, J1.73, J1.74, J1.79, J1.8, J1.80, J1.85, J1.86, J1.91, J1.92, J1.97, J1.98, J2.1, J2.13, J2.14, J2.2, J2.22, J2.23, J2.32, J2.33, J2.42, J2.43, J2.52, J2.53, J2.59, J2.60, J2.65, J2.66, J2.7, J2.71, J2.74, J2.8, J2.98, J3.1, J3.10, J3.13, J3.16, J3.19, J3.4, J3.7, J3.MH1, J3.MH2, J4.1, J4.10, J4.13, J4.16, J4.19, J4.4, J4.7, J4.MH1, J4.MH2, J7.1, J7.23, J7.28, J7.34, J7.35, J7.57, J7.62, J7.68, J7.MH1, J7.MH2, JP2.1, JP2.11, JP2.13, JP2.3, JP2.5, JP2.7, JP2.9, JP3.2, JP3.4, L4.1, PCIE.GND1, PCIE.GND10, PCIE.GND11, PCIE.GND12, PCIE.GND13, PCIE.GND14, PCIE.GND2, PCIE.GND3, PCIE.GND4, PCIE.GND5, PCIE.GND6, PCIE.GND7, PCIE.GND8, PCIE.GND9, PCIE.S1, PCIE.S2, R1.2, R103.1, R107.1, R11.2, R111.1, R115.1, R13.2, R2.2, R57.2, R73.2, R87.1, R91.1, R95.1, R99.1, SD1.MT1, SD1.MT2, SD1.MT3, SD1.MT4, SD1.VSS, SW1.1, SW1.3, SW1.4, TP_GND.P$1, USB3USBA.GND, USB3USBA.GND_DRAIN, USB3USBA.SHIELD, USB3USBB.GND, USB3USBB.GND_DRAIN, USB3USBB.SHIELD, USBC.SHIELD, X2.VSS
- net N$1: now also C2.1, R1.1, R9.2, X1.OUT; no longer IC2.ILIM, R2.1
- net N$2: now also JP-3V3-2.2, X3B.1; no longer LED1.C, R5.1
- net N$4: now also JP-3V3-1.2, X3A.1; no longer C11.1, ETH1.CT1, ETH1.CT2, ETH1.CT3, ETH1.CT4
- net SPI0_CS0: now also CS0.P$1, IC2.GPIO5, X3A.2; no longer DIO_CS.P$1, R29.1
- net SPI0_CS1: now also CS1.P$1, IC2.GPIO6, X3A.3; no longer R30.1
- net SPI0_MISO: now also IC2.GPIO4, MISO.P$1, X3A.7, X3B.7; no longer R27.1
- net SPI0_MOSI: now also IC2.GPIO3, MOSI.P$1, X3A.6, X3B.6; no longer IC22.DIN, R28.1
- net SPI0_SCK: now also IC2.GPIO2, SCK.P$1, X3A.5, X3B.5; no longer IC22.SCLK, R26.1
- net SPI1_MISO: now also IC2.GPIO12, X3A.26, X3B.26; no longer IC16.1B, IC16.2B, IC7.SDO, IC9.SDO, R18.1
- net SPI1_MOSI: now also IC2.GPIO11, X3A.27, X3B.27; no longer IC10.SDI, IC7.SDI, IC9.SDI, R17.1
- net SPI1_SCK: now also IC2.GPIO10, X3A.28, X3B.28; no longer IC10.SCLK, IC7.SCK, IC9.SCK, R25.1
- net VBUS: now also C78.1, C79.1, D1.A, ESD1.C3, R5.1, R63.1, USBC.VBUS, USBC.VBUS1, USBC.VBUS2, USBC.VBUS3, VBUS.P$1; no longer C6.1, C7.1, C8.1, IC2.OUT, TP-VBUS.P$1, USB3USBA.VBUS, USB3USBB.VBUS
- net V_OUT_REF: now also IC32.VREF_B, IC33.VREF_B, IC34.VREF_B, IC35.VREF_B, R10.1, R11.1, R127.1, R22.1, R8.1; no longer R127.2, R128.2, R129.2, R130.2
Other:
- note added: "12MHZ CRYSTAL"
- note added: "3.3V SYSTEM LDO"
- note added: "ADC VREF"
- note added: "BOARD CONNECTOR"
- note added: "DEBUG"
- note added: "DECOUPLING"
- note added: "DIGITAL CONNECTOR"
- note added: "DIGITAL IO"
- note added: "DIGITAL IO TESTPOINTS"
- note added: "David Sipos / DvidMakesThings"
- note added: "Enable SWD Debugging on Raspberry Pi: Install OpenOCD (sudo apt install openocd) Configure /boot/config.txt to enable GPIO-based debugging."
- note added: "POWER AND OUTPUT"
- note added: "RP2040 FLASH"
- note added: "RP2040 MCU"
- note added: "Rev 1.0"
- note added: "USB-C CONNECTOR"
- note removed: "+/-14V to +/12V LDO"
- note removed: "0 0 1 OUT0"
- note removed: "0 1 1 OUT1"
- note removed: "1 0 1 OUT2"
- note removed: "1 1 1 OUT3"
- note removed: "1000 BASE ETHERNET"
- note removed: "2.5V VREF"
- note removed: "3.3V TARGET LDO"
- note removed: "40-PIN GPIO HEADER"
- note removed: "5V to +/-14V BOOST CONVERTER"
- note removed: "A1 A0 EN ON"
- note removed: "ADC ON SPI1"
- note removed: "ADS9234R ADC"
- note removed: "ANALOG-IN TESTPOINTS"
- note removed: "ANALOG-OUT DAC"
- note removed: "ANALOG-OUT OUTPUT DRIVERS"
- note removed: "ANALOG-OUT TESTPOINTS"
- note removed: "CURRENT LIMIT SWITCH"
- note removed: "Choose R_ISOLATION = 68 Ω: 1. Stability with Capacitive Load: The combination of R_ISO and C_LOAD creates a low-pass filter. The cutoff frequency is: f_c = 1 / (2 * π * R_ISO * C_LOAD) For R_ISO = 68 Ω and C_LOAD = 20 nF: f_c = 1 / (2 * π * 68 * 20e-9) ≈ 117.2 kHz 2. Voltage Drop Across R_ISO: The voltage drop is: V_drop = I_load * R_ISO"
- note removed: "DAC8568 Output Calculation: V_OUT = (1 + R_FB/R_G2 + R_FB/R_G1) * V_DAC - (R_FB/R_G2) * V_REF Given: Supply voltage: +/-12V Reference voltage (V_REF): 2.5V DAC resolution: 16 bits Desired output range: -12V to +12V 1. Determine the Gain (G): G = (V_OUT_max - V_OUT_min) / (V_DAC_max - V_DAC_min) G = (12 - (-12)) / (2.5 - 0) = 24 / 2.5 = 9.6 2. Solve for Resistor Ratios: G = 1 + R_FB/R_G2 + R_FB/R_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"
- note removed: "DIO ON SPI0"
- note removed: "DPHY1 JUMPERS"
- note removed: "DSI/CSI CONNECTORS"
- note removed: "DUAL-HDMI CONNECTOR"
- note removed: "FAN CONNECTOR"
- note removed: "GPIO VOLTAGE SELECT"
- note removed: "IN0+ AND IN1-"
- note removed: "IN10+ AND IN11-"
- note removed: "IN12+ AND IN13-"
- note removed: "IN14+ AND IN15-"
- note removed: "IN2+ AND IN3-"
- note removed: "IN4+ AND IN5-"
- note removed: "IN6+ AND IN7-"
- note removed: "IN8+ AND IN9-"
- note removed: "INPUT MULTIPLEXER"
- note removed: "IO-GPIO JUMPERS"
- note removed: "JUMPERS"
- note removed: "MICRO-SD SOCKET"
- note removed: "Negative Channel: - Known Values: - VBUF = 1.184 V - VOUTN = -12 V - R2N = 10 kΩ - Formula: R1N = -(VOUTN × R2N) / VBUF - Calculation: R1N = -(-12 × 10) / 1.184 R1N = (120 / 1.184) = 101.4 kΩ - Closest Resistor Value (0.1% Tolerance): R1N = 101 kΩ Final Resistor Values: - Negative Channel: - R1N = 101 kΩ - R2N = 10 kΩ - Calculated VOUTN ≈ -12.0 V Negative Channel: - Target VOUTN = -12 V, adjustme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"
- note removed: "Negative Output (Vout_neg = -14V): - Given: - R1 = 1.3 MΩ - Calculated R2 ≈ 136.3 kΩ - Nearest E96 Standard Value: - R2 = 137 kΩ - Resulting Output Voltage: - Vout = 1.213 × (1 + R1 / R2) - Vout = 1.213 × (1 + 1300 / 137) ≈ 14.01 V - Final Pair: - R1 = 1.3 MΩ - R2 = 137 kΩ Negative Channel: - Target VOUTN = -14 V, adjustment range: -12.6 V to -15.4 V. - Configuration: - R2N = 137 kΩ (fixed). - R1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"
- note removed: "PCIE POWER SUPPLY"
- note removed: "PCIE-M.2 M-KEY CONNECTOR"
- note removed: "PGA"
- note removed: "POWER BUTTON AND LED"
- note removed: "Positive Channel: - Known Values: - VFBP = 1.184 V - VOUTP = 12 V - R2P = 10 kΩ - Formula: R1P = (VOUTP / VFBP - 1) × R2P - Calculation: R1P = (12 / 1.184 - 1) × 10 R1P = (10.14 - 1) × 10 = 91.4 kΩ - Closest Resistor Value (0.1% Tolerance): R1P = 91.5 kΩ Final Resistor Values: - Positive Channel: - R1P = 91.5 kΩ - R2P = 10 kΩ - Calculated VOUTP ≈ 12.0 V Positive Channel: - Target VOUTP = 12 V, ad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"
- note removed: "Positive Output (Vout_pos = 14V): - Given: - R1 = 976 kΩ - Calculated R2 ≈ 102.3 kΩ - Nearest E96 Standard Value: - R2 = 102 kΩ - Resulting Output Voltage: - Vout = 1.213 × (1 + R1 / R2) - Vout = 1.213 × (1 + 976 / 102) ≈ 13.98 V - Final Pair: - R1 = 976 kΩ - R2 = 102 kΩ Positive Channel: - Target VOUTP = 14 V, adjustment range: 12.6 V to 15.4 V. - Configuration: - R2P = 102 kΩ (fixed). - R1P = 9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"
- note removed: "RF DISABLE"
- note removed: "RTC BATTERY"
- note removed: "SPI0"
- note removed: "SPI1"
- note removed: "TEST CONNECTOR"
- note removed: "TESTPOINTS POWER"
- note removed: "USB-C POWER CONNECTOR"
- note removed: "USB3 CONNECTORS"
- note removed: "X X 0 -"

Commit message: Baseboard design ready
Changed lines of the file:
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@@
 <part name="R10" library="ds_passive" deviceset="R" device="0402" package3d_urn="urn:adsk.eagle:package:46683744/2" value="200K"/>
 <part name="R11" library="ds_passive" deviceset="R" device="0402" package3d_urn="urn:adsk.eagle:package:46683744/2" value="200K"/>
+<part name="NC15" library="ds_passive" deviceset="NC" device=""/>
 </parts>
 <sheets>
@@
 <attribute name="VALUE" x="63.5" y="152.4" size="1.778" layer="96" rot="R180"/>
 </instance>
+<instance part="NC15" gate="G$1" x="281.94" y="170.18" smashed="yes"/>
 </instances>
 <busses>
